Commit message: update rotations in urdf

File: manipulator_description/urdf/manipulator.urdf (robot description, URDF)
Before this commit: robot robot_diff, 9 links, 8 joints
Joints:
- joint base_motor1: origin xyz=0 0 0.09 rpy=1.571 0 1.571 -> xyz=0 0 0.09 rpy=0 0 1.571
- joint elo1_motor2: origin xyz=-0.04 0.0 -0.027 rpy=0 1.571 1.571 -> xyz=-0.04 0.0 -0.027 rpy=-1.571 1.571 1.571
- joint elo2_motor2: axis 1 0 0 -> 0 0 1; origin xyz=${0.2275-0.22765252} -0.04 ${-0.067+0.0381+0.02935} rpy=0 0 -1.571 -> xyz=0.0 0.0 -0.04 rpy=0 0 -1.571
- joint motor1_elo1: origin xyz=0.0 0.045 0.0 rpy=1.571 0 0 -> xyz=0.0 0.0 0.036 rpy=3.14 0 0
- joint motor2_fix: origin xyz=0.0 -0.094 0.0 rpy=1.571 0 0 -> xyz=0.0 0.0 -0.093 rpy=1.571 0 0
- joint motor3r_elo2: origin xyz=0.026 ${0.47211676-0.02086310} -0.03 rpy=0 1.571 0 -> xyz=-0.026 0.455 -0.027 rpy=0 3.14 0
- joint motor3t_elo2: origin xyz=-0.026 ${0.47211676-0.02086310} -0.03 rpy=0 -1.571 0 -> xyz=-0.026 0.455 0.027 rpy=0 0 0

Commit message: updating urdf

File: manipulator_description/urdf/manipulator.urdf (robot description, URDF)
Before this commit: robot robot_diff, 9 links, 8 joints
Links:
- added link Elo3, mass 0.59823526; collision mesh filename=package://manipulator_description/meshes/elo3.dae; visual mesh filename=package://manipulator_description/meshes/elo3.dae
Joints:
- removed joint motor3t_elo2
- added joint motor3r_motor3t: type fixed, parent Motor3R, child Motor3T, origin xyz=0 0 -0.05 rpy=0 3.14 0
- added joint motores_elo3: type revolute, parent Motor3T, child Elo3, origin xyz=0 ${0.019-0.02} -0.0375 rpy=0 0 0, axis 0 0 1, limit lower=-1.46 upper=2.46 effort=1000.0 velocity=0.5
- joint motor3r_elo2: origin xyz=-0.026 0.455 -0.027 rpy=0 3.14 0 -> xyz=-0.028 0.451 -0.024 rpy=0 3.14 0

Commit message: update urdf frame 4

File: manipulator_description/urdf/manipulator.urdf (robot description, URDF)
Before this commit: robot robot_diff, 10 links, 9 joints
Links:
- added link Frame4, mass 0.01873963; collision mesh filename=package://manipulator_description/meshes/frame4.dae; visual mesh filename=package://manipulator_description/meshes/frame4.dae
- added link Motor4, mass 0.16499216; collision mesh filename=package://manipulator_description/meshes/motor4.dae; visual mesh filename=package://manipulator_description/meshes/motor4.dae
Joints:
- added joint elo3_frame4: type revolute, parent Elo3, child Frame4, origin xyz=0 0.45 0.012 rpy=0 0 0, axis 0 0 1, limit lower=-1.90 upper=1.90 effort=1000.0 velocity=0.5
- added joint elo3_motor4: type fixed, parent Elo3, child Motor4, origin xyz=0 0.45 0.013 rpy=0 0 0

Commit message: update urdf withou changes in  link2

File: manipulator_description/urdf/manipulator.urdf (robot description, URDF)
Before this commit: robot robot_diff, 12 links, 11 joints
Joints:
- removed joint elo3_frame4
- added joint motor4_frame4: type revolute, parent Motor4, child Frame4, origin xyz=0 0 0 rpy=0 0 0, axis 0 0 1, limit lower=-1.90 upper=1.90 effort=1000.0 velocity=0.5
- joint motores_elo3: origin xyz=0 ${0.019-0.02} -0.0375 rpy=0 0 0 -> xyz=0 0.001 -0.0375 rpy=0 0 0

Commit message: change joint 2

File: manipulator_description/urdf/manipulator.urdf (robot description, URDF)
Before this commit: robot robot_diff, 12 links, 11 joints
Links:
- link Elo2: mass 0.88616841 -> 1.09212028
Joints:
- joint elo2_motor2: origin xyz=0.0 0.0 -0.04 rpy=0 0 -1.571 -> xyz=-0.0008 0 0 rpy=0 0 -1.571
- joint motor3r_elo2: origin xyz=-0.028 0.451 -0.024 rpy=0 3.14 0 -> xyz=0.03 0.451 0 rpy=0 0 0
