Commit message: Position base

File: manipulator_description/urdf/base.xacro (robot description, xacro)
@@ -24,5 +24,5 @@
         <parent link="base_link"/>
         <child link="base_to_manipulator"/>
-        <origin rpy="0 0 0" xyz="0.45 0 0"/>
+        <origin rpy="0 0 0" xyz="0.6 0 0"/>
       </joint>
 </robot>
