Commit message: redo aruco

File: manipulator_description/urdf/box.urdf.xacro (robot description, xacro)
@@ -4,5 +4,5 @@
   </link>
   <xacro:include filename="$(find manipulator_description)/urdf/caixa.xacro"/>
-  <xacro:include filename="$(find manipulator_description)/urdf/box_aruco.xacro"/>
+  <!-- <xacro:include filename="$(find manipulator_description)/urdf/box_aruco.xacro"/> -->
   <xacro:include filename="$(find manipulator_description)/urdf/tag.xacro"/>
 </robot>

File: manipulator_description/urdf/tag.xacro (robot description, xacro)
@@ -3,5 +3,5 @@
     <link name="tag_aruco_13">
         <inertial>
-            <origin xyz="0 0 0" rpy="1.571 0 0 "/>
+            <origin xyz="0 0 0" rpy="-1.571 0 0 "/>
             <mass value="1.0"/>
             <inertia ixx="0.0741666666"  ixy="0.0"  ixz="0.0" iyy="0.0585461666" iyz="0.0" izz="0.02604166666" />
@@ -14,5 +14,5 @@
         </collision>
         <visual>
-            <origin xyz="0.0 0.0 0.0" rpy="-1.571 1.571 0.0"/>
+            <origin xyz="0.0 0.0 0.0" rpy="1.571 -1.571 0.0"/>
             <geometry>
                 <mesh filename="package://manipulator_description/meshes/tag.dae"/>
@@ -28,6 +28,6 @@
         </gazebo>
     <joint name="box_to_tag" type="fixed">
-        <origin rpy="0 -1.571 0" xyz="0.0 0.0 0.0"/>
-        <parent link="box_aruco"/>
+        <origin rpy="0 1.571 0" xyz="0.0 -0.103 0.1"/>
+        <parent link="caixa"/>
         <child link = "tag_aruco_13"/>
     </joint>

Commit message: Update xacro files

File: manipulator_description/urdf/box.urdf.xacro (robot description, xacro)
@@ -1,6 +1,8 @@
 <?xml version="1.0" encoding="utf-8"?>
 <robot xmlns:xacro="http://www.ros.org/wiki/xacro" name="timon">
+  <link name="map">
+  </link>
   <xacro:include filename="$(find manipulator_description)/urdf/caixa.xacro"/>
-  <!-- <xacro:include filename="$(find manipulator_description)/urdf/box_aruco.xacro"/> -->
   <xacro:include filename="$(find manipulator_description)/urdf/tag.xacro"/>
+  <xacro:include filename="$(find manipulator_description)/urdf/botao.xacro"/>
 </robot>

File: manipulator_description/urdf/caixa.xacro (robot description, xacro)
@@ -17,11 +17,11 @@
       <origin rpy="0 0 0" xyz="0 0 0"/>
       <mass value="7.83641898"/>
-      <inertia ixx="1.14585569e-1" ixy="0" ixz="-4.92675504e-9" iyx="0" iyy="1.11284013e-1" iyz="-9.69960810e-4" izx="-4.92675504e-9" izy="-9.69960810e-4" izz="8.63706684e-2"/>
+      <inertia ixx="1.14439574e-1" ixy="0" ixz="-4.92675504e-9" iyx="0" iyy="1.11258168e-1" iyz="-1.02434023e-3" izx="-4.92675504e-9" izy="-1.02434023e-3" izz="8.62491763e-2"/>
     </inertial>
   </link>
- <!-- <joint name="base_to_caixa" type="fixed">
+ <joint name="base_to_caixa" type="fixed">
     <parent link="map"/>
     <child link="caixa"/>
     <origin rpy="0 0 1.571" xyz="0 0 0"/>
-  </joint>  -->
+  </joint>
 </robot>
