Commit message: adding box orientation

File: manipulator_description/urdf/tag.xacro (robot description, xacro)
@@ -28,5 +28,5 @@
         </gazebo>
     <joint name="box_to_tag" type="fixed">
-        <origin rpy="0 0 3.1415" xyz="0.0 0.06 0"/> <!--caixa na vertical: rpy="0 0 0" -->  <!-- horizontal: rpy="0 0 3.1415" -->
+        <origin rpy="0 0 0" xyz="0.0 -0.06 0"/> <!--caixa na vertical: rpy="0 0 0" -->  <!-- horizontal: rpy="0 0 3.1415" -->
         <parent link="botao"/>
         <child link = "tag_aruco_4"/>
