Commit message: adding push_button_4 to generic situations

File: manipulator_description/urdf/botao_horizontal.xacro (robot description, xacro)
@@ -20,6 +20,6 @@
     </inertial>
   </link>
-  <link name="fake_botao">
-  </link>
+  <link name="fake_botao"/>
+  <link name="botao_press"/>
  <joint name="caixa_to_botao" type="fixed">
     <parent link="caixa"/>
@@ -29,6 +29,11 @@
     <limit lower="0.0" upper="0.00" effort="1" velocity="1"/> -->
   </joint>
+  <joint name = "botao_pressed" type="fixed">
+    <parent link="botao"/>
+    <child link="botao_press"/>
+    <origin rpy="0.0 0.0 0.0" xyz="0.0 0.0 0.1"/>
+  </joint>
   <joint name ="botao_fake" type ="fixed">
-    <parent link="botao"/>
+    <parent link="botao_press"/>
     <child link="fake_botao"/>
     <origin rpy="0.0 0.0 0.0" xyz="0.0 0.0 0.2"/>

File: manipulator_description/urdf/botao_vertical.xacro (robot description, xacro)
@@ -20,6 +20,6 @@
     </inertial>
   </link>
-  <link name="fake_botao">
-  </link>
+  <link name="fake_botao"/>
+  <link name="botao_press"/>
  <joint name="caixa_to_botao" type="fixed">
     <parent link="caixa"/>
@@ -29,4 +29,9 @@
     <limit lower="0.0" upper="0.00" effort="1" velocity="1"/> -->
   </joint>
+  <joint name = "botao_pressed" type="fixed">
+    <parent link="botao"/>
+    <child link="botao_press"/>
+    <origin rpy="0.0 0.0 0.0" xyz="0.0 0.0 0.1"/>
+  </joint>
   <joint name ="botao_fake" type ="fixed">
     <parent link="botao"/>
