Commit message: fixing xacro files

File: manipulator_description/urdf/botao.xacro (robot description, xacro)
@@ -20,5 +20,5 @@
     </inertial>
   </link>
- <joint name="base_to_botao" type="fixed">
+ <joint name="caixa_to_botao" type="fixed">
     <parent link="caixa"/>
     <child link="botao"/>

File: manipulator_description/urdf/box.urdf.xacro (robot description, xacro)
@@ -1,6 +1,4 @@
 <?xml version="1.0" encoding="utf-8"?>
 <robot xmlns:xacro="http://www.ros.org/wiki/xacro" name="timon">
-  <link name="map">
-  </link>
   <xacro:include filename="$(find manipulator_description)/urdf/caixa.xacro"/>
   <xacro:include filename="$(find manipulator_description)/urdf/tag.xacro"/>

File: manipulator_description/urdf/caixa.xacro (robot description, xacro)
@@ -20,8 +20,3 @@
     </inertial>
   </link>
- <joint name="base_to_caixa" type="fixed">
-    <parent link="map"/>
-    <child link="caixa"/>
-    <origin rpy="0 0 1.571" xyz="0 0 0"/>
-  </joint>
 </robot>

Commit message: sending arm to button pose

File: manipulator_description/urdf/botao.xacro (robot description, xacro)
@@ -20,8 +20,17 @@
     </inertial>
   </link>
+  <link name="fake_botao">
+  </link>
  <joint name="caixa_to_botao" type="fixed">
     <parent link="caixa"/>
     <child link="botao"/>
     <origin rpy="1.571 0 0" xyz="0 -0.1165 0.215"/>
+    <!-- <axis xyz="0 1 0"/>
+    <limit lower="0.0" upper="0.00" effort="1" velocity="1"/> -->
+  </joint>
+  <joint name ="botao_fake" type ="fixed">
+    <parent link="botao"/>
+    <child link="fake_botao"/>
+    <origin rpy="0.0 0.0 0.0" xyz="0.0 0.0 0.1"/>
   </joint>
 </robot>

File: manipulator_description/urdf/caixa.xacro (robot description, xacro)
@@ -16,5 +16,5 @@
     <inertial>
       <origin rpy="0 0 0" xyz="0 0 0"/>
-      <mass value="7.83641898"/>
+      <mass value="100.83641898"/>
       <inertia ixx="1.14439574e-1" ixy="0" ixz="-4.92675504e-9" iyx="0" iyy="1.11258168e-1" iyz="-1.02434023e-3" izx="-4.92675504e-9" izy="-1.02434023e-3" izz="8.62491763e-2"/>
     </inertial>

Commit message: considering new possibilites to box orientation

File: manipulator_description/urdf/botao.xacro (robot description, xacro)
@@ -25,5 +25,5 @@
     <parent link="caixa"/>
     <child link="botao"/>
-    <origin rpy="1.571 0 0" xyz="0 -0.1165 0.215"/>
+    <origin rpy="0 0 0" xyz="0 0.215 0.1165"/> <!-- caixa na vertical: <origin rpy="1.571 0 0" xyz="0 -0.1165 0.215"/> -->
     <!-- <axis xyz="0 1 0"/>
     <limit lower="0.0" upper="0.00" effort="1" velocity="1"/> -->

File: manipulator_description/urdf/box.urdf.xacro (robot description, xacro)
@@ -7,5 +7,5 @@
   <xacro:include filename="$(find manipulator_description)/urdf/botao.xacro"/>
   <joint name="base_to_box" type="fixed">
-    <origin xyz="-0.4 0.0 1.56" rpy="0.0 0.0 1.571"/>
+    <origin xyz="-0.4 0.0 1.66" rpy="0 0 -1.571"/>   <!--vertical: xyz="-0.4 0.0 1.56" rpy="0 0 1.571"-->
     <parent link="box_link"/>
     <child link="caixa"/>

File: manipulator_description/urdf/caixa.xacro (robot description, xacro)
@@ -3,5 +3,5 @@
   <link name="caixa">
     <visual>
-      <origin rpy="0 0 0" xyz="0 0 0"/>
+      <origin rpy="-1.571 0 0" xyz="0 0 0"/> <!-- caixa na vertical : rpy="0 0 0" xyz="0 0 0-->
       <geometry>
         <mesh filename="package://manipulator_description/meshes/caixa.dae"/>
@@ -9,5 +9,5 @@
     </visual>
     <collision>
-      <origin rpy="0 0 0" xyz="0 0 0"/>
+      <origin rpy="-1.571 0 0" xyz="0 0 0"/>
       <geometry>
         <mesh filename="package://manipulator_description/meshes/caixa.stl"/>
@@ -15,6 +15,6 @@
     </collision>
     <inertial>
-      <origin rpy="0 0 0" xyz="0 0 0"/>
-      <mass value="100.83641898"/>
+      <origin rpy="-1.571 0 0" xyz="0 0 0"/>
+      <mass value="7.83641898"/>
       <inertia ixx="1.14439574e-1" ixy="0" ixz="-4.92675504e-9" iyx="0" iyy="1.11258168e-1" iyz="-1.02434023e-3" izx="-4.92675504e-9" izy="-1.02434023e-3" izz="8.62491763e-2"/>
     </inertial>

File: manipulator_description/urdf/tag.xacro (robot description, xacro)
@@ -3,5 +3,5 @@
     <link name="tag_aruco_4">
         <inertial>
-            <origin xyz="0 0 0" rpy="0 0 0 "/> <!-- "-1.571 0 0 " -->
+            <origin xyz="0 0 0" rpy="0 0 0 "/>
             <mass value="1.0"/>
             <inertia ixx="0.0741666666"  ixy="0.0"  ixz="0.0" iyy="0.0585461666" iyz="0.0" izz="0.02604166666" />
@@ -14,5 +14,5 @@
         </collision>
         <visual>
-            <origin xyz="0.0 0.0 0.0" rpy="0 0 0"/>   <!-- "1.571 -1.571 0.0" -->
+            <origin xyz="0.0 0.0 0.0" rpy="0 0 0"/>
             <geometry>
                 <mesh filename="package://manipulator_description/meshes/tag.dae"/>
@@ -28,5 +28,5 @@
         </gazebo>
     <joint name="box_to_tag" type="fixed">
-        <origin rpy="0 0 0" xyz="0.0 -0.1 -0.013"/> <!--"0.0 -0.103 0.1" -->
+        <origin rpy="0 0 3.1415" xyz="0.0 -0.1 -0.013"/> <!--caixa na vertical: rpy="0 0 0" -->
         <parent link="botao"/>
         <child link = "tag_aruco_4"/>

Commit message: fixing box orientation

File: manipulator_description/urdf/botao.xacro (robot description, xacro)
@@ -25,5 +25,5 @@
     <parent link="caixa"/>
     <child link="botao"/>
-    <origin rpy="0 0 0" xyz="0 0.215 0.1165"/> <!-- caixa na vertical: <origin rpy="1.571 0 0" xyz="0 -0.1165 0.215"/> -->
+    <origin rpy="1.571 0 0" xyz="0 -0.1165 0.215"/> <!--vertical: rpy="1.571 0 0" xyz="0 -0.1165 0.215" --> <!-- horizontal: rpy="0 0 0" xyz="0 0.215 0.1165"-->
     <!-- <axis xyz="0 1 0"/>
     <limit lower="0.0" upper="0.00" effort="1" velocity="1"/> -->

File: manipulator_description/urdf/box.urdf.xacro (robot description, xacro)
@@ -7,5 +7,5 @@
   <xacro:include filename="$(find manipulator_description)/urdf/botao.xacro"/>
   <joint name="base_to_box" type="fixed">
-    <origin xyz="-0.4 0.0 1.66" rpy="0 0 -1.571"/>   <!--vertical: xyz="-0.4 0.0 1.56" rpy="0 0 1.571"-->
+    <origin xyz="-0.4 0.0 1.56" rpy="0 0 1.571"/>   <!--vertical: xyz="-0.4 0.0 1.56" rpy="0 0 1.571"--> <!-- horizontal: xyz="-0.4 0.0 1.66" rpy="0 0 -1.571"-->
     <parent link="box_link"/>
     <child link="caixa"/>

File: manipulator_description/urdf/caixa.xacro (robot description, xacro)
@@ -3,5 +3,5 @@
   <link name="caixa">
     <visual>
-      <origin rpy="-1.571 0 0" xyz="0 0 0"/> <!-- caixa na vertical : rpy="0 0 0" xyz="0 0 0-->
+      <origin rpy="0 0 0" xyz="0 0 0"/> <!-- vertical : rpy="0 0 0" xyz="0 0 0"--> <!-- horizontal: rpy="-1.571 0 0" xyz="0 0 0"-->
       <geometry>
         <mesh filename="package://manipulator_description/meshes/caixa.dae"/>
@@ -9,5 +9,5 @@
     </visual>
     <collision>
-      <origin rpy="-1.571 0 0" xyz="0 0 0"/>
+      <origin rpy="0 0 0" xyz="0 0 0"/> <!-- vertical : rpy="0 0 0" xyz="0 0 0"--> <!-- horizontal: rpy="-1.571 0 0" xyz="0 0 0"-->
       <geometry>
         <mesh filename="package://manipulator_description/meshes/caixa.stl"/>
@@ -15,5 +15,5 @@
     </collision>
     <inertial>
-      <origin rpy="-1.571 0 0" xyz="0 0 0"/>
+      <origin rpy="0 0 0" xyz="0 0 0"/> <!-- vertical : rpy="0 0 0" xyz="0 0 0"--> <!-- horizontal: rpy="-1.571 0 0" xyz="0 0 0"-->
       <mass value="7.83641898"/>
       <inertia ixx="1.14439574e-1" ixy="0" ixz="-4.92675504e-9" iyx="0" iyy="1.11258168e-1" iyz="-1.02434023e-3" izx="-4.92675504e-9" izy="-1.02434023e-3" izz="8.62491763e-2"/>

File: manipulator_description/urdf/tag.xacro (robot description, xacro)
@@ -28,5 +28,5 @@
         </gazebo>
     <joint name="box_to_tag" type="fixed">
-        <origin rpy="0 0 3.1415" xyz="0.0 -0.1 -0.013"/> <!--caixa na vertical: rpy="0 0 0" -->
+        <origin rpy="0 0 0" xyz="0.0 -0.1 -0.013"/> <!--caixa na vertical: rpy="0 0 0" -->  <!-- horizontal: rpy="0 0 3.1415" -->
         <parent link="botao"/>
         <child link = "tag_aruco_4"/>

Commit message: delet old files

File: manipulator_description/urdf/botao.xacro (robot description, xacro)
@@ -25,5 +25,5 @@
     <parent link="caixa"/>
     <child link="botao"/>
-    <origin rpy="1.571 0 0" xyz="0 -0.1165 0.215"/> <!--vertical: rpy="1.571 0 0" xyz="0 -0.1165 0.215" --> <!-- horizontal: rpy="0 0 0" xyz="0 0.215 0.1165"-->
+    <origin rpy="0 0 0" xyz="0 0.215 0.1165"/> <!--vertical: rpy="1.571 0 0" xyz="0 -0.1165 0.215" --> <!-- horizontal: rpy="0 0 0" xyz="0 0.215 0.1165"-->
     <!-- <axis xyz="0 1 0"/>
     <limit lower="0.0" upper="0.00" effort="1" velocity="1"/> -->

File: manipulator_description/urdf/box.urdf.xacro (robot description, xacro)
@@ -7,5 +7,5 @@
   <xacro:include filename="$(find manipulator_description)/urdf/botao.xacro"/>
   <joint name="base_to_box" type="fixed">
-    <origin xyz="-0.4 0.0 1.56" rpy="0 0 1.571"/>   <!--vertical: xyz="-0.4 0.0 1.56" rpy="0 0 1.571"--> <!-- horizontal: xyz="-0.4 0.0 1.66" rpy="0 0 -1.571"-->
+    <origin xyz="-0.4 0.0 1.66" rpy="0 0 -1.571"/>   <!--vertical: xyz="-0.4 0.0 1.56" rpy="0 0 1.571"--> <!-- horizontal: xyz="-0.4 0.0 1.66" rpy="0 0 -1.571"-->
     <parent link="box_link"/>
     <child link="caixa"/>

File: manipulator_description/urdf/caixa.xacro (robot description, xacro)
@@ -3,5 +3,5 @@
   <link name="caixa">
     <visual>
-      <origin rpy="0 0 0" xyz="0 0 0"/> <!-- vertical : rpy="0 0 0" xyz="0 0 0"--> <!-- horizontal: rpy="-1.571 0 0" xyz="0 0 0"-->
+      <origin rpy="-1.571 0 0" xyz="0 0 0"/> <!-- vertical : rpy="0 0 0" xyz="0 0 0"--> <!-- horizontal: rpy="-1.571 0 0" xyz="0 0 0"-->
       <geometry>
         <mesh filename="package://manipulator_description/meshes/caixa.dae"/>
@@ -9,5 +9,5 @@
     </visual>
     <collision>
-      <origin rpy="0 0 0" xyz="0 0 0"/> <!-- vertical : rpy="0 0 0" xyz="0 0 0"--> <!-- horizontal: rpy="-1.571 0 0" xyz="0 0 0"-->
+      <origin rpy="-1.571 0 0" xyz="0 0 0"/> <!-- vertical : rpy="0 0 0" xyz="0 0 0"--> <!-- horizontal: rpy="-1.571 0 0" xyz="0 0 0"-->
       <geometry>
         <mesh filename="package://manipulator_description/meshes/caixa.stl"/>
@@ -15,5 +15,5 @@
     </collision>
     <inertial>
-      <origin rpy="0 0 0" xyz="0 0 0"/> <!-- vertical : rpy="0 0 0" xyz="0 0 0"--> <!-- horizontal: rpy="-1.571 0 0" xyz="0 0 0"-->
+      <origin rpy="-1.571 0 0" xyz="0 0 0"/> <!-- vertical : rpy="0 0 0" xyz="0 0 0"--> <!-- horizontal: rpy="-1.571 0 0" xyz="0 0 0"-->
       <mass value="7.83641898"/>
       <inertia ixx="1.14439574e-1" ixy="0" ixz="-4.92675504e-9" iyx="0" iyy="1.11258168e-1" iyz="-1.02434023e-3" izx="-4.92675504e-9" izy="-1.02434023e-3" izz="8.62491763e-2"/>

File: manipulator_description/urdf/tag.xacro (robot description, xacro)
@@ -28,5 +28,5 @@
         </gazebo>
     <joint name="box_to_tag" type="fixed">
-        <origin rpy="0 0 0" xyz="0.0 -0.1 -0.013"/> <!--caixa na vertical: rpy="0 0 0" -->  <!-- horizontal: rpy="0 0 3.1415" -->
+        <origin rpy="0 0 3.1415" xyz="0.0 -0.1 -0.013"/> <!--caixa na vertical: rpy="0 0 0" -->  <!-- horizontal: rpy="0 0 3.1415" -->
         <parent link="botao"/>
         <child link = "tag_aruco_4"/>

Commit message: Add test_rr

File: manipulator_description/urdf/botao.xacro (robot description, xacro)
@@ -20,6 +20,6 @@
     </inertial>
   </link>
-  <link name="fake_botao">
-  </link>
+  <link name="fake_botao"/>
+  <link name="botao_press"/>
  <joint name="caixa_to_botao" type="fixed">
     <parent link="box_link"/>
@@ -27,6 +27,11 @@
     <origin rpy="0 0 0" xyz="0 0 0"/>
   </joint>
+  <joint name="botao_pressed" type="fixed">
+    <parent link="botao"/>
+    <child link="botao_press"/>
+    <origin rpy="0 0 0" xyz="0 0 0"/>  <!-- 0.0825-->
+  </joint>
   <joint name ="botao_fake" type ="fixed">
-    <parent link="botao"/>
+    <parent link="botao_press"/>
     <child link="fake_botao"/>
     <origin rpy="0.0 0.0 0.0" xyz="0.0 0.0 0.25"/>

Commit message: add tests

File: manipulator_description/urdf/botao.xacro (robot description, xacro)
@@ -30,8 +30,8 @@
     <parent link="botao"/>
     <child link="botao_press"/>
-    <origin rpy="0 0 0" xyz="0 0 0"/>  <!-- 0.0825-->
+    <origin rpy="0 0 0" xyz="0 0 0.075"/>
   </joint>
   <joint name ="botao_fake" type ="fixed">
-    <parent link="botao_press"/>
+    <parent link="botao"/>
     <child link="fake_botao"/>
     <origin rpy="0.0 0.0 0.0" xyz="0.0 0.0 0.25"/>
