Commit message: update xacro files

File: manipulator_description/robots/hand.xacro (robot description, xacro)
@@ -11,48 +11,4 @@
     <link name="${ns}_hand">
       <visual>
-        <origin xyz="0.0 0.0 0.0" rpy="0.0 0.0 0.0" />
-        <geometry>
-          <mesh filename="package://manipulator_description/meshes/visual/link9.dae"/>
-        </geometry>
-      </visual>
-      <collision>
-        <origin xyz="0.0 0.0 0.0" rpy="0.0 0.0 0.0" />
-        <geometry>
-          <mesh filename="package://manipulator_description/meshes/collision/link9.stl"/>
-        </geometry>
-      </collision>
-      <inertial>
-        <origin xyz="0.0 0.0 0.0" rpy="0.0 0.0 0.0"/>
-        <mass value="0.16499216"/>
-        <inertia ixx="7.88952550e-5"  ixy="-3.13065901e-9"  ixz="4.40693303e-9" iyy="4.39861799e-5" iyz="-2.02737764e-6" izz="6.23603662e-5" />
-      </inertial>
-    </link>
-    <link name="${ns}_hand1">
-      <visual>
-        <origin xyz="0.0 0.0 0.0" rpy="1.571 0.0 0.0" />
-        <geometry>
-          <mesh filename="package://manipulator_description/meshes/visual/link10.dae"/>
-        </geometry>
-      </visual>
-      <collision>
-        <origin xyz="0.0 0.0 0.0" rpy="1.571 0.0 0.0" />
-        <geometry>
-          <mesh filename="package://manipulator_description/meshes/collision/link10.stl"/>
-        </geometry>
-      </collision>
-      <inertial>
-        <origin xyz="0.0 0.0 0.0" rpy="1.571 0.0 0.0"/>
-        <mass value="0.007"/>
-        <inertia ixx="1.48840827e-6"  ixy="2.49592487e-8"  ixz="5.30644674e-12" iyy="2.08108627e-6" iyz="2.38181240e-14" izz="6.88193128e-7" />
-      </inertial>
-    </link>
-    <joint name="${ns}_hand_joint1" type="continuous">
-      <origin rpy="0 0 1.571" xyz="0 0 0.025"/>
-      <parent link="${ns}_hand"/>
-      <child link="${ns}_hand1"/>
-      <axis xyz="0 0 1" rpy="0 0 0"/>
-    </joint>
-    <link name="${ns}_hand2">
-      <visual>
         <origin xyz="0.0225 -0.007 0.0" rpy="0.0 0.0 0.0" />
         <geometry>
@@ -63,5 +19,5 @@
         <origin xyz="0.0225 -0.007 0.0" rpy="0.0 0.0 0.0" />
         <geometry>
-          <mesh filename="package://manipulator_description/meshes/collision/link11.stl"/>
+          <mesh filename="package://manipulator_description/meshes/visual/link11.dae"/>
         </geometry>
       </collision>
@@ -72,10 +28,5 @@
       </inertial>
     </link>
-    <joint name="${ns}_hand_joint_2" type="fixed">
-      <origin rpy="1.5701 0.0 0.0" xyz="0.0 -0.001 0.055"/>
-      <parent link="${ns}_hand1"/>
-      <child link="${ns}_hand2"/>
-    </joint>
-   <link name="${ns}_hand3">
+   <link name="${ns}_hand1">
       <visual>
         <origin xyz="0.0 0.0 0.0" rpy="0.0 1.571 0.0" />
@@ -87,5 +38,5 @@
         <origin xyz="0.0 0.0 0.0" rpy="0.0 1.571 0.0" />
         <geometry>
-          <mesh filename="package://manipulator_description/meshes/collision/link12.stl"/>
+          <mesh filename="package://manipulator_description/meshes/visual/link12.dae"/>
         </geometry>
       </collision>
@@ -96,8 +47,9 @@
       </inertial>
     </link>
-    <joint name="${ns}_hand_joint_3" type="revolute">
+    <joint name="${ns}_hand_joint_1" type="revolute">
+      <safety_controller k_position="100.0" k_velocity="40.0" soft_lower_limit="-1.90" soft_upper_limit="1.90"/>
       <origin rpy="0.0 0.0 0.0" xyz="0.0 0.0 0.0"/>
-      <parent link="${ns}_hand2"/>
-      <child link="${ns}_hand3"/>
+      <parent link="${ns}_hand"/>
+      <child link="${ns}_hand1"/>
       <axis xyz="0 0 1"/>
       <limit effort="1000.0" lower="-1.90" upper="1.90" velocity="0.5"/>

File: manipulator_description/robots/timon_arm.xacro (robot description, xacro)
@@ -10,5 +10,5 @@
       <collision>
         <geometry>
-          <mesh filename="package://${description_pkg}/meshes/collision/link0.stl"/>
+          <mesh filename="package://${description_pkg}/meshes/visual/link0.dae"/>
         </geometry>
       </collision>
@@ -29,5 +29,5 @@
         <origin xyz="0 0 0" rpy="1.571 0 0" />
         <geometry>
-          <mesh filename="package://${description_pkg}/meshes/collision/link1.stl"/>
+          <mesh filename="package://${description_pkg}/meshes/visual/link1.dae"/>
         </geometry>
       </collision>
@@ -53,5 +53,5 @@
         <origin xyz="0 0 0" rpy="-3.14 0 0" />
         <geometry>
-          <mesh filename="package://${description_pkg}/meshes/collision/link2.stl"/>
+          <mesh filename="package://${description_pkg}/meshes/visual/link2.dae"/>
         </geometry>
       </collision>
@@ -63,4 +63,5 @@
     </link>
     <joint name="${arm_id}_joint2" type="continuous">
+      <safety_controller k_position="100.0" k_velocity="40.0"/>
       <origin rpy="3.14 0 0" xyz="0 0 0.036"/>
       <parent link="${arm_id}_link1"/>
@@ -78,5 +79,5 @@
         <origin xyz="0 0 0" rpy="1.571 0 0" />
         <geometry>
-          <mesh filename="package://${description_pkg}/meshes/collision/link3.stl"/>
+          <mesh filename="package://${description_pkg}/meshes/visual/link3.dae"/>
         </geometry>
       </collision>
@@ -102,5 +103,5 @@
         <origin xyz="0 0 0" rpy="1.571 0 0" />
         <geometry>
-          <mesh filename="package://${description_pkg}/meshes/collision/link4.stl"/>
+          <mesh filename="package://${description_pkg}/meshes/visual/link4.dae"/>
         </geometry>
       </collision>
@@ -126,5 +127,5 @@
         <origin xyz="-0.0292 0.2289 -0.04" rpy="0 1.571 0" />
         <geometry>
-          <mesh filename="package://${description_pkg}/meshes/collision/link5.stl"/>
+          <mesh filename="package://${description_pkg}/meshes/visual/link5.dae"/>
         </geometry>
       </collision>
@@ -136,5 +137,6 @@
     </link>
     <joint name="${arm_id}_joint5" type="revolute">
-      <origin rpy="0 -1.571 -1.571" xyz="-0.0008 0.093 0"/>
+      <safety_controller k_position="100.0" k_velocity="40.0" soft_lower_limit="-1.77" soft_upper_limit="1.77"/>
+      <origin rpy="0 -1.571 -1.571" xyz="-0.0008 0.093 0.001"/>
       <parent link="${arm_id}_link4"/>
       <child link="${arm_id}_link5"/>
@@ -152,5 +154,5 @@
         <origin xyz="0.0 0.0 0.0" rpy="0 0 -0.75" />
         <geometry>
-          <mesh filename="package://${description_pkg}/meshes/collision/link6.stl"/>
+          <mesh filename="package://${description_pkg}/meshes/visual/link6.dae"/>
         </geometry>
       </collision>
@@ -176,5 +178,5 @@
         <origin xyz="0.0 0.0 0.0" rpy="0 0 0.75" />
         <geometry>
-          <mesh filename="package://${description_pkg}/meshes/collision/link7.stl"/>
+          <mesh filename="package://${description_pkg}/meshes/visual/link7.dae"/>
         </geometry>
       </collision>
@@ -200,5 +202,5 @@
         <origin xyz="-0.01 0.015 0.0" rpy="0.0 1.571 0.0" />
         <geometry>
-          <mesh filename="package://${description_pkg}/meshes/collision/link8.stl"/>
+          <mesh filename="package://${description_pkg}/meshes/visual/link8.dae"/>
         </geometry>
       </collision>
@@ -210,4 +212,5 @@
     </link>
     <joint name="${arm_id}_joint8" type="revolute">
+      <safety_controller k_position="100.0" k_velocity="40.0" soft_lower_limit="-0.95" soft_upper_limit="2.36"/>
       <origin rpy="0.0 0.0 0.0" xyz="0.0 0.001 -0.0375"/>
       <parent link="${arm_id}_link7"/>
@@ -216,4 +219,53 @@
       <limit effort="1000.0" lower="-0.95" upper="2.36" velocity="0.5"/>
     </joint>
+    <link name="${arm_id}_link9">
+      <visual>
+        <origin xyz="0.0 0.0 0.0" rpy="0.0 0.0 0.0" />
+        <geometry>
+          <mesh filename="package://manipulator_description/meshes/visual/link9.dae"/>
+        </geometry>
+      </visual>
+      <collision>
+        <origin xyz="0.0 0.0 0.0" rpy="0.0 0.0 0.0" />
+        <geometry>
+          <mesh filename="package://manipulator_description/meshes/visual/link9.dae"/>
+        </geometry>
+      </collision>
+      <inertial>
+        <origin xyz="0.0 0.0 0.0" rpy="0.0 0.0 0.0"/>
+        <mass value="0.16499216"/>
+        <inertia ixx="7.88952550e-5"  ixy="-3.13065901e-9"  ixz="4.40693303e-9" iyy="4.39861799e-5" iyz="-2.02737764e-6" izz="6.23603662e-5" />
+      </inertial>
+    </link>
+    <joint name="${arm_id}_joint9" type="fixed">
+      <origin rpy="0 -1.571 -1.571" xyz="0 0.41 0.013"/>
+      <parent link="${arm_id}_link8"/>
+      <child link="${arm_id}_link9"/>
+    </joint>
+    <link name="${arm_id}_link10">
+      <visual>
+        <origin xyz="0.0 0.0 0.0" rpy="1.571 0.0 0.0" />
+        <geometry>
+          <mesh filename="package://manipulator_description/meshes/visual/link10.dae"/>
+        </geometry>
+      </visual>
+      <collision>
+        <origin xyz="0.0 0.0 0.0" rpy="1.571 0.0 0.0" />
+        <geometry>
+          <mesh filename="package://manipulator_description/meshes/visual/link10.dae"/>
+        </geometry>
+      </collision>
+      <inertial>
+        <origin xyz="0.0 0.0 0.0" rpy="1.571 0.0 0.0"/>
+        <mass value="0.007"/>
+        <inertia ixx="1.48840827e-6"  ixy="2.49592487e-8"  ixz="5.30644674e-12" iyy="2.08108627e-6" iyz="2.38181240e-14" izz="6.88193128e-7" />
+      </inertial>
+    </link>
+    <joint name="${arm_id}_joint10" type="continuous">
+      <origin rpy="0 0 1.571" xyz="0 0 0.025"/>
+      <parent link="${arm_id}_link9"/>
+      <child link="${arm_id}_link10"/>
+      <axis xyz="0 0 1" rpy="0 0 0"/>
+    </joint>
   </xacro:macro>
 </robot>

File: manipulator_description/robots/timon_arm_hand.urdf.xacro (robot description, xacro)
@@ -4,4 +4,4 @@
   <xacro:include filename="$(find manipulator_description)/robots/hand.xacro"/>
   <xacro:timon_arm />
-  <xacro:hand ns="timon" rpy="0 -1.571 -1.571" xyz="0 0.41 0.013" connected_to="timon_link8"/>
+  <xacro:hand ns="timon" rpy="1.5701 0.0 0.0" xyz="0.0 -0.001 0.055" connected_to="timon_link10"/>
 </robot>

Commit message: organized xacro files

File: manipulator_description/robots/hand.xacro (robot description, xacro)
@@ -11,48 +11,4 @@
     <link name="${ns}_hand">
       <visual>
-        <origin xyz="0.0 0.0 0.0" rpy="0.0 0.0 0.0" />
-        <geometry>
-          <mesh filename="package://manipulator_description/meshes/visual/link9.dae"/>
-        </geometry>
-      </visual>
-      <collision>
-        <origin xyz="0.0 0.0 0.0" rpy="0.0 0.0 0.0" />
-        <geometry>
-          <mesh filename="package://manipulator_description/meshes/collision/link9.stl"/>
-        </geometry>
-      </collision>
-      <inertial>
-        <origin xyz="0.0 0.0 0.0" rpy="0.0 0.0 0.0"/>
-        <mass value="0.16499216"/>
-        <inertia ixx="7.88952550e-5"  ixy="-3.13065901e-9"  ixz="4.40693303e-9" iyy="4.39861799e-5" iyz="-2.02737764e-6" izz="6.23603662e-5" />
-      </inertial>
-    </link>
-    <link name="${ns}_hand1">
-      <visual>
-        <origin xyz="0.0 0.0 0.0" rpy="1.571 0.0 0.0" />
-        <geometry>
-          <mesh filename="package://manipulator_description/meshes/visual/link10.dae"/>
-        </geometry>
-      </visual>
-      <collision>
-        <origin xyz="0.0 0.0 0.0" rpy="1.571 0.0 0.0" />
-        <geometry>
-          <mesh filename="package://manipulator_description/meshes/collision/link10.stl"/>
-        </geometry>
-      </collision>
-      <inertial>
-        <origin xyz="0.0 0.0 0.0" rpy="1.571 0.0 0.0"/>
-        <mass value="0.007"/>
-        <inertia ixx="1.48840827e-6"  ixy="2.49592487e-8"  ixz="5.30644674e-12" iyy="2.08108627e-6" iyz="2.38181240e-14" izz="6.88193128e-7" />
-      </inertial>
-    </link>
-    <joint name="${ns}_hand_joint1" type="continuous">
-      <origin rpy="0 0 1.571" xyz="0 0 0.025"/>
-      <parent link="${ns}_hand"/>
-      <child link="${ns}_hand1"/>
-      <axis xyz="0 0 1" rpy="0 0 0"/>
-    </joint>
-    <link name="${ns}_hand2">
-      <visual>
         <origin xyz="0.0225 -0.007 0.0" rpy="0.0 0.0 0.0" />
         <geometry>
@@ -63,5 +19,5 @@
         <origin xyz="0.0225 -0.007 0.0" rpy="0.0 0.0 0.0" />
         <geometry>
-          <mesh filename="package://manipulator_description/meshes/collision/link11.stl"/>
+          <mesh filename="package://manipulator_description/meshes/visual/link11.dae"/>
         </geometry>
       </collision>
@@ -72,10 +28,5 @@
       </inertial>
     </link>
-    <joint name="${ns}_hand_joint_2" type="fixed">
-      <origin rpy="1.5701 0.0 0.0" xyz="0.0 -0.001 0.055"/>
-      <parent link="${ns}_hand1"/>
-      <child link="${ns}_hand2"/>
-    </joint>
-   <link name="${ns}_hand3">
+   <link name="${ns}_hand1">
       <visual>
         <origin xyz="0.0 0.0 0.0" rpy="0.0 1.571 0.0" />
@@ -87,5 +38,5 @@
         <origin xyz="0.0 0.0 0.0" rpy="0.0 1.571 0.0" />
         <geometry>
-          <mesh filename="package://manipulator_description/meshes/collision/link12.stl"/>
+          <mesh filename="package://manipulator_description/meshes/visual/link12.dae"/>
         </geometry>
       </collision>
@@ -96,11 +47,22 @@
       </inertial>
     </link>
-    <joint name="${ns}_hand_joint_3" type="revolute">
+    <joint name="${ns}_hand_joint_1" type="revolute">
+      <safety_controller k_position="100.0" k_velocity="40.0" soft_lower_limit="-1.90" soft_upper_limit="1.90"/>
       <origin rpy="0.0 0.0 0.0" xyz="0.0 0.0 0.0"/>
-      <parent link="${ns}_hand2"/>
-      <child link="${ns}_hand3"/>
+      <parent link="${ns}_hand"/>
+      <child link="${ns}_hand1"/>
       <axis xyz="0 0 1"/>
       <limit effort="1000.0" lower="-1.90" upper="1.90" velocity="0.5"/>
     </joint>
+    <transmission name="trans_timon_hand_joint_1">
+        <type>transmission_interface/SimpleTransmission</type>
+        <joint name="timon_hand_joint_1">
+            <hardwareInterface>hardware_interface/EffortJointInterface</hardwareInterface>
+        </joint>
+        <actuator name="timon_hand_joint_1_motor">
+            <hardwareInterface>hardware_interface/EffortJointInterface</hardwareInterface>
+            <mechanicalReduction>1</mechanicalReduction>
+        </actuator>
+    </transmission>
   </xacro:macro>
 </robot>

File: manipulator_description/robots/timon_arm.xacro (robot description, xacro)
@@ -2,4 +2,18 @@
 <robot xmlns:xacro="http://www.ros.org/wiki/xacro" name="timon">
   <xacro:macro name="timon_arm" params="arm_id:='timon' description_pkg:='manipulator_description' connected_to:='' xyz:='0 0 0' rpy:='0 0 0'">
+    <link name="invisible_link">
+      <visual>
+        <origin xyz="0 0 0" rpy="0 0 0" />
+        <geometry>
+          <box size="0.000001 0.000001 0.000001"/>
+        </geometry>
+      </visual>
+      <collision>
+        <origin xyz="0 0 0" rpy="0 0 0" />
+        <geometry>
+          <box size="0.000001 0.000001 0.000001"/>
+        </geometry>
+      </collision>
+    </link>
     <link name="${arm_id}_link0">
       <visual>
@@ -21,7 +35,7 @@
       </inertial>
     </link>
-     <joint name ="base_to_base_link" type="fixed">
-        <origin rpy="0 0 -1.571" xyz="0 0 0.1"/>
-        <parent link="base_to_manipulator"/>
+     <joint name ="invisble_joint" type="fixed">
+        <origin rpy="0 0 0" xyz="0 0 0"/>
+        <parent link="invisible_link"/>
         <child link = "${arm_id}_link0"/>
       </joint>

File: manipulator_description/robots/timon_arm_hand.urdf.xacro (robot description, xacro)
@@ -1,11 +1,4 @@
 <?xml version="1.0" encoding="utf-8"?>
 <robot xmlns:xacro="http://www.ros.org/wiki/xacro" name="timon">
-  <link name ="base_link">
-  </link>
-  <xacro:include filename="$(find manipulator_description)/urdf/base.xacro"/>
-  <xacro:include filename="$(find manipulator_description)/robots/timon_arm.xacro"/>
-  <xacro:include filename="$(find manipulator_description)/robots/hand.xacro"/>
-  <xacro:timon_arm />
-  <xacro:hand ns="timon" rpy="1.5701 0.0 0.0" xyz="0.0 -0.001 0.055" connected_to="timon_link9"/>
   <gazebo>
       <plugin name="gazebo_ros_control" filename="libgazebo_ros_control.so">
@@ -13,3 +6,7 @@
       </plugin>
   </gazebo>
+  <xacro:include filename="$(find manipulator_description)/robots/timon_arm.xacro"/>
+  <xacro:include filename="$(find manipulator_description)/robots/hand.xacro"/>
+  <xacro:timon_arm />
+  <xacro:hand ns="timon" rpy="1.5701 0.0 0.0" xyz="0.0 -0.001 0.055" connected_to="timon_link9"/>
 </robot>

Commit message: new moveit files

File: manipulator_description/robots/hand.xacro (robot description, xacro)
@@ -55,4 +55,14 @@
       <limit effort="1000.0" lower="-1.90" upper="1.90" velocity="0.5"/>
     </joint>
+    <transmission name="trans_timon_hand_joint_1">
+        <type>transmission_interface/SimpleTransmission</type>
+        <joint name="timon_hand_joint_1">
+            <hardwareInterface>hardware_interface/EffortJointInterface</hardwareInterface>
+        </joint>
+        <actuator name="timon_hand_joint_1_motor">
+            <hardwareInterface>hardware_interface/EffortJointInterface</hardwareInterface>
+            <mechanicalReduction>1</mechanicalReduction>
+        </actuator>
+    </transmission>
   </xacro:macro>
 </robot>

File: manipulator_description/robots/timon_arm.xacro (robot description, xacro)
@@ -2,5 +2,17 @@
 <robot xmlns:xacro="http://www.ros.org/wiki/xacro" name="timon">
   <xacro:macro name="timon_arm" params="arm_id:='timon' description_pkg:='manipulator_description' connected_to:='' xyz:='0 0 0' rpy:='0 0 0'">
-    <link name = "base_link">
+    <link name="invisible_link">
+      <visual>
+        <origin xyz="0 0 0" rpy="0 0 0" />
+        <geometry>
+          <box size="0.000001 0.000001 0.000001"/>
+        </geometry>
+      </visual>
+      <collision>
+        <origin xyz="0 0 0" rpy="0 0 0" />
+        <geometry>
+          <box size="0.000001 0.000001 0.000001"/>
+        </geometry>
+      </collision>
     </link>
     <link name="${arm_id}_link0">
@@ -23,7 +35,7 @@
       </inertial>
     </link>
-      <joint name ="base_to_arm" type="fixed">
+     <joint name ="invisble_joint" type="fixed">
         <origin rpy="0 0 0" xyz="0 0 0"/>
-        <parent link="base_link"/>
+        <parent link="invisible_link"/>
         <child link = "${arm_id}_link0"/>
       </joint>
@@ -253,4 +265,44 @@
       <axis xyz="0 0 1" rpy="0 0 0"/>
     </joint>
+    <transmission name="trans_timon_joint1">
+        <type>transmission_interface/SimpleTransmission</type>
+        <joint name="timon_joint1">
+            <hardwareInterface>hardware_interface/PositionJointInterface</hardwareInterface>
+        </joint>
+        <actuator name="timon_joint1_motor">
+            <hardwareInterface>hardware_interface/PositionJointInterface</hardwareInterface>
+            <mechanicalReduction>1</mechanicalReduction>
+        </actuator>
+    </transmission>
+    <transmission name="trans_timon_joint4">
+        <type>transmission_interface/SimpleTransmission</type>
+        <joint name="timon_joint4">
+            <hardwareInterface>hardware_interface/PositionJointInterface</hardwareInterface>
+        </joint>
+        <actuator name="timon_joint4_motor">
+            <hardwareInterface>hardware_interface/PositionJointInterface</hardwareInterface>
+            <mechanicalReduction>1</mechanicalReduction>
+        </actuator>
+    </transmission>
+    <transmission name="trans_timon_joint7">
+        <type>transmission_interface/SimpleTransmission</type>
+        <joint name="timon_joint7">
+            <hardwareInterface>hardware_interface/PositionJointInterface</hardwareInterface>
+        </joint>
+        <actuator name="timon_joint7_motor">
+            <hardwareInterface>hardware_interface/PositionJointInterface</hardwareInterface>
+            <mechanicalReduction>1</mechanicalReduction>
+        </actuator>
+    </transmission>
+    <transmission name="trans_timon_joint9">
+        <type>transmission_interface/SimpleTransmission</type>
+        <joint name="timon_joint9">
+            <hardwareInterface>hardware_interface/PositionJointInterface</hardwareInterface>
+        </joint>
+        <actuator name="timon_joint9_motor">
+            <hardwareInterface>hardware_interface/PositionJointInterface</hardwareInterface>
+            <mechanicalReduction>1</mechanicalReduction>
+        </actuator>
+    </transmission>
     <!-- <link name="${arm_id}_link11">
       <visual>

File: manipulator_description/robots/timon_arm_hand.urdf.xacro (robot description, xacro)
@@ -1,4 +1,9 @@
 <?xml version="1.0" encoding="utf-8"?>
 <robot xmlns:xacro="http://www.ros.org/wiki/xacro" name="timon">
+  <gazebo>
+      <plugin name="gazebo_ros_control" filename="libgazebo_ros_control.so">
+          <robotNamespace>timon</robotNamespace>
+      </plugin>
+  </gazebo>
   <xacro:include filename="$(find manipulator_description)/robots/timon_arm.xacro"/>
   <xacro:include filename="$(find manipulator_description)/robots/hand.xacro"/>
