Commit message: urdf camera + plugin

File: manipulator_description/robots/timon_arm_hand_base.urdf.xacro (robot description, xacro)
@@ -5,4 +5,5 @@
   <xacro:include filename="$(find manipulator_description)/urdf/base.xacro"/>
   <xacro:include filename="$(find manipulator_description)/robots/timon_arm_hand.urdf.xacro"/>
+  <xacro:include filename="$(find manipulator_description)/robots/camera.xacro"/>
     <joint name ="base_to_base_link" type="fixed">
         <origin rpy="0 0 -1.571" xyz="0 0 0.1"/>
@@ -10,3 +11,8 @@
         <child link = "invisible_link"/>
     </joint>
+    <joint name ="base_to_camera" type="fixed">
+        <origin rpy="1.571 3.1415 -1.571" xyz="0.0661 0.426 0.0123"/>
+        <parent link="timon_link7"/>
+        <child link = "camera"/>
+    </joint>
 </robot>

Commit message: adding camera

File: manipulator_description/robots/timon_arm_hand_base.urdf.xacro (robot description, xacro)
@@ -5,4 +5,5 @@
   <xacro:include filename="$(find manipulator_description)/urdf/base.xacro"/>
   <xacro:include filename="$(find manipulator_description)/robots/timon_arm_hand.urdf.xacro"/>
+  <xacro:include filename="$(find manipulator_description)/robots/camera.xacro"/>
     <joint name ="base_to_base_link" type="fixed">
         <origin rpy="0 0 -1.571" xyz="0 0 0.1"/>
@@ -10,3 +11,8 @@
         <child link = "invisible_link"/>
     </joint>
+    <joint name ="base_to_camera" type="fixed">
+        <origin rpy="-1.571 3.1415 -1.571" xyz="0.0661 0.426 0.0123"/>
+        <parent link="timon_link7"/>
+        <child link = "camera"/>
+    </joint>
 </robot>

Commit message: inserting aruco in world

File: manipulator_description/robots/timon_arm_hand_base.urdf.xacro (robot description, xacro)
@@ -3,4 +3,5 @@
   <link name ="base_link">
   </link>
+  <xacro:include filename="$(find manipulator_description)/robots/tag.xacro"/>
   <xacro:include filename="$(find manipulator_description)/urdf/base.xacro"/>
   <xacro:include filename="$(find manipulator_description)/robots/timon_arm_hand.urdf.xacro"/>
@@ -16,3 +17,8 @@
         <child link = "camera"/>
     </joint>
+    <joint name="base_to_tag" type="fixed">
+        <origin rpy="0 0 0" xyz="0 0 0"/>
+        <parent link="base_link"/>
+        <child link="box_tag" />
+    </joint>
 </robot>

Commit message: adding box xacro

File: manipulator_description/robots/timon_arm_hand_base.urdf.xacro (robot description, xacro)
@@ -3,5 +3,5 @@
   <link name ="base_link">
   </link>
-  <xacro:include filename="$(find manipulator_description)/robots/tag.xacro"/>
+  <xacro:include filename="$(find manipulator_description)/urdf/caixa.xacro"/>
   <xacro:include filename="$(find manipulator_description)/urdf/base.xacro"/>
   <xacro:include filename="$(find manipulator_description)/robots/timon_arm_hand.urdf.xacro"/>
@@ -17,8 +17,3 @@
         <child link = "camera"/>
     </joint>
-    <joint name="base_to_tag" type="fixed">
-        <origin rpy="0 0 0" xyz="0 0 0"/>
-        <parent link="base_link"/>
-        <child link="box_tag" />
-    </joint>
 </robot>

Commit message: adding aruco marker

File: manipulator_description/robots/timon_arm_hand_base.urdf.xacro (robot description, xacro)
@@ -7,4 +7,5 @@
   <xacro:include filename="$(find manipulator_description)/robots/timon_arm_hand.urdf.xacro"/>
   <xacro:include filename="$(find manipulator_description)/robots/camera.xacro"/>
+  <xacro:include filename="$(find manipulator_description)/urdf/tag.xacro"/>
     <joint name ="base_to_base_link" type="fixed">
         <origin rpy="0 0 -1.571" xyz="0 0 0.1"/>

File: manipulator_description/urdf/tag.xacro (robot description, xacro)
@@ -10,9 +10,9 @@
             <origin xyz="0.0 0.0 0.0" rpy="0.0 0.0 0.0"/>
             <geometry>
-                <box size="0.2 0.2 0.2"/>
+                <box size="0.1 0.1 0.1"/>
             </geometry>
         </collision>
         <visual>
-            <origin xyz="0.0 0.0 0.0" rpy="0.0 0.0 0.0"/>
+            <origin xyz="0.0 0.0 0.0" rpy="-1.571 1.571 0.0"/>
             <geometry>
                 <mesh filename="package://manipulator_description/meshes/tag.dae"/>
@@ -27,3 +27,8 @@
             <fdir1>1 0 0</fdir1>
         </gazebo>
+    <joint name="caixa_to_tag" type="fixed">
+        <origin rpy="0 0 0" xyz="0.0 -0.10 0.10"/>
+        <parent link="caixa"/>
+        <child link = "box_tag"/>
+    </joint>
 </robot>

Commit message: aruco_box.xacro

File: manipulator_description/robots/timon_arm_hand_base.urdf.xacro (robot description, xacro)
@@ -4,4 +4,5 @@
   </link>
   <xacro:include filename="$(find manipulator_description)/urdf/caixa.xacro"/>
+  <xacro:include filename="$(find manipulator_description)/urdf/box_aruco.xacro"/>
   <xacro:include filename="$(find manipulator_description)/urdf/base.xacro"/>
   <xacro:include filename="$(find manipulator_description)/robots/timon_arm_hand.urdf.xacro"/>

File: manipulator_description/urdf/box_aruco.xacro (robot description, xacro)
@@ -20,8 +20,8 @@
     </inertial>
   </link>
- <!-- <joint name="base_to_box" type="fixed">
-    <parent link=""/>
-    <child link=""/>
-    <origin rpy="0 0 1.571" xyz="-0.35 0 0"/>
-  </joint>  -->
+ <joint name="base_to_box" type="fixed">
+    <parent link="base_link"/>
+    <child link="box_aruco"/>
+    <origin rpy="0 0 1.571" xyz="0.0 -0.10 0.10"/>
+  </joint>
 </robot>

Commit message: reading aruco pose in code

File: manipulator_description/robots/timon_arm_hand_base.urdf.xacro (robot description, xacro)
@@ -1,6 +1,6 @@
 <?xml version="1.0" encoding="utf-8"?>
 <robot xmlns:xacro="http://www.ros.org/wiki/xacro" name="timon_base">
-  <!-- <link name ="ground">
-  </link> -->
+  <link name = "ground">
+  </link>
   <!-- <xacro:include filename="$(find manipulator_description)/urdf/caixa.xacro"/>
   <xacro:include filename="$(find manipulator_description)/urdf/box_aruco.xacro"/> -->
@@ -9,5 +9,10 @@
   <xacro:include filename="$(find manipulator_description)/robots/camera.xacro"/>
   <!-- <xacro:include filename="$(find manipulator_description)/urdf/tag.xacro"/> -->
-    <joint name ="base_to_base_link" type="fixed">
+    <joint name ="ground_to_base" type="fixed">
+        <origin rpy="0 0 0" xyz="0 0 0"/>
+        <parent link="ground"/>
+        <child link = "base_to_manipulator"/>
+    </joint>
+    <joint name ="base_to_timon" type="fixed">
         <origin rpy="0 0 -1.571" xyz="0 0 0.1"/>
         <parent link="base_to_manipulator"/>

File: manipulator_description/urdf/base.xacro (robot description, xacro)
@@ -18,5 +18,5 @@
         <origin rpy="0 0 0" xyz="0 0 0"/>
         <mass value="1000.86661792"/>
-        <inertia ixx="8.72078676e-3" ixy="-9.55785583e-9" ixz="0" iyx="-9.55785583e-9" iyy="4.66430350e-2" iyz="0" izx="0" izy="-0" izz="5.35109282e-2"/>
+        <inertia ixx="8.72078676e-1" ixy="-9.55785583e-7" ixz="0" iyx="-9.55785583e-7" iyy="4.66430350" iyz="0" izx="0" izy="-0" izz="5.35109282"/>
       </inertial>
     </link>

File: manipulator_description/urdf/tag.xacro (robot description, xacro)
@@ -3,5 +3,5 @@
     <link name="tag_aruco_4">
         <inertial>
-            <origin xyz="0 0 0" rpy="-1.571 0 0 "/>
+            <origin xyz="0 0 0" rpy="0 0 0 "/> <!-- "-1.571 0 0 " -->
             <mass value="1.0"/>
             <inertia ixx="0.0741666666"  ixy="0.0"  ixz="0.0" iyy="0.0585461666" iyz="0.0" izz="0.02604166666" />
@@ -14,5 +14,5 @@
         </collision>
         <visual>
-            <origin xyz="0.0 0.0 0.0" rpy="1.571 -1.571 0.0"/>
+            <origin xyz="0.0 0.0 0.0" rpy="0 0 0"/>   <!-- "1.571 -1.571 0.0" -->
             <geometry>
                 <mesh filename="package://manipulator_description/meshes/tag.dae"/>
@@ -28,5 +28,5 @@
         </gazebo>
     <joint name="box_to_tag" type="fixed">
-        <origin rpy="0 1.571 0" xyz="0.0 -0.103 0.1"/>
+        <origin rpy="1.571 0 0" xyz="0.0 -0.103 0.1"/> <!--"0.0 -0.103 0.1" -->
         <parent link="caixa"/>
         <child link = "tag_aruco_4"/>
