Commit message: add moveit_config_package

File: manipulator_description/robots/base.xacro (robot description, xacro)
@@ -17,6 +17,6 @@
       <inertial>
         <origin rpy="0 0 0" xyz="0 0 0"/>
-        <mass value="1000.86661792"/>
-        <inertia ixx="8.72078676e-1" ixy="-9.55785583e-7" ixz="0" iyx="-9.55785583e-7" iyy="4.66430350" iyz="0" izx="0" izy="-0" izz="5.35109282"/>
+        <mass value="10000.86661792"/>
+        <inertia ixx="8.72078676" ixy="-9.55785583e-7" ixz="0" iyx="-9.55785583e-7" iyy="4.66430350" iyz="0" izx="0" izy="-0" izz="5.35109282"/>
       </inertial>
     </link>

Commit message: Separate base from id_1

File: manipulator_description/robots/base.xacro (robot description, xacro)
@@ -6,5 +6,5 @@
         <origin rpy="0 0 0" xyz="0 0 0"/>
         <geometry>
-          <mesh filename="package://manipulator_description/meshes/basem.dae"/>
+          <mesh filename="package://manipulator_description/meshes/JeRoTIMON/base.dae"/>
         </geometry>
       </visual>
@@ -12,5 +12,5 @@
         <origin rpy="0 0 0" xyz="0 0 0"/>
         <geometry>
-          <mesh filename="package://manipulator_description/meshes/basem.stl"/>
+          <mesh filename="package://manipulator_description/meshes/JeRoTIMON/base.stl"/>
         </geometry>
       </collision>

Commit message: adding camera

File: manipulator_description/robots/base.xacro (robot description, xacro)
@@ -6,5 +6,5 @@
         <origin rpy="0 0 0" xyz="0 0 0"/>
         <geometry>
-          <mesh filename="package://manipulator_description/meshes/JeRoTIMON/base.dae"/>
+          <mesh filename="package://manipulator_description/meshes/basem.dae"/>
         </geometry>
       </visual>
@@ -12,5 +12,5 @@
         <origin rpy="0 0 0" xyz="0 0 0"/>
         <geometry>
-          <mesh filename="package://manipulator_description/meshes/JeRoTIMON/base.stl"/>
+          <mesh filename="package://manipulator_description/meshes/basem.stl"/>
         </geometry>
       </collision>

File: manipulator_description/robots/timon_arm_hand_base.urdf.xacro (robot description, xacro)
@@ -1,24 +1,23 @@
 <?xml version="1.0" encoding="utf-8"?>
-<robot xmlns:xacro="http://www.ros.org/wiki/xacro" name="timon_base">
+<robot xmlns:xacro="http://www.ros.org/wiki/xacro" name="timon">
   <link name = "world">
   </link>
-  <!-- <xacro:include filename="$(find manipulator_description)/robots/base.xacro"/> -->
+  <xacro:include filename="$(find manipulator_description)/robots/base.xacro"/>
   <xacro:include filename="$(find manipulator_description)/robots/timon_arm.urdf.xacro"/>
-  <!-- <xacro:include filename="$(find manipulator_description)/robots/camera.xacro"/>
-   -->
-    <!-- <joint name ="world_to_base" type="fixed">
-        <origin rpy="0 0 0" xyz="0.6 0 1.56"/>
+  <xacro:include filename="$(find manipulator_description)/robots/camera.xacro"/>
+    <joint name ="world_to_base" type="fixed">
+        <origin rpy="0 0 0" xyz="0.0 0 0.0"/>
         <parent link="world"/>
         <child link = "base_to_manipulator"/>
-    </joint> -->
+    </joint>
     <joint name ="base_to_timon" type="fixed">
-        <origin rpy="0 0 -1.571" xyz="0 0 0.1"/>
+        <origin rpy="0 0 0" xyz="0 0 0.0"/>
         <parent link="world"/>
         <child link = "invisible_link"/>
     </joint>
-    <!-- <joint name ="base_to_camera" type="fixed">
-        <origin rpy="-1.571 3.1415 -1.571" xyz="0.0661 0.426 0.0123"/>
-        <parent link="timon_link7"/>
+    <joint name ="base_to_camera" type="fixed">
+        <origin rpy="0 -1.5751 -1.5751" xyz="0.0 -0.07 -0.0435"/>
+        <parent link="timon_link4"/>
         <child link = "camera"/>
-    </joint> -->
+    </joint>
 </robot>

Commit message: adding base

File: manipulator_description/robots/base.xacro (robot description, xacro)
@@ -6,5 +6,5 @@
         <origin rpy="0 0 0" xyz="0 0 0"/>
         <geometry>
-          <mesh filename="package://manipulator_description/meshes/JeRoTIMON/base.dae"/>
+          <mesh filename="package://manipulator_description/meshes/basem.dae"/>
         </geometry>
       </visual>
@@ -12,11 +12,11 @@
         <origin rpy="0 0 0" xyz="0 0 0"/>
         <geometry>
-          <mesh filename="package://manipulator_description/meshes/JeRoTIMON/base.stl"/>
+          <mesh filename="package://manipulator_description/meshes/basem.stl"/>
         </geometry>
       </collision>
       <inertial>
         <origin rpy="0 0 0" xyz="0 0 0"/>
-        <mass value="1000.86661792"/>
-        <inertia ixx="8.72078676e-1" ixy="-9.55785583e-7" ixz="0" iyx="-9.55785583e-7" iyy="4.66430350" iyz="0" izx="0" izy="-0" izz="5.35109282"/>
+        <mass value="10000.86661792"/>
+        <inertia ixx="8.72078676" ixy="-9.55785583e-7" ixz="0" iyx="-9.55785583e-7" iyy="4.66430350" iyz="0" izx="0" izy="-0" izz="5.35109282"/>
       </inertial>
     </link>

File: manipulator_description/robots/timon_arm_hand_base.urdf.xacro (robot description, xacro)
@@ -3,14 +3,14 @@
   <link name = "world">
   </link>
-  <!-- <xacro:include filename="$(find manipulator_description)/robots/base.xacro"/> -->
+  <xacro:include filename="$(find manipulator_description)/robots/base.xacro"/>
   <xacro:include filename="$(find manipulator_description)/robots/timon_arm.urdf.xacro"/>
    <xacro:include filename="$(find manipulator_description)/robots/camera.xacro"/>
-    <!-- <joint name ="world_to_base" type="fixed">
-        <origin rpy="0 0 0" xyz="0.6 0 1.56"/>
+    <joint name ="world_to_base" type="fixed">
+        <origin rpy="0 0 0" xyz="0.0 0 -0.01"/>
         <parent link="world"/>
         <child link = "base_to_manipulator"/>
-    </joint> -->
+    </joint>
     <joint name ="base_to_timon" type="fixed">
-        <origin rpy="0 0 -1.571" xyz="0 0 0.1"/>
+        <origin rpy="0 0 3.1415" xyz="0 0 0"/>
         <parent link="world"/>
         <child link = "invisible_link"/>
