Commit message: Delete lente.xacro

File: manipulator_description/robots/camera.xacro (robot description, xacro)
@@ -16,6 +16,6 @@
       <inertial>
         <origin rpy="0 0 0" xyz="0 0 0"/>
-        <mass value="0.11174388"/>
-        <inertia ixx="3.99530361e-5" ixy="9.06442969e-7" ixz="-2.47470599e-8" iyx="9.06442969e-7" iyy="2.06558682e-5" iyz="9.01711118e-8" izx="-2.47470599e-8" izy="9.01711118e-8" izz="4.39214904e-5"/>
+        <mass value="0.12163455"/>
+        <inertia ixx="2.11041984e-5" ixy="-9.60070950e-7" ixz="-9.64986145e-8" iyx="-9.60070950e-7" iyy="4.52382361e-5" iyz="-2.48143698e-8" izx="-9.64986145e-8" izy="-2.48143698e-8" izz="4.92072530e-5"/>
       </inertial>
     </link>

Commit message: settings camera file

File: manipulator_description/robots/camera.xacro (robot description, xacro)
@@ -21,5 +21,5 @@
     </link>
     <gazebo reference="camera">
-      <sensor type="camera" name="camera_top">
+      <sensor type="camera" name="camera_timon">
         <update_rate>30.0</update_rate>
         <camera name="head">
@@ -36,5 +36,5 @@
         </camera>
         <plugin name="camera_controller" filename="libgazebo_ros_camera.so">
-            <!-- <robotNamespace>raja</robotNamespace> -->
+            <robotNamespace>timon</robotNamespace>
             <alwaysOn>true</alwaysOn>
             <updateRate>0.0</updateRate>

File: manipulator_description/robots/timon_arm_hand_base.urdf.xacro (robot description, xacro)
@@ -12,5 +12,5 @@
     </joint>
     <joint name ="base_to_camera" type="fixed">
-        <origin rpy="1.571 3.1415 -1.571" xyz="0.0661 0.426 0.0123"/>
+        <origin rpy="-1.571 3.1415 -1.571" xyz="0.0661 0.426 0.0123"/>
         <parent link="timon_link7"/>
         <child link = "camera"/>

Commit message: adding tf_tree for aruco

File: manipulator_description/robots/camera.xacro (robot description, xacro)
@@ -39,5 +39,5 @@
             <alwaysOn>true</alwaysOn>
             <updateRate>0.0</updateRate>
-            <cameraName>camera_top</cameraName>
+            <cameraName>camera</cameraName>
             <imageTopicName>image_raw</imageTopicName>
             <cameraInfoTopicName>camera_info</cameraInfoTopicName>

File: manipulator_description/robots/timon_arm_hand_base.urdf.xacro (robot description, xacro)
@@ -3,10 +3,10 @@
   <link name ="base_link">
   </link>
-  <xacro:include filename="$(find manipulator_description)/urdf/caixa.xacro"/>
-  <xacro:include filename="$(find manipulator_description)/urdf/box_aruco.xacro"/>
+  <!-- <xacro:include filename="$(find manipulator_description)/urdf/caixa.xacro"/>
+  <xacro:include filename="$(find manipulator_description)/urdf/box_aruco.xacro"/> -->
   <xacro:include filename="$(find manipulator_description)/urdf/base.xacro"/>
   <xacro:include filename="$(find manipulator_description)/robots/timon_arm_hand.urdf.xacro"/>
   <xacro:include filename="$(find manipulator_description)/robots/camera.xacro"/>
-  <xacro:include filename="$(find manipulator_description)/urdf/tag.xacro"/>
+  <!-- <xacro:include filename="$(find manipulator_description)/urdf/tag.xacro"/> -->
     <joint name ="base_to_base_link" type="fixed">
         <origin rpy="0 0 -1.571" xyz="0 0 0.1"/>

File: manipulator_description/urdf/box_aruco.xacro (robot description, xacro)
@@ -20,8 +20,8 @@
     </inertial>
   </link>
- <joint name="base_to_box" type="fixed">
-    <parent link="base_link"/>
+ <joint name="caixa_to_box" type="fixed">
+    <parent link="caixa"/>
     <child link="box_aruco"/>
-    <origin rpy="0 0 1.571" xyz="0.0 -0.10 0.10"/>
+    <origin rpy="0 0 3.1415" xyz="0.0 -0.12 0.10"/>
   </joint>
 </robot>

File: manipulator_description/urdf/caixa.xacro (robot description, xacro)
@@ -21,7 +21,7 @@
   </link>
  <joint name="base_to_caixa" type="fixed">
-    <parent link="base_link"/>
+    <parent link="map"/>
     <child link="caixa"/>
-    <origin rpy="0 0 1.571" xyz="-0.35 0 0"/>
+    <origin rpy="0 0 1.571" xyz="0 0 0"/>
   </joint>
 </robot>

File: manipulator_description/urdf/tag.xacro (robot description, xacro)
@@ -1,5 +1,5 @@
 <?xml version="1.0" encoding="utf-8"?>
 <robot xmlns:xacro="http://www.ros.org/wiki/xacro" name="tag">
-    <link name="box_tag">
+    <link name="tag_aruco_13">
         <inertial>
             <origin xyz="0 0 0" rpy="1.571 0 0 "/>
@@ -20,5 +20,5 @@
         </visual>
     </link>
-        <gazebo reference="box_tag">
+        <gazebo reference="tag_aruco_13">
             <kp>100000.0</kp>
             <kd>100000.0</kd>
@@ -27,8 +27,8 @@
             <fdir1>1 0 0</fdir1>
         </gazebo>
-    <joint name="caixa_to_tag" type="fixed">
-        <origin rpy="0 0 0" xyz="0.0 -0.10 0.10"/>
-        <parent link="caixa"/>
-        <child link = "box_tag"/>
+    <joint name="box_to_tag" type="fixed">
+        <origin rpy="0 -1.571 0" xyz="0.0 0.0 0.0"/>
+        <parent link="box_aruco"/>
+        <child link = "tag_aruco_13"/>
     </joint>
 </robot>

Commit message: changing camera axes/ adding nem moveit package

File: manipulator_description/robots/camera.xacro (robot description, xacro)
@@ -3,5 +3,5 @@
     <link name="camera">
       <visual>
-        <origin rpy="0 0 0" xyz="0 0 0"/>
+        <origin rpy="0 -1.571 0" xyz="0 0 0"/>
         <geometry>
           <mesh filename="package://manipulator_description/meshes/camera.dae"/>
@@ -9,5 +9,5 @@
       </visual>
       <collision>
-        <origin rpy="0 0 0" xyz="0 0 0"/>
+        <origin rpy="0 -1.571 0" xyz="0 0 0"/>
         <geometry>
           <mesh filename="package://manipulator_description/meshes/camera.stl"/>
@@ -15,5 +15,5 @@
       </collision>
       <inertial>
-        <origin rpy="0 0 0" xyz="0 0 0"/>
+        <origin rpy="0 -1.571 0" xyz="0 0 0"/>
         <mass value="0.12163455"/>
         <inertia ixx="2.11041984e-5" ixy="-9.60070950e-7" ixz="-9.64986145e-8" iyx="-9.60070950e-7" iyy="4.52382361e-5" iyz="-2.48143698e-8" izx="-9.64986145e-8" izy="-2.48143698e-8" izz="4.92072530e-5"/>
@@ -26,6 +26,6 @@
             <horizontal_fov>1.3962634</horizontal_fov>
             <image>
-                <width>1366</width>
-                <height>768</height>
+                <width>2592</width>
+                <height>2048</height>
                 <format>R8G8B8</format>
             </image>

File: manipulator_description/robots/timon_arm.urdf.xacro (robot description, xacro)
@@ -1,4 +1,9 @@
 <?xml version='1.0' encoding='utf-8'?>
 <robot xmlns:xacro="http://www.ros.org/wiki/xacro" name="timon">
+  <gazebo>
+      <plugin name="gazebo_ros_control" filename="libgazebo_ros_control.so">
+          <robotNamespace>timon</robotNamespace>
+      </plugin>
+  </gazebo>
   <xacro:include filename="$(find manipulator_description)/robots/timon_arm.xacro" />
   <xacro:timon_arm />

File: manipulator_description/robots/timon_arm.xacro (robot description, xacro)
@@ -265,45 +265,5 @@
       <axis xyz="0 0 1" rpy="0 0 0"/>
     </joint>
-    <transmission name="trans_timon_joint1">
-        <type>transmission_interface/SimpleTransmission</type>
-        <joint name="timon_joint1">
-            <hardwareInterface>hardware_interface/PositionJointInterface</hardwareInterface>
-        </joint>
-        <actuator name="timon_joint1_motor">
-            <hardwareInterface>hardware_interface/PositionJointInterface</hardwareInterface>
-            <mechanicalReduction>1</mechanicalReduction>
-        </actuator>
-    </transmission>
-    <transmission name="trans_timon_joint4">
-        <type>transmission_interface/SimpleTransmission</type>
-        <joint name="timon_joint4">
-            <hardwareInterface>hardware_interface/PositionJointInterface</hardwareInterface>
-        </joint>
-        <actuator name="timon_joint4_motor">
-            <hardwareInterface>hardware_interface/PositionJointInterface</hardwareInterface>
-            <mechanicalReduction>1</mechanicalReduction>
-        </actuator>
-    </transmission>
-    <transmission name="trans_timon_joint7">
-        <type>transmission_interface/SimpleTransmission</type>
-        <joint name="timon_joint7">
-            <hardwareInterface>hardware_interface/PositionJointInterface</hardwareInterface>
-        </joint>
-        <actuator name="timon_joint7_motor">
-            <hardwareInterface>hardware_interface/PositionJointInterface</hardwareInterface>
-            <mechanicalReduction>1</mechanicalReduction>
-        </actuator>
-    </transmission>
-    <transmission name="trans_timon_joint9">
-        <type>transmission_interface/SimpleTransmission</type>
-        <joint name="timon_joint9">
-            <hardwareInterface>hardware_interface/PositionJointInterface</hardwareInterface>
-        </joint>
-        <actuator name="timon_joint9_motor">
-            <hardwareInterface>hardware_interface/PositionJointInterface</hardwareInterface>
-            <mechanicalReduction>1</mechanicalReduction>
-        </actuator>
-    </transmission>
-    <!-- <link name="${arm_id}_link11">
+    <link name="${arm_id}_link10">
       <visual>
         <origin xyz="0.0225 -0.007 0.0" rpy="0.0 0.0 0.0" />
@@ -324,10 +284,10 @@
       </inertial>
     </link>
-    <joint name="${arm_id}_joint11" type="fixed">
+    <joint name="${arm_id}_joint10" type="fixed">
       <origin rpy="1.5701 0.0 0.0" xyz="0.0 -0.001 0.055"/>
-      <parent link="${arm_id}_link10"/>
-      <child link="${arm_id}_link11"/>
-    </joint>
-   <link name="${arm_id}_link12">
+      <parent link="${arm_id}_link9"/>
+      <child link="${arm_id}_link10"/>
+    </joint>
+   <link name="${arm_id}_link11">
       <visual>
         <origin xyz="0.0 0.0 0.0" rpy="0.0 1.571 0.0" />
@@ -348,12 +308,62 @@
       </inertial>
     </link>
-    <joint name="${arm_id}_joint12" type="revolute">
+    <joint name="${arm_id}_joint11" type="revolute">
       <safety_controller k_position="100.0" k_velocity="40.0" soft_lower_limit="-1.90" soft_upper_limit="1.90"/>
       <origin rpy="0.0 0.0 0.0" xyz="0.0 0.0 0.0"/>
-      <parent link="${arm_id}_link11"/>
-      <child link="${arm_id}_link12"/>
+      <parent link="${arm_id}_link10"/>
+      <child link="${arm_id}_link11"/>
       <axis xyz="0 0 1"/>
       <limit effort="1000.0" lower="-1.90" upper="1.90" velocity="0.5"/>
-    </joint>  -->
+    </joint>
+    <transmission name="trans_timon_joint1">
+        <type>transmission_interface/SimpleTransmission</type>
+        <joint name="timon_joint1">
+            <hardwareInterface>hardware_interface/PositionJointInterface</hardwareInterface>
+        </joint>
+        <actuator name="timon_joint1_motor">
+            <hardwareInterface>hardware_interface/PositionJointInterface</hardwareInterface>
+            <mechanicalReduction>1</mechanicalReduction>
+        </actuator>
+    </transmission>
+    <transmission name="trans_timon_joint4">
+        <type>transmission_interface/SimpleTransmission</type>
+        <joint name="timon_joint4">
+            <hardwareInterface>hardware_interface/PositionJointInterface</hardwareInterface>
+        </joint>
+        <actuator name="timon_joint4_motor">
+            <hardwareInterface>hardware_interface/PositionJointInterface</hardwareInterface>
+            <mechanicalReduction>1</mechanicalReduction>
+        </actuator>
+    </transmission>
+    <transmission name="trans_timon_joint7">
+        <type>transmission_interface/SimpleTransmission</type>
+        <joint name="timon_joint7">
+            <hardwareInterface>hardware_interface/PositionJointInterface</hardwareInterface>
+        </joint>
+        <actuator name="timon_joint7_motor">
+            <hardwareInterface>hardware_interface/PositionJointInterface</hardwareInterface>
+            <mechanicalReduction>1</mechanicalReduction>
+        </actuator>
+    </transmission>
+    <transmission name="trans_timon_joint9">
+        <type>transmission_interface/SimpleTransmission</type>
+        <joint name="timon_joint9">
+            <hardwareInterface>hardware_interface/PositionJointInterface</hardwareInterface>
+        </joint>
+        <actuator name="timon_joint9_motor">
+            <hardwareInterface>hardware_interface/PositionJointInterface</hardwareInterface>
+            <mechanicalReduction>1</mechanicalReduction>
+        </actuator>
+    </transmission>
+    <transmission name="trans_timon_joint11">
+        <type>transmission_interface/SimpleTransmission</type>
+        <joint name="timon_joint11">
+            <hardwareInterface>hardware_interface/PositionJointInterface</hardwareInterface>
+        </joint>
+        <actuator name="timon_joint11_motor">
+            <hardwareInterface>hardware_interface/PositionJointInterface</hardwareInterface>
+            <mechanicalReduction>1</mechanicalReduction>
+        </actuator>
+    </transmission>
   </xacro:macro>
 </robot>

File: manipulator_description/robots/timon_arm_hand_base.urdf.xacro (robot description, xacro)
@@ -6,5 +6,5 @@
   <xacro:include filename="$(find manipulator_description)/urdf/box_aruco.xacro"/> -->
   <xacro:include filename="$(find manipulator_description)/urdf/base.xacro"/>
-  <xacro:include filename="$(find manipulator_description)/robots/timon_arm_hand.urdf.xacro"/>
+  <xacro:include filename="$(find manipulator_description)/robots/timon_arm.urdf.xacro"/>
   <xacro:include filename="$(find manipulator_description)/robots/camera.xacro"/>
   <!-- <xacro:include filename="$(find manipulator_description)/urdf/tag.xacro"/> -->
@@ -15,5 +15,5 @@
     </joint>
     <joint name ="base_to_camera" type="fixed">
-        <origin rpy="-1.571 3.1415 -1.571" xyz="0.0661 0.426 0.0123"/>
+        <origin rpy="-1.571 3.1415 0" xyz="0.0661 0.426 0.0123"/>
         <parent link="timon_link7"/>
         <child link = "camera"/>

Commit message: fixing links

File: manipulator_description/robots/camera.xacro (robot description, xacro)
@@ -3,5 +3,5 @@
     <link name="camera">
       <visual>
-        <origin rpy="0 -1.571 0" xyz="0 0 0"/>
+        <origin rpy="0 0 0" xyz="0 0 0"/>
         <geometry>
           <mesh filename="package://manipulator_description/meshes/camera.dae"/>
@@ -9,5 +9,5 @@
       </visual>
       <collision>
-        <origin rpy="0 -1.571 0" xyz="0 0 0"/>
+        <origin rpy="0 0 0" xyz="0 0 0"/>
         <geometry>
           <mesh filename="package://manipulator_description/meshes/camera.stl"/>
@@ -15,5 +15,5 @@
       </collision>
       <inertial>
-        <origin rpy="0 -1.571 0" xyz="0 0 0"/>
+        <origin rpy="0 0 0" xyz="0 0 0"/>
         <mass value="0.12163455"/>
         <inertia ixx="2.11041984e-5" ixy="-9.60070950e-7" ixz="-9.64986145e-8" iyx="-9.60070950e-7" iyy="4.52382361e-5" iyz="-2.48143698e-8" izx="-9.64986145e-8" izy="-2.48143698e-8" izz="4.92072530e-5"/>

File: manipulator_description/robots/timon_arm_hand_base.urdf.xacro (robot description, xacro)
@@ -1,6 +1,6 @@
 <?xml version="1.0" encoding="utf-8"?>
 <robot xmlns:xacro="http://www.ros.org/wiki/xacro" name="timon_base">
-  <link name ="base_link">
-  </link>
+  <!-- <link name ="ground">
+  </link> -->
   <!-- <xacro:include filename="$(find manipulator_description)/urdf/caixa.xacro"/>
   <xacro:include filename="$(find manipulator_description)/urdf/box_aruco.xacro"/> -->
@@ -15,5 +15,5 @@
     </joint>
     <joint name ="base_to_camera" type="fixed">
-        <origin rpy="-1.571 3.1415 0" xyz="0.0661 0.426 0.0123"/>
+        <origin rpy="-1.571 3.1415 -1.571" xyz="0.0661 0.426 0.0123"/>
         <parent link="timon_link7"/>
         <child link = "camera"/>

File: manipulator_description/urdf/base.xacro (robot description, xacro)
@@ -21,8 +21,9 @@
       </inertial>
     </link>
-      <joint name="base_to_world1" type="fixed">
+      <!-- <joint name="base_to_world1" type="fixed">
         <parent link="base_link"/>
         <child link="base_to_manipulator"/>
         <origin rpy="0 0 0" xyz="0.6 0 0"/>
       </joint>
+    -->
 </robot>

File: manipulator_description/urdf/box.urdf.xacro (robot description, xacro)
@@ -1,6 +1,4 @@
 <?xml version="1.0" encoding="utf-8"?>
 <robot xmlns:xacro="http://www.ros.org/wiki/xacro" name="timon">
-  <link name="map">
-  </link>
   <xacro:include filename="$(find manipulator_description)/urdf/caixa.xacro"/>
   <!-- <xacro:include filename="$(find manipulator_description)/urdf/box_aruco.xacro"/> -->

File: manipulator_description/urdf/caixa.xacro (robot description, xacro)
@@ -20,8 +20,8 @@
     </inertial>
   </link>
- <joint name="base_to_caixa" type="fixed">
+ <!-- <joint name="base_to_caixa" type="fixed">
     <parent link="map"/>
     <child link="caixa"/>
     <origin rpy="0 0 1.571" xyz="0 0 0"/>
-  </joint>
+  </joint>  -->
 </robot>

Commit message: using bir_marker to get aruco's pose

File: manipulator_description/robots/camera.xacro (robot description, xacro)
@@ -20,4 +20,11 @@
       </inertial>
     </link>
+    <link name="virtual_camera">
+    </link>
+    <joint name ="virtual_camera" type="fixed">
+        <origin rpy="0 -1.5701 0" xyz="0 0 0"/>  <!--rpy="1.5701 3.1415 1.5701"-->
+        <parent link="camera"/>
+        <child link = "virtual_camera"/>
+    </joint>
     <gazebo reference="camera">
       <sensor type="camera" name="camera_timon">

File: manipulator_description/urdf/base.xacro (robot description, xacro)
@@ -17,5 +17,5 @@
       <inertial>
         <origin rpy="0 0 0" xyz="0 0 0"/>
-        <mass value="2.86661792"/>
+        <mass value="1000.86661792"/>
         <inertia ixx="8.72078676e-3" ixy="-9.55785583e-9" ixz="0" iyx="-9.55785583e-9" iyy="4.66430350e-2" iyz="0" izx="0" izy="-0" izz="5.35109282e-2"/>
       </inertial>

File: manipulator_description/urdf/tag.xacro (robot description, xacro)
@@ -1,5 +1,5 @@
 <?xml version="1.0" encoding="utf-8"?>
 <robot xmlns:xacro="http://www.ros.org/wiki/xacro" name="tag">
-    <link name="tag_aruco_13">
+    <link name="tag_aruco_4">
         <inertial>
             <origin xyz="0 0 0" rpy="-1.571 0 0 "/>
@@ -20,5 +20,5 @@
         </visual>
     </link>
-        <gazebo reference="tag_aruco_13">
+        <gazebo reference="tag_aruco_4">
             <kp>100000.0</kp>
             <kd>100000.0</kd>
@@ -30,5 +30,5 @@
         <origin rpy="0 1.571 0" xyz="0.0 -0.103 0.1"/>
         <parent link="caixa"/>
-        <child link = "tag_aruco_13"/>
+        <child link = "tag_aruco_4"/>
     </joint>
 </robot>

Commit message: fixing camera orientation

File: manipulator_description/robots/camera.xacro (robot description, xacro)
@@ -23,5 +23,5 @@
     </link>
     <joint name ="virtual_camera" type="fixed">
-        <origin rpy="0 -1.5701 0" xyz="0 0 0"/>  <!--rpy="1.5701 3.1415 1.5701"-->
+        <origin rpy="-1.5701 0 -1.5701" xyz="0 0 0"/>  <!--rpy="1.5701 3.1415 1.5701"-->
         <parent link="camera"/>
         <child link = "virtual_camera"/>

File: manipulator_description/robots/timon_arm_hand_base.urdf.xacro (robot description, xacro)
@@ -1,15 +1,12 @@
 <?xml version="1.0" encoding="utf-8"?>
 <robot xmlns:xacro="http://www.ros.org/wiki/xacro" name="timon_base">
-  <link name = "ground">
+  <link name = "world">
   </link>
-  <!-- <xacro:include filename="$(find manipulator_description)/urdf/caixa.xacro"/>
-  <xacro:include filename="$(find manipulator_description)/urdf/box_aruco.xacro"/> -->
-  <xacro:include filename="$(find manipulator_description)/urdf/base.xacro"/>
+  <xacro:include filename="$(find manipulator_description)/robots/base.xacro"/>
   <xacro:include filename="$(find manipulator_description)/robots/timon_arm.urdf.xacro"/>
   <xacro:include filename="$(find manipulator_description)/robots/camera.xacro"/>
-  <!-- <xacro:include filename="$(find manipulator_description)/urdf/tag.xacro"/> -->
-    <joint name ="ground_to_base" type="fixed">
-        <origin rpy="0 0 0" xyz="0 0 0"/>
-        <parent link="ground"/>
+    <joint name ="world_to_base" type="fixed">
+        <origin rpy="0 0 0" xyz="0.6 0 1.56"/>
+        <parent link="world"/>
         <child link = "base_to_manipulator"/>
     </joint>

File: manipulator_description/urdf/box.urdf.xacro (robot description, xacro)
@@ -1,6 +1,13 @@
 <?xml version="1.0" encoding="utf-8"?>
 <robot xmlns:xacro="http://www.ros.org/wiki/xacro" name="timon">
+  <link name ="box_link">
+  </link>
   <xacro:include filename="$(find manipulator_description)/urdf/caixa.xacro"/>
   <xacro:include filename="$(find manipulator_description)/urdf/tag.xacro"/>
   <xacro:include filename="$(find manipulator_description)/urdf/botao.xacro"/>
+  <joint name="base_to_box" type="fixed">
+    <origin xyz="-0.4 0.0 1.56" rpy="0.0 0.0 1.571"/>
+    <parent link="box_link"/>
+    <child link="caixa"/>
+  </joint>
 </robot>

File: manipulator_description/urdf/tag.xacro (robot description, xacro)
@@ -28,6 +28,6 @@
         </gazebo>
     <joint name="box_to_tag" type="fixed">
-        <origin rpy="1.571 0 0" xyz="0.0 -0.103 0.1"/> <!--"0.0 -0.103 0.1" -->
-        <parent link="caixa"/>
+        <origin rpy="0 0 0" xyz="0.0 -0.1 -0.013"/> <!--"0.0 -0.103 0.1" -->
+        <parent link="botao"/>
         <child link = "tag_aruco_4"/>
     </joint>
