Commit message: updating moveit package

File: manipulator_description/robots/camera.xacro (robot description, xacro)
@@ -1,7 +1,4 @@
 <?xml version="1.0" encoding="utf-8"?>
 <robot xmlns:xacro="http://www.ros.org/wiki/xacro" name="camera">
-<<<<<<< HEAD
-=======
->>>>>>> f451ba46d1161c3b1b89d31203e39e97da13cce7
     <link name="camera">
       <visual>

File: manipulator_description/robots/timon_arm.xacro (robot description, xacro)
@@ -136,5 +136,5 @@
     </link>
     <joint name="suport_cam" type="fixed">
-      <origin rpy="0 0.0 0.0" xyz="-0.00754115 -0.03075116 0.37653086"/>
+      <origin rpy="0 0.0 3.1415" xyz="-0.00754115 -0.03075116 0.37653086"/>
       <parent link="${arm_id}_link3"/>
       <child link="${arm_id}_link4"/>

File: manipulator_description/robots/timon_arm_hand_base.urdf.xacro (robot description, xacro)
@@ -5,32 +5,18 @@
   <xacro:include filename="$(find manipulator_description)/robots/base.xacro"/>
   <xacro:include filename="$(find manipulator_description)/robots/timon_arm.urdf.xacro"/>
-<<<<<<< HEAD
-  <xacro:include filename="$(find manipulator_description)/robots/camera.xacro"/>
-    <joint name ="world_to_base" type="fixed">
-        <origin rpy="0 0 0" xyz="0.0 0 0.0"/>
-=======
    <xacro:include filename="$(find manipulator_description)/robots/camera.xacro"/>
     <joint name ="world_to_base" type="fixed">
         <origin rpy="0 0 0" xyz="0.0 0 -0.01"/>
->>>>>>> f451ba46d1161c3b1b89d31203e39e97da13cce7
         <parent link="world"/>
         <child link = "base_to_manipulator"/>
     </joint>
     <joint name ="base_to_timon" type="fixed">
-<<<<<<< HEAD
-        <origin rpy="0 0 0" xyz="0 0 0.0"/>
-=======
-        <origin rpy="0 0 3.1415" xyz="0 0 0"/>
->>>>>>> f451ba46d1161c3b1b89d31203e39e97da13cce7
+        <origin rpy="0 0 0" xyz="0 0 0"/>
         <parent link="world"/>
         <child link = "invisible_link"/>
     </joint>
     <joint name ="base_to_camera" type="fixed">
-<<<<<<< HEAD
-        <origin rpy="0 -1.5751 -1.5751" xyz="0.0 -0.07 -0.0435"/>
-=======
         <origin rpy="0 -1.57 -1.57" xyz="0 0.07134918 0.02016139"/>
         <!-- <origin rpy="-1.571 3.1415 -1.571" xyz="0.0661 0.426 0.0123"/> -->
->>>>>>> f451ba46d1161c3b1b89d31203e39e97da13cce7
         <parent link="timon_link4"/>
         <child link = "camera"/>

Commit message: fix urdf

File: manipulator_description/robots/camera.xacro (robot description, xacro)
@@ -5,5 +5,5 @@
         <origin rpy="0 0 0" xyz="0 0 0"/>
         <geometry>
-          <mesh filename="package://manipulator_description/meshes/camera.dae"/>
+          <mesh filename="package://manipulator_description/meshes/cam.dae"/>
         </geometry>
       </visual>
@@ -11,5 +11,5 @@
         <origin rpy="0 0 0" xyz="0 0 0"/>
         <geometry>
-          <mesh filename="package://manipulator_description/meshes/camera.stl"/>
+          <mesh filename="package://manipulator_description/meshes/cam.stl"/>
         </geometry>
       </collision>
@@ -23,5 +23,5 @@
     </link>
     <joint name ="virtual_camera" type="fixed">
-        <origin rpy="-1.5701 0 -1.5701" xyz="0 0 0"/>  <!--rpy="1.5701 3.1415 1.5701"-->
+        <origin rpy="0 0 0" xyz="0 0 0.04363353"/>  <!--rpy="1.5701 3.1415 1.5701"-->
         <parent link="camera"/>
         <child link = "virtual_camera"/>

File: manipulator_description/robots/timon_arm.xacro (robot description, xacro)
@@ -86,8 +86,8 @@
     </link>
     <joint name="id_2" type="revolute">
-      <origin rpy="0 0 0" xyz="0 0 0.03900000"/>
+      <origin rpy="0 0 0" xyz="0.01099894 0 0.03900000"/>
       <parent link="${arm_id}_link1"/>
       <child link="${arm_id}_link2"/>
-      <axis xyz="-1 0 0" rpy="0 0 0"/>
+      <axis xyz="1 0 0" rpy="0 0 0"/>
       <limit effort="1000.0" lower="-1.5708" upper="1.5708" velocity="0.5"/> <!-- -1.5708   1.5708-->
     </joint>
@@ -106,5 +106,5 @@
       </collision>
       <inertial>
-        <origin xyz="0 0 0" rpy="0 0 0 "/>
+        <origin xyz="0 0 0" rpy="0 0 0"/>
         <mass value="1.96131158"/>
         <inertia ixx="0.0593682"  ixy="0.00019981"  ixz="0.0024082" iyy="0.06052018" iyz="-0.00320203" izz="0.00314458" />
@@ -112,11 +112,11 @@
     </link>
     <joint name="id_3" type="revolute">
-      <origin rpy="0 0.0 0.0" xyz="0 0.02683555 0.46242180"/>
+      <origin rpy="0 0.0 0.0" xyz="-0.00872107 -0.02468844 0.46468251"/>
       <parent link="${arm_id}_link2"/>
       <child link="${arm_id}_link3"/>
-      <axis xyz="-1 0 0" rpy="0 0 0"/>
+      <axis xyz="1 0 0" rpy="0 0 0"/>
       <limit effort="1000.0" lower="-0.74" upper="3.03" velocity="0.5"/>  <!-- -0.74    3.03-->
     </joint>
-    <link name="${arm_id}_link4">
+    <!-- <link name="${arm_id}_link4">
       <visual>
         <origin xyz="0 0 0" rpy="0 0 0" />
@@ -142,6 +142,6 @@
       <child link="${arm_id}_link4"/>
       <axis xyz="0 0 0" rpy="0 0 0"/>
-    </joint>
-    <link name="${arm_id}_link5">
+    </joint> -->
+    <link name="${arm_id}_link4">
       <visual>
         <origin xyz="0 0 0" rpy="0 0 0" />
@@ -164,12 +164,12 @@
     <joint name="id_4" type="revolute">
       <safety_controller k_position="100.0" k_velocity="40.0" soft_lower_limit="-1.77" soft_upper_limit="1.77"/>
-      <origin rpy="0 0 0" xyz="0 0 0.06370001"/>
+      <origin rpy="0 0 0" xyz="0.00025000 0.02278775 0.44101451"/>
       <!-- 0.00739115 -->
-      <parent link="${arm_id}_link4"/>
-      <child link="${arm_id}_link5"/>
+      <parent link="${arm_id}_link3"/>
+      <child link="${arm_id}_link4"/>
       <axis xyz="0 0 -1"/>
       <limit effort="1000.0" lower="-1.5708" upper="1.5708" velocity="0.5"/>   <!-- -1.5708     1.5708  -->
     </joint>
-    <link name="${arm_id}_link6">
+    <link name="${arm_id}_link5">
       <visual>
         <origin xyz="0.0 0.0 0.0" rpy="0 0 0" />
@@ -191,8 +191,8 @@
     </link>
     <joint name="id_5" type="revolute">
-      <origin rpy="0 0 0" xyz="0 -0.00607092 0.027"/>
-      <parent link="${arm_id}_link5"/>
-      <child link="${arm_id}_link6"/>
-      <axis xyz="0 1 0" rpy="0 0 0"/>
+      <origin rpy="0 0 1.5751" xyz="0 0 0.02699559"/>
+      <parent link="${arm_id}_link4"/>
+      <child link="${arm_id}_link5"/>
+      <axis xyz="0 -1 0" rpy="0 0 0"/>
       <limit effort="1000.0" lower="-1.5708" upper="1.5708" velocity="0.5"/> <!-- -1.5708     1.5708  -->
     </joint>

File: manipulator_description/robots/timon_arm_hand_base.urdf.xacro (robot description, xacro)
@@ -17,7 +17,7 @@
     </joint>
     <joint name ="base_to_camera" type="fixed">
-        <origin rpy="0 -1.57 -1.57" xyz="0 0.07134918 0.02016139"/>
+        <origin rpy="0 0 0" xyz="0.00015000 0.10012477 0.35338054"/>
         <!-- <origin rpy="-1.571 3.1415 -1.571" xyz="0.0661 0.426 0.0123"/> -->
-        <parent link="timon_link4"/>
+        <parent link="timon_link3"/>
         <child link = "camera"/>
     </joint>

Commit message: push button in simulation

File: manipulator_description/robots/camera.xacro (robot description, xacro)
@@ -27,5 +27,4 @@
         <child link = "virtual_camera"/>
     </joint>
-<!--
     <gazebo reference="camera">
       <sensor type="camera" name="camera_timon">
@@ -59,4 +58,4 @@
         </plugin>
       </sensor>
-    </gazebo>        -->
+    </gazebo>
 </robot>

File: manipulator_description/urdf/botao_vertical.xacro (robot description, xacro)
@@ -32,5 +32,5 @@
     <parent link="botao"/>
     <child link="fake_botao"/>
-    <origin rpy="0.0 0.0 0.0" xyz="0.0 0.0 1.0"/>
+    <origin rpy="0.0 0.0 0.0" xyz="0.0 0.0 0.2"/>
   </joint>
 </robot>

Commit message: fix frame and virtual_camera

File: manipulator_description/robots/camera.xacro (robot description, xacro)
@@ -3,5 +3,5 @@
     <link name="camera">
       <visual>
-        <origin rpy="0 0 0" xyz="0 0 0"/>
+        <origin rpy="0 1.571 0" xyz="0 0 0"/>
         <geometry>
           <mesh filename="package://manipulator_description/meshes/cam.dae"/>
@@ -9,5 +9,5 @@
       </visual>
       <collision>
-        <origin rpy="0 0 0" xyz="0 0 0"/>
+        <origin rpy="0 1.571 0" xyz="0 0 0"/>
         <geometry>
           <mesh filename="package://manipulator_description/meshes/cam.stl"/>
@@ -15,5 +15,5 @@
       </collision>
       <inertial>
-        <origin rpy="0 0 0" xyz="0 0 0"/>
+        <origin rpy="0 1.571 0" xyz="0 0 0"/>
         <mass value="0.12163455"/>
         <inertia ixx="2.11041984e-5" ixy="-9.60070950e-7" ixz="-9.64986145e-8" iyx="-9.60070950e-7" iyy="4.52382361e-5" iyz="-2.48143698e-8" izx="-9.64986145e-8" izy="-2.48143698e-8" izz="4.92072530e-5"/>
@@ -23,5 +23,5 @@
     </link>
     <joint name ="virtual_camera" type="fixed">
-        <origin rpy="0 0 0" xyz="0 0 0.04363353"/>  <!--rpy="1.5701 3.1415 1.5701"-->
+        <origin rpy="0 1.571 0" xyz="0.04363353 0 0 "/>  <!--rpy="1.5701 3.1415 1.5701"-->
         <parent link="camera"/>
         <child link = "virtual_camera"/>

File: manipulator_description/robots/timon_arm.xacro (robot description, xacro)
@@ -191,5 +191,5 @@
     </link>
     <joint name="id_5" type="revolute">
-      <origin rpy="0 0 1.5751" xyz="0 0 0.02699559"/>
+      <origin rpy="0 0 0" xyz="0 0 0.02699559"/>
       <parent link="${arm_id}_link4"/>
       <child link="${arm_id}_link5"/>

File: manipulator_description/robots/timon_arm_hand_base.urdf.xacro (robot description, xacro)
@@ -17,5 +17,5 @@
     </joint>
     <joint name ="base_to_camera" type="fixed">
-        <origin rpy="0 0 0" xyz="0.00015000 0.10012477 0.35338054"/>
+        <origin rpy="0 -1.571 0" xyz="0.00015000 0.10012477 0.35338054"/>
         <!-- <origin rpy="-1.571 3.1415 -1.571" xyz="0.0661 0.426 0.0123"/> -->
         <parent link="timon_link3"/>

Commit message: fix tf camera

File: manipulator_description/robots/camera.xacro (robot description, xacro)
@@ -3,5 +3,5 @@
     <link name="camera">
       <visual>
-        <origin rpy="0 1.571 0" xyz="0 0 0"/>
+        <origin rpy="0 1.571 0" xyz="-0.04363353 0 0"/>
         <geometry>
           <mesh filename="package://manipulator_description/meshes/cam.dae"/>
@@ -9,5 +9,5 @@
       </visual>
       <collision>
-        <origin rpy="0 1.571 0" xyz="0 0 0"/>
+        <origin rpy="0 1.571 0" xyz="-0.04363353 0 0"/>
         <geometry>
           <mesh filename="package://manipulator_description/meshes/cam.stl"/>
@@ -15,5 +15,5 @@
       </collision>
       <inertial>
-        <origin rpy="0 1.571 0" xyz="0 0 0"/>
+        <origin rpy="0 1.571 0" xyz="-0.04363353 0 0"/>
         <mass value="0.12163455"/>
         <inertia ixx="2.11041984e-5" ixy="-9.60070950e-7" ixz="-9.64986145e-8" iyx="-9.60070950e-7" iyy="4.52382361e-5" iyz="-2.48143698e-8" izx="-9.64986145e-8" izy="-2.48143698e-8" izz="4.92072530e-5"/>

File: manipulator_description/robots/timon_arm.xacro (robot description, xacro)
@@ -194,5 +194,5 @@
       <parent link="${arm_id}_link4"/>
       <child link="${arm_id}_link5"/>
-      <axis xyz="0 -1 0" rpy="0 0 0"/>
+      <axis xyz="0 1 0" rpy="0 0 0"/>
       <limit effort="1000.0" lower="-1.5708" upper="1.5708" velocity="0.5"/> <!-- -1.5708     1.5708  -->
     </joint>

File: manipulator_description/robots/timon_arm_hand_base.urdf.xacro (robot description, xacro)
@@ -17,5 +17,5 @@
     </joint>
     <joint name ="base_to_camera" type="fixed">
-        <origin rpy="0 -1.571 0" xyz="0.00015000 0.10012477 0.35338054"/>
+        <origin rpy="0 -1.571 0" xyz="0.00015000 0.10012477 0.39638054"/>
         <!-- <origin rpy="-1.571 3.1415 -1.571" xyz="0.0661 0.426 0.0123"/> -->
         <parent link="timon_link3"/>

Commit message: fix tf camera

File: manipulator_description/robots/camera.xacro (robot description, xacro)
@@ -3,5 +3,5 @@
     <link name="camera">
       <visual>
-        <origin rpy="0 1.571 0" xyz="-0.04363353 0 0"/>
+        <origin rpy="1.5701 0 1.5701" xyz="-0.04363353 0 0"/>
         <geometry>
           <mesh filename="package://manipulator_description/meshes/cam.dae"/>
@@ -9,5 +9,5 @@
       </visual>
       <collision>
-        <origin rpy="0 1.571 0" xyz="-0.04363353 0 0"/>
+        <origin rpy="1.5701 0 1.5701" xyz="-0.04363353 0 0"/>
         <geometry>
           <mesh filename="package://manipulator_description/meshes/cam.stl"/>
@@ -15,5 +15,5 @@
       </collision>
       <inertial>
-        <origin rpy="0 1.571 0" xyz="-0.04363353 0 0"/>
+        <origin rpy="1.5701 0 1.5701" xyz="-0.04363353 0 0"/>
         <mass value="0.12163455"/>
         <inertia ixx="2.11041984e-5" ixy="-9.60070950e-7" ixz="-9.64986145e-8" iyx="-9.60070950e-7" iyy="4.52382361e-5" iyz="-2.48143698e-8" izx="-9.64986145e-8" izy="-2.48143698e-8" izz="4.92072530e-5"/>
@@ -23,5 +23,5 @@
     </link>
     <joint name ="virtual_camera" type="fixed">
-        <origin rpy="0 1.571 0" xyz="0.04363353 0 0 "/>  <!--rpy="1.5701 3.1415 1.5701"-->
+        <origin rpy="-1.5701 0 -1.5701" xyz="0 0 0 "/>  <!--rpy="1.5701 3.1415 1.5701"-->
         <parent link="camera"/>
         <child link = "virtual_camera"/>

File: manipulator_description/robots/timon_arm_hand_base.urdf.xacro (robot description, xacro)
@@ -17,5 +17,5 @@
     </joint>
     <joint name ="base_to_camera" type="fixed">
-        <origin rpy="0 -1.571 0" xyz="0.00015000 0.10012477 0.39638054"/>
+        <origin rpy="-1.5701 -1.5701 0" xyz="0.00015000 0.10012477 0.39638054"/>
         <!-- <origin rpy="-1.571 3.1415 -1.571" xyz="0.0661 0.426 0.0123"/> -->
         <parent link="timon_link3"/>

Commit message: updating to real push button

File: manipulator_description/robots/camera.xacro (robot description, xacro)
@@ -27,5 +27,5 @@
         <child link = "virtual_camera"/>
     </joint>
-    <gazebo reference="camera">
+    <!-- <gazebo reference="camera">
       <sensor type="camera" name="camera_timon">
         <update_rate>30.0</update_rate>
@@ -58,4 +58,4 @@
         </plugin>
       </sensor>
-    </gazebo>
+    </gazebo>        -->
 </robot>

File: manipulator_description/robots/timon_arm.xacro (robot description, xacro)
@@ -163,5 +163,5 @@
     </link>
     <joint name="id_4" type="revolute">
-      <safety_controller k_position="100.0" k_velocity="40.0" soft_lower_limit="-1.77" soft_upper_limit="1.77"/>
+      <safety_controller k_position="100.0" k_velocity="40.0" soft_lower_limit="-2.974" soft_upper_limit="2.974"/>
       <origin rpy="0 0 0" xyz="0.00025000 0.02278775 0.44101451"/>
       <!-- 0.00739115 -->
@@ -169,5 +169,5 @@
       <child link="${arm_id}_link4"/>
       <axis xyz="0 0 -1"/>
-      <limit effort="1000.0" lower="-1.5708" upper="1.5708" velocity="0.5"/>   <!-- -1.5708     1.5708  -->
+      <limit effort="1000.0" lower="-2.974" upper="2.974" velocity="0.5"/>   <!-- -1.5708     1.5708  -->
     </joint>
     <link name="${arm_id}_link5">

File: manipulator_description/urdf/tag.xacro (robot description, xacro)
@@ -28,5 +28,5 @@
         </gazebo>
     <joint name="box_to_tag" type="fixed">
-        <origin rpy="0 0 0" xyz="0.0 -0.06 0"/> <!--caixa na vertical: rpy="0 0 0" -->  <!-- horizontal: rpy="0 0 3.1415" -->
+        <origin rpy="0 0 0" xyz="0.0 -0.08 0"/> <!--caixa na vertical: rpy="0 0 0" -->  <!-- horizontal: rpy="0 0 3.1415" -->
         <parent link="botao"/>
         <child link = "tag_aruco_4"/>

Commit message: adding code to simulation push button

File: manipulator_description/robots/camera.xacro (robot description, xacro)
@@ -27,5 +27,5 @@
         <child link = "virtual_camera"/>
     </joint>
-    <!-- <gazebo reference="camera">
+    <gazebo reference="camera">
       <sensor type="camera" name="camera_timon">
         <update_rate>30.0</update_rate>
@@ -58,4 +58,4 @@
         </plugin>
       </sensor>
-    </gazebo>        -->
+    </gazebo>
 </robot>

File: manipulator_description/robots/timon_arm_hand_base.urdf.xacro (robot description, xacro)
@@ -3,12 +3,12 @@
   <link name = "world">
   </link>
-  <!-- <xacro:include filename="$(find manipulator_description)/robots/base.xacro"/> -->
+  <xacro:include filename="$(find manipulator_description)/robots/base.xacro"/>
   <xacro:include filename="$(find manipulator_description)/robots/timon_arm.urdf.xacro"/>
    <xacro:include filename="$(find manipulator_description)/robots/camera.xacro"/>
-    <!-- <joint name ="world_to_base" type="fixed">
+    <joint name ="world_to_base" type="fixed">
         <origin rpy="0 0 0" xyz="0.0 0 -0.01"/>
         <parent link="world"/>
         <child link = "base_to_manipulator"/>
-    </joint> -->
+    </joint>
     <joint name ="base_to_timon" type="fixed">
         <origin rpy="0 0 0" xyz="0 0 0"/>
