Commit message: creating xacro for endeffector

File: manipulator_description/robots/timon_arm.xacro (robot description, xacro)
@@ -1,5 +1,5 @@
 <?xml version='1.0' encoding='utf-8'?>
 <robot xmlns:xacro="http://www.ros.org/wiki/xacro" name="timon">
-    <xacro:macro name="timon_arm" params="arm_id:='timon' description_pkg:='manipulator_description' connected_to:='' xyz:='0 0 0' rpy:='0 0 0'">
+  <xacro:macro name="timon_arm" params="arm_id:='timon' description_pkg:='manipulator_description' connected_to:='' xyz:='0 0 0' rpy:='0 0 0'">
     <link name="${arm_id}_link0">
       <visual>
@@ -216,103 +216,4 @@
       <limit effort="1000.0" lower="-0.95" upper="2.36" velocity="0.5"/>
     </joint>
-    <link name="${arm_id}_link9">
-      <visual>
-        <origin xyz="0.0 0.0 0.0" rpy="0.0 0.0 0.0" />
-        <geometry>
-          <mesh filename="package://${description_pkg}/meshes/visual/link9.dae"/>
-        </geometry>
-      </visual>
-      <collision>
-        <origin xyz="0.0 0.0 0.0" rpy="0.0 0.0 0.0" />
-        <geometry>
-          <mesh filename="package://${description_pkg}/meshes/collision/link9.stl"/>
-        </geometry>
-      </collision>
-      <inertial>
-        <origin xyz="0.0 0.0 0.0" rpy="0.0 0.0 0.0"/>
-        <mass value="0.16499216"/>
-        <inertia ixx="7.88952550e-5"  ixy="-3.13065901e-9"  ixz="4.40693303e-9" iyy="4.39861799e-5" iyz="-2.02737764e-6" izz="6.23603662e-5" />
-      </inertial>
-    </link>
-    <joint name="${arm_id}_joint9" type="fixed">
-      <origin rpy="0.0 -1.571 -1.571" xyz="0 0.41 0.013"/>
-      <parent link="${arm_id}_link8"/>
-      <child link="${arm_id}_link9"/>
-    </joint>
-    <link name="${arm_id}_link10">
-      <visual>
-        <origin xyz="0.0 0.0 0.0" rpy="1.571 0.0 0.0" />
-        <geometry>
-          <mesh filename="package://${description_pkg}/meshes/visual/link10.dae"/>
-        </geometry>
-      </visual>
-      <collision>
-        <origin xyz="0.0 0.0 0.0" rpy="1.571 0.0 0.0" />
-        <geometry>
-          <mesh filename="package://${description_pkg}/meshes/collision/link10.stl"/>
-        </geometry>
-      </collision>
-      <inertial>
-        <origin xyz="0.0 0.0 0.0" rpy="1.571 0.0 0.0"/>
-        <mass value="0.007"/>
-        <inertia ixx="1.48840827e-6"  ixy="2.49592487e-8"  ixz="5.30644674e-12" iyy="2.08108627e-6" iyz="2.38181240e-14" izz="6.88193128e-7" />
-      </inertial>
-    </link>
-    <joint name="${arm_id}_joint10" type="continuous">
-      <origin rpy="0 0 1.571" xyz="0 0 0.025"/>
-      <parent link="${arm_id}_link9"/>
-      <child link="${arm_id}_link10"/>
-      <axis xyz="0 0 1" rpy="0 0 0"/>
-    </joint>
-    <link name="${arm_id}_link11">
-      <visual>
-        <origin xyz="0.0225 -0.007 0.0" rpy="0.0 0.0 0.0" />
-        <geometry>
-          <mesh filename="package://${description_pkg}/meshes/visual/link11.dae"/>
-        </geometry>
-      </visual>
-      <collision>
-        <origin xyz="0.0225 -0.007 0.0" rpy="0.0 0.0 0.0" />
-        <geometry>
-          <mesh filename="package://${description_pkg}/meshes/collision/link11.stl"/>
-        </geometry>
-      </collision>
-      <inertial>
-        <origin xyz="0.0225 -0.007 0.0" rpy="0.0 0.0 0.0"/>
-        <mass value="0.16499216"/>
-        <inertia ixx="7.88952550e-5"  ixy="-3.13065901e-9"  ixz="4.40693303e-9" iyy="4.39861799e-5" iyz="-2.02737764e-6" izz="6.23603662e-5" />
-      </inertial>
-    </link>
-    <joint name="${arm_id}_joint11" type="fixed">
-      <origin rpy="1.5701 0.0 0.0" xyz="0.0 -0.001 0.055"/>
-      <parent link="${arm_id}_link10"/>
-      <child link="${arm_id}_link11"/>
-    </joint>
-    <link name="${arm_id}_link12">
-      <visual>
-        <origin xyz="0.0 0.0 0.0" rpy="0.0 1.571 0.0" />
-        <geometry>
-          <mesh filename="package://${description_pkg}/meshes/visual/link12.dae"/>
-        </geometry>
-      </visual>
-      <collision>
-        <origin xyz="0.0 0.0 0.0" rpy="0.0 1.571 0.0" />
-        <geometry>
-          <mesh filename="package://${description_pkg}/meshes/collision/link12.stl"/>
-        </geometry>
-      </collision>
-      <inertial>
-        <origin xyz="0.0 0.0 0.0" rpy="0.0 1.571 0.0"/>
-        <mass value="0.01873963"/>
-        <inertia ixx="4.49588271e-6"  ixy="0.00000000e+0"  ixz="0.00000000e+0" iyy="1.08113872e-5" iyz="0.00000000e+0" izz="1.12040418e-5" />
-      </inertial>
-    </link>
-    <joint name="${arm_id}_joint12" type="revolute">
-      <origin rpy="0.0 0.0 0.0" xyz="0.0 0.0 0.0"/>
-      <parent link="${arm_id}_link11"/>
-      <child link="${arm_id}_link12"/>
-      <axis xyz="0 0 1"/>
-      <limit effort="1000.0" lower="-1.90" upper="1.90" velocity="0.5"/>
-    </joint>
   </xacro:macro>
 </robot>

File: manipulator_description/robots/timon_arm_hand.urdf.xacro (robot description, xacro)
@@ -1,7 +1,7 @@
 <?xml version="1.0" encoding="utf-8"?>
 <robot xmlns:xacro="http://www.ros.org/wiki/xacro" name="timon">
-  <xacro:include filename="$(find franka_description)/robots/timon_arm.xacro"/>
-  <xacro:include filename="$(find franka_description)/robots/hand.xacro"/>
+  <xacro:include filename="$(find manipulator_description)/robots/timon_arm.xacro"/>
+  <xacro:include filename="$(find manipulator_description)/robots/hand.xacro"/>
   <xacro:timon_arm />
-  <xacro:hand ns="timon" rpy="0 0 ${-pi/4}" connected_to="timon_link8"/>
+  <xacro:hand ns="timon" rpy="0 -1.571 -1.571" xyz="0 0.41 0.013" connected_to="timon_link8"/>
 </robot>

Commit message: fix xacro

File: manipulator_description/robots/timon_arm.xacro (robot description, xacro)
@@ -2,5 +2,5 @@
 <robot xmlns:xacro="http://www.ros.org/wiki/xacro" name="timon">
   <xacro:macro name="timon_arm" params="arm_id:='timon' description_pkg:='manipulator_description' connected_to:='' xyz:='0 0 0' rpy:='0 0 0'">
-    <link name="${arm_id}_link0">
+    <!-- <link name="${arm_id}_link0">
       <visual>
         <geometry>
@@ -18,5 +18,5 @@
         <inertia ixx="7.77716e+3"  ixy="0.00000e+0"  ixz="0.00000e+0" iyy="4.619e+4" iyz="0.00000e+0" izz="5.29561e+4" />
       </inertial>
-    </link>
+    </link> -->
     <link name="${arm_id}_link1">
       <visual>
@@ -38,9 +38,9 @@
       </inertial>
     </link>
-    <joint name="${arm_id}_joint1" type="fixed">
+    <!-- <joint name="${arm_id}_joint1" type="fixed">
       <origin rpy="0 0 1.571" xyz="0 0 0.09"/>
       <parent link="${arm_id}_link0"/>
       <child link="${arm_id}_link1"/>
-    </joint>
+    </joint> -->
     <link name="${arm_id}_link2">
       <visual>

Commit message: testing new branch

File: manipulator_description/robots/timon_arm.xacro (robot description, xacro)
@@ -2,5 +2,5 @@
 <robot xmlns:xacro="http://www.ros.org/wiki/xacro" name="timon">
   <xacro:macro name="timon_arm" params="arm_id:='timon' description_pkg:='manipulator_description' connected_to:='' xyz:='0 0 0' rpy:='0 0 0'">
-    <!-- <link name="${arm_id}_link0">
+    <!--<link name="${arm_id}_link0">
       <visual>
         <geometry>

Commit message: trying new xacro

File: manipulator_description/robots/timon_arm.xacro (robot description, xacro)
@@ -268,4 +268,55 @@
       <axis xyz="0 0 1" rpy="0 0 0"/>
     </joint>
+    <link name="${arm_id}_link11">
+      <visual>
+        <origin xyz="0.0225 -0.007 0.0" rpy="0.0 0.0 0.0" />
+        <geometry>
+          <mesh filename="package://manipulator_description/meshes/visual/link11.dae"/>
+        </geometry>
+      </visual>
+      <collision>
+        <origin xyz="0.0225 -0.007 0.0" rpy="0.0 0.0 0.0" />
+        <geometry>
+          <mesh filename="package://manipulator_description/meshes/visual/link11.dae"/>
+        </geometry>
+      </collision>
+      <inertial>
+        <origin xyz="0.0225 -0.007 0.0" rpy="0.0 0.0 0.0"/>
+        <mass value="0.16499216"/>
+        <inertia ixx="7.88952550e-5"  ixy="-3.13065901e-9"  ixz="4.40693303e-9" iyy="4.39861799e-5" iyz="-2.02737764e-6" izz="6.23603662e-5" />
+      </inertial>
+    </link>
+    <joint name="${arm_id}_joint11" type="fixed">
+      <origin rpy="1.5701 0.0 0.0" xyz="0.0 -0.001 0.055"/>
+      <parent link="${arm_id}_link10"/>
+      <child link="${arm_id}_link11"/>
+    </joint>
+   <link name="${arm_id}_link12">
+      <visual>
+        <origin xyz="0.0 0.0 0.0" rpy="0.0 1.571 0.0" />
+        <geometry>
+          <mesh filename="package://manipulator_description/meshes/visual/link12.dae"/>
+        </geometry>
+      </visual>
+      <collision>
+        <origin xyz="0.0 0.0 0.0" rpy="0.0 1.571 0.0" />
+        <geometry>
+          <mesh filename="package://manipulator_description/meshes/visual/link12.dae"/>
+        </geometry>
+      </collision>
+      <inertial>
+        <origin xyz="0.0 0.0 0.0" rpy="0.0 1.571 0.0"/>
+        <mass value="0.01873963"/>
+        <inertia ixx="4.49588271e-6"  ixy="0.00000000e+0"  ixz="0.00000000e+0" iyy="1.08113872e-5" iyz="0.00000000e+0" izz="1.12040418e-5" />
+      </inertial>
+    </link>
+    <joint name="${arm_id}_joint12" type="revolute">
+      <safety_controller k_position="100.0" k_velocity="40.0" soft_lower_limit="-1.90" soft_upper_limit="1.90"/>
+      <origin rpy="0.0 0.0 0.0" xyz="0.0 0.0 0.0"/>
+      <parent link="${arm_id}_link11"/>
+      <child link="${arm_id}_link12"/>
+      <axis xyz="0 0 1"/>
+      <limit effort="1000.0" lower="-1.90" upper="1.90" velocity="0.5"/>
+    </joint>
   </xacro:macro>
 </robot>

Commit message: fixing home pose

File: manipulator_description/robots/timon_arm.xacro (robot description, xacro)
@@ -2,22 +2,7 @@
 <robot xmlns:xacro="http://www.ros.org/wiki/xacro" name="timon">
   <xacro:macro name="timon_arm" params="arm_id:='timon' description_pkg:='manipulator_description' connected_to:='' xyz:='0 0 0' rpy:='0 0 0'">
-    <!-- <link name="${arm_id}_link0">
-      <visual>
-        <geometry>
-          <mesh filename="package://${description_pkg}/meshes/visual/link0.dae"/>
-        </geometry>
-      </visual>
-      <collision>
-        <geometry>
-          <mesh filename="package://${description_pkg}/meshes/visual/link0.dae"/>
-        </geometry>
-      </collision>
-      <inertial>
-        <origin xyz="0 0 0" rpy="0 0 0 "/>
-        <mass value="2.6"/>
-        <inertia ixx="7.77716e+3"  ixy="0.00000e+0"  ixz="0.00000e+0" iyy="4.619e+4" iyz="0.00000e+0" izz="5.29561e+4" />
-      </inertial>
-    </link> -->
-    <link name="${arm_id}_link1">
+    <link name = "base_link">
+    </link>
+    <link name="${arm_id}_link0">
       <visual>
         <origin xyz="0 0 0" rpy="1.571 0 0" />
@@ -38,10 +23,10 @@
       </inertial>
     </link>
-    <!-- <joint name="${arm_id}_joint1" type="fixed">
-      <origin rpy="0 0 1.571" xyz="0 0 0.09"/>
-      <parent link="${arm_id}_link0"/>
-      <child link="${arm_id}_link1"/>
-    </joint> -->
-    <link name="${arm_id}_link2">
+      <joint name ="base_to_arm" type="fixed">
+        <origin rpy="0 0 0" xyz="0 0 0"/>
+        <parent link="base_link"/>
+        <child link = "${arm_id}_link0"/>
+      </joint>
+    <link name="${arm_id}_link1">
       <visual>
         <origin xyz="0 0 0" rpy="-3.14 0 0" />
@@ -62,12 +47,12 @@
       </inertial>
     </link>
-    <joint name="${arm_id}_joint2" type="continuous">
+    <joint name="${arm_id}_joint1" type="continuous">
       <safety_controller k_position="100.0" k_velocity="40.0"/>
       <origin rpy="3.14 0 0" xyz="0 0 0.036"/>
-      <parent link="${arm_id}_link1"/>
-      <child link="${arm_id}_link2"/>
+      <parent link="${arm_id}_link0"/>
+      <child link="${arm_id}_link1"/>
       <axis xyz="0 0 1" rpy="0 0 0"/>
     </joint>
-    <link name="${arm_id}_link3">
+    <link name="${arm_id}_link2">
       <visual>
         <origin xyz="0 0 0" rpy="1.571 0 0" />
@@ -88,10 +73,10 @@
       </inertial>
     </link>
-    <joint name="${arm_id}_joint3" type="fixed">
+    <joint name="${arm_id}_joint2" type="fixed">
       <origin rpy="-1.571 1.571 1.571" xyz="-0.04 0.0 -0.039"/>
-      <parent link="${arm_id}_link2"/>
-      <child link="${arm_id}_link3"/>
-    </joint>
-    <link name="${arm_id}_link4">
+      <parent link="${arm_id}_link1"/>
+      <child link="${arm_id}_link2"/>
+    </joint>
+    <link name="${arm_id}_link3">
       <visual>
         <origin xyz="0 0 0" rpy="1.571 0 0" />
@@ -112,10 +97,10 @@
       </inertial>
     </link>
-    <joint name="${arm_id}_joint4" type="fixed">
+    <joint name="${arm_id}_joint3" type="fixed">
       <origin rpy="1.571 0.0 0.0" xyz="0.0 0.0 -0.093"/>
-      <parent link="${arm_id}_link3"/>
-      <child link="${arm_id}_link4"/>
-    </joint>
-    <link name="${arm_id}_link5">
+      <parent link="${arm_id}_link2"/>
+      <child link="${arm_id}_link3"/>
+    </joint>
+    <link name="${arm_id}_link4">
       <visual>
         <origin xyz="-0.0292 0.2289 -0.04" rpy="0 1.571 0" />
@@ -136,13 +121,13 @@
       </inertial>
     </link>
-    <joint name="${arm_id}_joint5" type="revolute">
+    <joint name="${arm_id}_joint4" type="revolute">
       <safety_controller k_position="100.0" k_velocity="40.0" soft_lower_limit="-1.77" soft_upper_limit="1.77"/>
       <origin rpy="0 -1.571 -1.571" xyz="-0.0008 0.093 0.001"/>
-      <parent link="${arm_id}_link4"/>
-      <child link="${arm_id}_link5"/>
+      <parent link="${arm_id}_link3"/>
+      <child link="${arm_id}_link4"/>
       <axis xyz="0 0 1"/>
       <limit effort="1000.0" lower="-1.77" upper="1.77" velocity="0.5"/>
     </joint>
-    <link name="${arm_id}_link6">
+    <link name="${arm_id}_link5">
       <visual>
         <origin xyz="0.0 0.0 0.0" rpy="0 0 -0.75" />
@@ -163,10 +148,10 @@
       </inertial>
     </link>
-    <joint name="${arm_id}_joint6" type="fixed">
+    <joint name="${arm_id}_joint5" type="fixed">
       <origin rpy="0 0 0" xyz="0.03 0.451 -0.015"/>
-      <parent link="${arm_id}_link5"/>
-      <child link="${arm_id}_link6"/>
-    </joint>
-    <link name="${arm_id}_link7">
+      <parent link="${arm_id}_link4"/>
+      <child link="${arm_id}_link5"/>
+    </joint>
+    <link name="${arm_id}_link6">
       <visual>
         <origin xyz="0.0 0.0 0.0" rpy="0 0 0.75" />
@@ -187,10 +172,10 @@
       </inertial>
     </link>
-    <joint name="${arm_id}_joint7" type="fixed">
+    <joint name="${arm_id}_joint6" type="fixed">
       <origin rpy="0 3.14 0" xyz="0.0 0.0 -0.05"/>
-      <parent link="${arm_id}_link6"/>
-      <child link="${arm_id}_link7"/>
-    </joint>
-    <link name="${arm_id}_link8">
+      <parent link="${arm_id}_link5"/>
+      <child link="${arm_id}_link6"/>
+    </joint>
+    <link name="${arm_id}_link7">
       <visual>
         <origin xyz="-0.01 0.015 0.0" rpy="0.0 1.571 0.0" />
@@ -211,13 +196,13 @@
       </inertial>
     </link>
-    <joint name="${arm_id}_joint8" type="revolute">
+    <joint name="${arm_id}_joint7" type="revolute">
       <safety_controller k_position="100.0" k_velocity="40.0" soft_lower_limit="-0.95" soft_upper_limit="2.36"/>
       <origin rpy="0.0 0.0 0.0" xyz="0.0 0.001 -0.0375"/>
-      <parent link="${arm_id}_link7"/>
-      <child link="${arm_id}_link8"/>
+      <parent link="${arm_id}_link6"/>
+      <child link="${arm_id}_link7"/>
       <axis xyz="0 0 1"/>
       <limit effort="1000.0" lower="-0.95" upper="2.36" velocity="0.5"/>
     </joint>
-    <link name="${arm_id}_link9">
+    <link name="${arm_id}_link8">
       <visual>
         <origin xyz="0.0 0.0 0.0" rpy="0.0 0.0 0.0" />
@@ -238,10 +223,10 @@
       </inertial>
     </link>
-    <joint name="${arm_id}_joint9" type="fixed">
+    <joint name="${arm_id}_joint8" type="fixed">
       <origin rpy="0 -1.571 -1.571" xyz="0 0.41 0.013"/>
-      <parent link="${arm_id}_link8"/>
-      <child link="${arm_id}_link9"/>
-    </joint>
-    <link name="${arm_id}_link10">
+      <parent link="${arm_id}_link7"/>
+      <child link="${arm_id}_link8"/>
+    </joint>
+    <link name="${arm_id}_link9">
       <visual>
         <origin xyz="0.0 0.0 0.0" rpy="1.571 0.0 0.0" />
@@ -262,11 +247,11 @@
       </inertial>
     </link>
-    <joint name="${arm_id}_joint10" type="continuous">
+    <joint name="${arm_id}_joint9" type="continuous">
       <origin rpy="0 0 1.571" xyz="0 0 0.025"/>
-      <parent link="${arm_id}_link9"/>
-      <child link="${arm_id}_link10"/>
+      <parent link="${arm_id}_link8"/>
+      <child link="${arm_id}_link9"/>
       <axis xyz="0 0 1" rpy="0 0 0"/>
     </joint>
-    <link name="${arm_id}_link11">
+    <!-- <link name="${arm_id}_link11">
       <visual>
         <origin xyz="0.0225 -0.007 0.0" rpy="0.0 0.0 0.0" />
@@ -318,5 +303,5 @@
       <axis xyz="0 0 1"/>
       <limit effort="1000.0" lower="-1.90" upper="1.90" velocity="0.5"/>
-    </joint>
+    </joint>  -->
   </xacro:macro>
 </robot>

File: manipulator_description/robots/timon_arm_hand.urdf.xacro (robot description, xacro)
@@ -4,4 +4,4 @@
   <xacro:include filename="$(find manipulator_description)/robots/hand.xacro"/>
   <xacro:timon_arm />
-  <xacro:hand ns="timon" rpy="1.5701 0.0 0.0" xyz="0.0 -0.001 0.055" connected_to="timon_link10"/>
+  <xacro:hand ns="timon" rpy="1.5701 0.0 0.0" xyz="0.0 -0.001 0.055" connected_to="timon_link9"/>
 </robot>
