Commit message: manipulator at position

File: manipulator_description/robots/timon_arm.xacro (robot description, xacro)
@@ -2,22 +2,5 @@
 <robot xmlns:xacro="http://www.ros.org/wiki/xacro" name="timon">
   <xacro:macro name="timon_arm" params="arm_id:='timon' description_pkg:='manipulator_description' connected_to:='' xyz:='0 0 0' rpy:='0 0 0'">
-    <!--<link name="${arm_id}_link0">
-      <visual>
-        <geometry>
-          <mesh filename="package://${description_pkg}/meshes/visual/link0.dae"/>
-        </geometry>
-      </visual>
-      <collision>
-        <geometry>
-          <mesh filename="package://${description_pkg}/meshes/collision/link0.stl"/>
-        </geometry>
-      </collision>
-      <inertial>
-        <origin xyz="0 0 0" rpy="0 0 0 "/>
-        <mass value="2.6"/>
-        <inertia ixx="7.77716e+3"  ixy="0.00000e+0"  ixz="0.00000e+0" iyy="4.619e+4" iyz="0.00000e+0" izz="5.29561e+4" />
-      </inertial>
-    </link> -->
-    <link name="${arm_id}_link1">
+    <link name="${arm_id}_link0">
       <visual>
         <origin xyz="0 0 0" rpy="1.571 0 0" />
@@ -29,5 +12,5 @@
         <origin xyz="0 0 0" rpy="1.571 0 0" />
         <geometry>
-          <mesh filename="package://${description_pkg}/meshes/collision/link1.stl"/>
+          <mesh filename="package://${description_pkg}/meshes/visual/link1.dae"/>
         </geometry>
       </collision>
@@ -38,10 +21,10 @@
       </inertial>
     </link>
-    <!-- <joint name="${arm_id}_joint1" type="fixed">
-      <origin rpy="0 0 1.571" xyz="0 0 0.09"/>
-      <parent link="${arm_id}_link0"/>
-      <child link="${arm_id}_link1"/>
-    </joint> -->
-    <link name="${arm_id}_link2">
+     <joint name ="base_to_base_link" type="fixed">
+        <origin rpy="0 0 -1.571" xyz="0 0 0.1"/>
+        <parent link="base_to_manipulator"/>
+        <child link = "${arm_id}_link0"/>
+      </joint>
+    <link name="${arm_id}_link1">
       <visual>
         <origin xyz="0 0 0" rpy="-3.14 0 0" />
@@ -53,5 +36,5 @@
         <origin xyz="0 0 0" rpy="-3.14 0 0" />
         <geometry>
-          <mesh filename="package://${description_pkg}/meshes/collision/link2.stl"/>
+          <mesh filename="package://${description_pkg}/meshes/visual/link2.dae"/>
         </geometry>
       </collision>
@@ -62,11 +45,12 @@
       </inertial>
     </link>
-    <joint name="${arm_id}_joint2" type="continuous">
+    <joint name="${arm_id}_joint1" type="continuous">
+      <safety_controller k_position="100.0" k_velocity="40.0"/>
       <origin rpy="3.14 0 0" xyz="0 0 0.036"/>
-      <parent link="${arm_id}_link1"/>
-      <child link="${arm_id}_link2"/>
+      <parent link="${arm_id}_link0"/>
+      <child link="${arm_id}_link1"/>
       <axis xyz="0 0 1" rpy="0 0 0"/>
     </joint>
-    <link name="${arm_id}_link3">
+    <link name="${arm_id}_link2">
       <visual>
         <origin xyz="0 0 0" rpy="1.571 0 0" />
@@ -78,5 +62,5 @@
         <origin xyz="0 0 0" rpy="1.571 0 0" />
         <geometry>
-          <mesh filename="package://${description_pkg}/meshes/collision/link3.stl"/>
+          <mesh filename="package://${description_pkg}/meshes/visual/link3.dae"/>
         </geometry>
       </collision>
@@ -87,10 +71,10 @@
       </inertial>
     </link>
-    <joint name="${arm_id}_joint3" type="fixed">
+    <joint name="${arm_id}_joint2" type="fixed">
       <origin rpy="-1.571 1.571 1.571" xyz="-0.04 0.0 -0.039"/>
-      <parent link="${arm_id}_link2"/>
-      <child link="${arm_id}_link3"/>
-    </joint>
-    <link name="${arm_id}_link4">
+      <parent link="${arm_id}_link1"/>
+      <child link="${arm_id}_link2"/>
+    </joint>
+    <link name="${arm_id}_link3">
       <visual>
         <origin xyz="0 0 0" rpy="1.571 0 0" />
@@ -102,5 +86,5 @@
         <origin xyz="0 0 0" rpy="1.571 0 0" />
         <geometry>
-          <mesh filename="package://${description_pkg}/meshes/collision/link4.stl"/>
+          <mesh filename="package://${description_pkg}/meshes/visual/link4.dae"/>
         </geometry>
       </collision>
@@ -111,10 +95,10 @@
       </inertial>
     </link>
-    <joint name="${arm_id}_joint4" type="fixed">
+    <joint name="${arm_id}_joint3" type="fixed">
       <origin rpy="1.571 0.0 0.0" xyz="0.0 0.0 -0.093"/>
-      <parent link="${arm_id}_link3"/>
-      <child link="${arm_id}_link4"/>
-    </joint>
-    <link name="${arm_id}_link5">
+      <parent link="${arm_id}_link2"/>
+      <child link="${arm_id}_link3"/>
+    </joint>
+    <link name="${arm_id}_link4">
       <visual>
         <origin xyz="-0.0292 0.2289 -0.04" rpy="0 1.571 0" />
@@ -126,5 +110,5 @@
         <origin xyz="-0.0292 0.2289 -0.04" rpy="0 1.571 0" />
         <geometry>
-          <mesh filename="package://${description_pkg}/meshes/collision/link5.stl"/>
+          <mesh filename="package://${description_pkg}/meshes/visual/link5.dae"/>
         </geometry>
       </collision>
@@ -135,12 +119,13 @@
       </inertial>
     </link>
-    <joint name="${arm_id}_joint5" type="revolute">
-      <origin rpy="0 -1.571 -1.571" xyz="-0.0008 0.093 0"/>
-      <parent link="${arm_id}_link4"/>
-      <child link="${arm_id}_link5"/>
+    <joint name="${arm_id}_joint4" type="revolute">
+      <safety_controller k_position="100.0" k_velocity="40.0" soft_lower_limit="-1.77" soft_upper_limit="1.77"/>
+      <origin rpy="0 -1.571 -1.571" xyz="-0.0008 0.093 0.001"/>
+      <parent link="${arm_id}_link3"/>
+      <child link="${arm_id}_link4"/>
       <axis xyz="0 0 1"/>
       <limit effort="1000.0" lower="-1.77" upper="1.77" velocity="0.5"/>
     </joint>
-    <link name="${arm_id}_link6">
+    <link name="${arm_id}_link5">
       <visual>
         <origin xyz="0.0 0.0 0.0" rpy="0 0 -0.75" />
@@ -152,5 +137,5 @@
         <origin xyz="0.0 0.0 0.0" rpy="0 0 -0.75" />
         <geometry>
-          <mesh filename="package://${description_pkg}/meshes/collision/link6.stl"/>
+          <mesh filename="package://${description_pkg}/meshes/visual/link6.dae"/>
         </geometry>
       </collision>
@@ -161,10 +146,10 @@
       </inertial>
     </link>
-    <joint name="${arm_id}_joint6" type="fixed">
+    <joint name="${arm_id}_joint5" type="fixed">
       <origin rpy="0 0 0" xyz="0.03 0.451 -0.015"/>
-      <parent link="${arm_id}_link5"/>
-      <child link="${arm_id}_link6"/>
-    </joint>
-    <link name="${arm_id}_link7">
+      <parent link="${arm_id}_link4"/>
+      <child link="${arm_id}_link5"/>
+    </joint>
+    <link name="${arm_id}_link6">
       <visual>
         <origin xyz="0.0 0.0 0.0" rpy="0 0 0.75" />
@@ -176,5 +161,5 @@
         <origin xyz="0.0 0.0 0.0" rpy="0 0 0.75" />
         <geometry>
-          <mesh filename="package://${description_pkg}/meshes/collision/link7.stl"/>
+          <mesh filename="package://${description_pkg}/meshes/visual/link7.dae"/>
         </geometry>
       </collision>
@@ -185,10 +170,10 @@
       </inertial>
     </link>
-    <joint name="${arm_id}_joint7" type="fixed">
+    <joint name="${arm_id}_joint6" type="fixed">
       <origin rpy="0 3.14 0" xyz="0.0 0.0 -0.05"/>
-      <parent link="${arm_id}_link6"/>
-      <child link="${arm_id}_link7"/>
-    </joint>
-    <link name="${arm_id}_link8">
+      <parent link="${arm_id}_link5"/>
+      <child link="${arm_id}_link6"/>
+    </joint>
+    <link name="${arm_id}_link7">
       <visual>
         <origin xyz="-0.01 0.015 0.0" rpy="0.0 1.571 0.0" />
@@ -200,5 +185,5 @@
         <origin xyz="-0.01 0.015 0.0" rpy="0.0 1.571 0.0" />
         <geometry>
-          <mesh filename="package://${description_pkg}/meshes/collision/link8.stl"/>
+          <mesh filename="package://${description_pkg}/meshes/visual/link8.dae"/>
         </geometry>
       </collision>
@@ -209,11 +194,152 @@
       </inertial>
     </link>
-    <joint name="${arm_id}_joint8" type="revolute">
+    <joint name="${arm_id}_joint7" type="revolute">
+      <safety_controller k_position="100.0" k_velocity="40.0" soft_lower_limit="-0.95" soft_upper_limit="2.36"/>
       <origin rpy="0.0 0.0 0.0" xyz="0.0 0.001 -0.0375"/>
+      <parent link="${arm_id}_link6"/>
+      <child link="${arm_id}_link7"/>
+      <axis xyz="0 0 1"/>
+      <limit effort="1000.0" lower="-0.95" upper="2.36" velocity="0.5"/>
+    </joint>
+    <link name="${arm_id}_link8">
+      <visual>
+        <origin xyz="0.0 0.0 0.0" rpy="0.0 0.0 0.0" />
+        <geometry>
+          <mesh filename="package://manipulator_description/meshes/visual/link9.dae"/>
+        </geometry>
+      </visual>
+      <collision>
+        <origin xyz="0.0 0.0 0.0" rpy="0.0 0.0 0.0" />
+        <geometry>
+          <mesh filename="package://manipulator_description/meshes/visual/link9.dae"/>
+        </geometry>
+      </collision>
+      <inertial>
+        <origin xyz="0.0 0.0 0.0" rpy="0.0 0.0 0.0"/>
+        <mass value="0.16499216"/>
+        <inertia ixx="7.88952550e-5"  ixy="-3.13065901e-9"  ixz="4.40693303e-9" iyy="4.39861799e-5" iyz="-2.02737764e-6" izz="6.23603662e-5" />
+      </inertial>
+    </link>
+    <joint name="${arm_id}_joint8" type="fixed">
+      <origin rpy="0 -1.571 -1.571" xyz="0 0.41 0.013"/>
       <parent link="${arm_id}_link7"/>
       <child link="${arm_id}_link8"/>
+    </joint>
+    <link name="${arm_id}_link9">
+      <visual>
+        <origin xyz="0.0 0.0 0.0" rpy="1.571 0.0 0.0" />
+        <geometry>
+          <mesh filename="package://manipulator_description/meshes/visual/link10.dae"/>
+        </geometry>
+      </visual>
+      <collision>
+        <origin xyz="0.0 0.0 0.0" rpy="1.571 0.0 0.0" />
+        <geometry>
+          <mesh filename="package://manipulator_description/meshes/visual/link10.dae"/>
+        </geometry>
+      </collision>
+      <inertial>
+        <origin xyz="0.0 0.0 0.0" rpy="1.571 0.0 0.0"/>
+        <mass value="0.007"/>
+        <inertia ixx="1.48840827e-6"  ixy="2.49592487e-8"  ixz="5.30644674e-12" iyy="2.08108627e-6" iyz="2.38181240e-14" izz="6.88193128e-7" />
+      </inertial>
+    </link>
+    <joint name="${arm_id}_joint9" type="continuous">
+      <origin rpy="0 0 1.571" xyz="0 0 0.025"/>
+      <parent link="${arm_id}_link8"/>
+      <child link="${arm_id}_link9"/>
+      <axis xyz="0 0 1" rpy="0 0 0"/>
+    </joint>
+    <transmission name="trans_timon_joint1">
+        <type>transmission_interface/SimpleTransmission</type>
+        <joint name="timon_joint1">
+            <hardwareInterface>hardware_interface/PositionJointInterface</hardwareInterface>
+        </joint>
+        <actuator name="timon_joint1_motor">
+            <hardwareInterface>hardware_interface/PositionJointInterface</hardwareInterface>
+            <mechanicalReduction>1</mechanicalReduction>
+        </actuator>
+    </transmission>
+    <transmission name="trans_timon_joint4">
+        <type>transmission_interface/SimpleTransmission</type>
+        <joint name="timon_joint4">
+            <hardwareInterface>hardware_interface/PositionJointInterface</hardwareInterface>
+        </joint>
+        <actuator name="timon_joint4_motor">
+            <hardwareInterface>hardware_interface/PositionJointInterface</hardwareInterface>
+            <mechanicalReduction>1</mechanicalReduction>
+        </actuator>
+    </transmission>
+    <transmission name="trans_timon_joint7">
+        <type>transmission_interface/SimpleTransmission</type>
+        <joint name="timon_joint7">
+            <hardwareInterface>hardware_interface/PositionJointInterface</hardwareInterface>
+        </joint>
+        <actuator name="timon_joint7_motor">
+            <hardwareInterface>hardware_interface/PositionJointInterface</hardwareInterface>
+            <mechanicalReduction>1</mechanicalReduction>
+        </actuator>
+    </transmission>
+    <transmission name="trans_timon_joint9">
+        <type>transmission_interface/SimpleTransmission</type>
+        <joint name="timon_joint9">
+            <hardwareInterface>hardware_interface/PositionJointInterface</hardwareInterface>
+        </joint>
+        <actuator name="timon_joint9_motor">
+            <hardwareInterface>hardware_interface/PositionJointInterface</hardwareInterface>
+            <mechanicalReduction>1</mechanicalReduction>
+        </actuator>
+    </transmission>
+    <!-- <link name="${arm_id}_link11">
+      <visual>
+        <origin xyz="0.0225 -0.007 0.0" rpy="0.0 0.0 0.0" />
+        <geometry>
+          <mesh filename="package://manipulator_description/meshes/visual/link11.dae"/>
+        </geometry>
+      </visual>
+      <collision>
+        <origin xyz="0.0225 -0.007 0.0" rpy="0.0 0.0 0.0" />
+        <geometry>
+          <mesh filename="package://manipulator_description/meshes/visual/link11.dae"/>
+        </geometry>
+      </collision>
+      <inertial>
+        <origin xyz="0.0225 -0.007 0.0" rpy="0.0 0.0 0.0"/>
+        <mass value="0.16499216"/>
+        <inertia ixx="7.88952550e-5"  ixy="-3.13065901e-9"  ixz="4.40693303e-9" iyy="4.39861799e-5" iyz="-2.02737764e-6" izz="6.23603662e-5" />
+      </inertial>
+    </link>
+    <joint name="${arm_id}_joint11" type="fixed">
+      <origin rpy="1.5701 0.0 0.0" xyz="0.0 -0.001 0.055"/>
+      <parent link="${arm_id}_link10"/>
+      <child link="${arm_id}_link11"/>
+    </joint>
+   <link name="${arm_id}_link12">
+      <visual>
+        <origin xyz="0.0 0.0 0.0" rpy="0.0 1.571 0.0" />
+        <geometry>
+          <mesh filename="package://manipulator_description/meshes/visual/link12.dae"/>
+        </geometry>
+      </visual>
+      <collision>
+        <origin xyz="0.0 0.0 0.0" rpy="0.0 1.571 0.0" />
+        <geometry>
+          <mesh filename="package://manipulator_description/meshes/visual/link12.dae"/>
+        </geometry>
+      </collision>
+      <inertial>
+        <origin xyz="0.0 0.0 0.0" rpy="0.0 1.571 0.0"/>
+        <mass value="0.01873963"/>
+        <inertia ixx="4.49588271e-6"  ixy="0.00000000e+0"  ixz="0.00000000e+0" iyy="1.08113872e-5" iyz="0.00000000e+0" izz="1.12040418e-5" />
+      </inertial>
+    </link>
+    <joint name="${arm_id}_joint12" type="revolute">
+      <safety_controller k_position="100.0" k_velocity="40.0" soft_lower_limit="-1.90" soft_upper_limit="1.90"/>
+      <origin rpy="0.0 0.0 0.0" xyz="0.0 0.0 0.0"/>
+      <parent link="${arm_id}_link11"/>
+      <child link="${arm_id}_link12"/>
       <axis xyz="0 0 1"/>
-      <limit effort="1000.0" lower="-0.95" upper="2.36" velocity="0.5"/>
-    </joint>
+      <limit effort="1000.0" lower="-1.90" upper="1.90" velocity="0.5"/>
+    </joint>  -->
   </xacro:macro>
 </robot>

File: manipulator_description/robots/timon_arm_hand.urdf.xacro (robot description, xacro)
@@ -1,7 +1,15 @@
 <?xml version="1.0" encoding="utf-8"?>
 <robot xmlns:xacro="http://www.ros.org/wiki/xacro" name="timon">
+  <link name ="base_link">
+  </link>
+  <xacro:include filename="$(find manipulator_description)/urdf/base.xacro"/>
   <xacro:include filename="$(find manipulator_description)/robots/timon_arm.xacro"/>
   <xacro:include filename="$(find manipulator_description)/robots/hand.xacro"/>
   <xacro:timon_arm />
-  <xacro:hand ns="timon" rpy="0 -1.571 -1.571" xyz="0 0.41 0.013" connected_to="timon_link8"/>
+  <xacro:hand ns="timon" rpy="1.5701 0.0 0.0" xyz="0.0 -0.001 0.055" connected_to="timon_link9"/>
+  <gazebo>
+      <plugin name="gazebo_ros_control" filename="libgazebo_ros_control.so">
+          <robotNamespace>timon</robotNamespace>
+      </plugin>
+  </gazebo>
 </robot>

File: manipulator_description/urdf/base.xacro (robot description, xacro)
@@ -1,28 +1,28 @@
 <?xml version="1.0"?>
 <robot name="manipulador_base" xmlns:xacro="http://ros.org/wiki/xacro">
-<!--Base_to_manipulator-->
-  <link name="base_to_manipulator">
-    <visual>
-      <origin rpy="0 0 0" xyz="0 0 0"/>
-      <geometry>
-        <mesh filename="package://manipulator_description/meshes/basem.dae"/>
-      </geometry>
-    </visual>
-    <collision>
-      <origin rpy="0 0 0" xyz="0 0 0"/>
-      <geometry>
-        <mesh filename="package://manipulator_description/meshes/basem.stl"/>
-      </geometry>
-    </collision>
-    <inertial>
-      <origin rpy="0 0 0" xyz="0 0 0"/>
-      <mass value="2.86661792"/>
-      <inertia ixx="8.72078676e-3" ixy="-9.55785583e-9" ixz="0" iyx="-9.55785583e-9" iyy="4.66430350e-2" iyz="0" izx="0" izy="-0" izz="5.35109282e-2"/>
-    </inertial>
+  <!--Base_to_manipulator-->
+    <link name="base_to_manipulator">
+      <visual>
+        <origin rpy="0 0 0" xyz="0 0 0"/>
+        <geometry>
+          <mesh filename="package://manipulator_description/meshes/basem.dae"/>
+        </geometry>
+      </visual>
+      <collision>
+        <origin rpy="0 0 0" xyz="0 0 0"/>
+        <geometry>
+          <mesh filename="package://manipulator_description/meshes/basem.stl"/>
+        </geometry>
+      </collision>
+      <inertial>
+        <origin rpy="0 0 0" xyz="0 0 0"/>
+        <mass value="2.86661792"/>
+        <inertia ixx="8.72078676e-3" ixy="-9.55785583e-9" ixz="0" iyx="-9.55785583e-9" iyy="4.66430350e-2" iyz="0" izx="0" izy="-0" izz="5.35109282e-2"/>
+      </inertial>
     </link>
-    <joint name="base_to_world1" type="fixed">
-      <parent link="world"/>
-      <child link="base_to_manipulator"/>
-      <origin rpy="0 0 1.57" xyz="0.45 0 1.56"/>
-    </joint>
+      <joint name="base_to_world1" type="fixed">
+        <parent link="base_link"/>
+        <child link="base_to_manipulator"/>
+        <origin rpy="0 0 0" xyz="0.45 0 0"/>
+      </joint>
 </robot>
