Commit message: new urdf

File: manipulator_description/robots/timon_arm.xacro (robot description, xacro)
@@ -18,19 +18,19 @@
     <link name="${arm_id}_link0">
       <visual>
-        <origin xyz="0 0 0" rpy="1.571 0 0" />
-        <geometry>
-          <mesh filename="package://${description_pkg}/meshes/visual/link1.dae"/>
-        </geometry>
-      </visual>
-      <collision>
-        <origin xyz="0 0 0" rpy="1.571 0 0" />
-        <geometry>
-          <mesh filename="package://${description_pkg}/meshes/visual/link1.dae"/>
-        </geometry>
-      </collision>
-      <inertial>
-        <origin xyz="0 0 0" rpy="1.571 0 0 "/>
-        <mass value="0.856"/>
-        <inertia ixx="1.26094285e-3"  ixy="0.00000e+0"  ixz="0.00000e+0" iyy="3.79002180e-4" iyz="-5.78993250e-9" izz="1.26040377e-3" />
+        <origin xyz="0 0 0" rpy="0 0 0" />
+        <geometry>
+          <mesh filename="package://${description_pkg}/meshes/JeRoTIMON/id_1.dae"/>
+        </geometry>
+      </visual>
+      <collision>
+        <origin xyz="0 0 0" rpy="0 0 0" />
+        <geometry>
+          <mesh filename="package://${description_pkg}/meshes/JeRoTIMON/id_1.dae"/>
+        </geometry>
+      </collision>
+      <inertial>
+        <origin xyz="0 0 0" rpy="0 0 0 "/>
+        <mass value="3.72486532"/>
+        <inertia ixx="0.011"  ixy="-9.466e-9"  ixz="-0.00000563" iyy="0.04868026" iyz="0" izz="0.05388592" />
       </inertial>
     </link>
@@ -42,24 +42,24 @@
     <link name="${arm_id}_link1">
       <visual>
-        <origin xyz="0 0 0" rpy="-3.14 0 0" />
-        <geometry>
-          <mesh filename="package://${description_pkg}/meshes/visual/link2.dae"/>
-        </geometry>
-      </visual>
-      <collision>
-        <origin xyz="0 0 0" rpy="-3.14 0 0" />
-        <geometry>
-          <mesh filename="package://${description_pkg}/meshes/visual/link2.dae"/>
-        </geometry>
-      </collision>
-      <inertial>
-        <origin xyz="0 0 0" rpy="-3.14 0 0 "/>
-        <mass value="0.15040432"/>
-        <inertia ixx="3.45063e+1"  ixy="0.00000e+0"  ixz="0.00000e+0" iyy="1.07762e+2" iyz="0.00000e+0" izz="1.38659e+2" />
+        <origin xyz="0 0 0" rpy="0 0 0" />
+        <geometry>
+          <mesh filename="package://${description_pkg}/meshes/JeRoTIMON/id_2.dae"/>
+        </geometry>
+      </visual>
+      <collision>
+        <origin xyz="0 0 0" rpy="0 0 0" />
+        <geometry>
+          <mesh filename="package://${description_pkg}/meshes/JeRoTIMON/id_2.dae"/>
+        </geometry>
+      </collision>
+      <inertial>
+        <origin xyz="0 0 0" rpy="0 0 0 "/>
+        <mass value="1.00643107"/>
+        <inertia ixx="0.00055282"  ixy="0"  ixz="-0.00005159" iyy="0.00152712" iyz="0.00000e+0" izz="0.00141817" />
       </inertial>
     </link>
     <joint name="${arm_id}_joint1" type="continuous">
       <safety_controller k_position="100.0" k_velocity="40.0"/>
-      <origin rpy="3.14 0 0" xyz="0 0 0.036"/>
+      <origin rpy="0 0 0" xyz="0 0 0.12715351"/>
       <parent link="${arm_id}_link0"/>
       <child link="${arm_id}_link1"/>
@@ -68,72 +68,74 @@
     <link name="${arm_id}_link2">
       <visual>
-        <origin xyz="0 0 0" rpy="1.571 0 0" />
-        <geometry>
-          <mesh filename="package://${description_pkg}/meshes/visual/link3.dae"/>
-        </geometry>
-      </visual>
-      <collision>
-        <origin xyz="0 0 0" rpy="1.571 0 0" />
-        <geometry>
-          <mesh filename="package://${description_pkg}/meshes/visual/link3.dae"/>
-        </geometry>
-      </collision>
-      <inertial>
-        <origin xyz="0 0 0" rpy="1.571 0 0 "/>
-        <mass value="0.856"/>
-        <inertia ixx="1.26094285e-3"  ixy="0.00000e+0"  ixz="0.00000e+0" iyy="3.79002180e-4" iyz="-5.78993250e-9" izz="1.26040377e-3" />
-      </inertial>
-    </link>
-    <joint name="${arm_id}_joint2" type="fixed">
-      <origin rpy="-1.571 1.571 1.571" xyz="-0.04 0.0 -0.039"/>
+        <origin xyz="0 0 0" rpy="0 0 0" />
+        <geometry>
+          <mesh filename="package://${description_pkg}/meshes/JeRoTIMON/id_3.dae"/>
+        </geometry>
+      </visual>
+      <collision>
+        <origin xyz="0 0 0" rpy="0 0 0" />
+        <geometry>
+          <mesh filename="package://${description_pkg}/meshes/JeRoTIMON/id_3.dae"/>
+        </geometry>
+      </collision>
+      <inertial>
+        <origin xyz="0 0 0" rpy="0 0 0 "/>
+        <mass value="1.96131158"/>
+        <inertia ixx="0.0593682"  ixy="0.00019981"  ixz="0.0024082" iyy="0.06052018" iyz="-0.00320203" izz="0.00314458" />
+      </inertial>
+    </link>
+    <joint name="${arm_id}_joint2" type="continuous">
+      <origin rpy="0 0 0" xyz="0 0 0.03900000"/>
       <parent link="${arm_id}_link1"/>
       <child link="${arm_id}_link2"/>
+      <axis xyz="-1 0 0" rpy="0 0 0"/>
     </joint>
     <link name="${arm_id}_link3">
       <visual>
-        <origin xyz="0 0 0" rpy="1.571 0 0" />
-        <geometry>
-          <mesh filename="package://${description_pkg}/meshes/visual/link4.dae"/>
-        </geometry>
-      </visual>
-      <collision>
-        <origin xyz="0 0 0" rpy="1.571 0 0" />
-        <geometry>
-          <mesh filename="package://${description_pkg}/meshes/visual/link4.dae"/>
-        </geometry>
-      </collision>
-      <inertial>
-        <origin xyz="0 0 0" rpy="1.571 0 0 "/>
-        <mass value="0.03239855"/>
-        <inertia ixx="9.57551961e-6"  ixy="-1.52519365e-14"  ixz="7.17291197e-16" iyy="9.41926366e-6" iyz="1.37735170e-11" izz="1.88295847e-5" />
-      </inertial>
-    </link>
-    <joint name="${arm_id}_joint3" type="fixed">
-      <origin rpy="1.571 0.0 0.0" xyz="0.0 0.0 -0.093"/>
+        <origin xyz="0 0 0" rpy="0 0 0" />
+        <geometry>
+          <mesh filename="package://${description_pkg}/meshes/JeRoTIMON/id_4.dae"/>
+        </geometry>
+      </visual>
+      <collision>
+        <origin xyz="0 0 0" rpy="0 0 0" />
+        <geometry>
+          <mesh filename="package://${description_pkg}/meshes/JeRoTIMON/id_4.dae"/>
+        </geometry>
+      </collision>
+      <inertial>
+        <origin xyz="0 0 0" rpy="0 0 0 "/>
+        <mass value="1.96131158"/>
+        <inertia ixx="0.0593682"  ixy="0.00019981"  ixz="0.0024082" iyy="0.06052018" iyz="-0.00320203" izz="0.00314458" />
+      </inertial>
+    </link>
+    <joint name="${arm_id}_joint3" type="continuous">
+      <origin rpy="0 0.0 0.0" xyz="0 0.02683555 0.46242180"/>
       <parent link="${arm_id}_link2"/>
       <child link="${arm_id}_link3"/>
+      <axis xyz="-1 0 0" rpy="0 0 0"/>
     </joint>
     <link name="${arm_id}_link4">
       <visual>
-        <origin xyz="-0.0292 0.2289 -0.04" rpy="0 1.571 0" />
-        <geometry>
-          <mesh filename="package://${description_pkg}/meshes/visual/link5.dae"/>
-        </geometry>
-      </visual>
-      <collision>
-        <origin xyz="-0.0292 0.2289 -0.04" rpy="0 1.571 0" />
-        <geometry>
-          <mesh filename="package://${description_pkg}/meshes/visual/link5.dae"/>
-        </geometry>
-      </collision>
-      <inertial>
-        <origin xyz="-0.0292 0.2289 -0.04" rpy="0 1.571 0 "/>
-        <mass value="1.09212028"/>
-        <inertia ixx="2.47891806e-2"  ixy="-5.41904580e-4"  ixz="-2.41956050e-7" iyy="1.48343837e-3" iyz="-8.20873087e-6" izz="2.53662704e-2" />
+        <origin xyz="0 0 0" rpy="0 0 0" />
+        <geometry>
+          <mesh filename="package://${description_pkg}/meshes/JeRoTIMON/id_5.dae"/>
+        </geometry>
+      </visual>
+      <collision>
+        <origin xyz="0 0 0" rpy="0 0 0" />
+        <geometry>
+          <mesh filename="package://${description_pkg}/meshes/JeRoTIMON/id_5.dae"/>
+        </geometry>
+      </collision>
+      <inertial>
+        <origin xyz="0 0 0" rpy="0 0 0 "/>
+        <mass value="0.37561629"/>
+        <inertia ixx="0.00025385"  ixy="0"  ixz="0" iyy="0.00011288" iyz="0.00000228" izz="0.00025011" />
       </inertial>
     </link>
     <joint name="${arm_id}_joint4" type="revolute">
       <safety_controller k_position="100.0" k_velocity="40.0" soft_lower_limit="-1.77" soft_upper_limit="1.77"/>
-      <origin rpy="0 -1.571 -1.571" xyz="-0.0008 0.093 0.001"/>
+      <origin rpy="0 0 0" xyz="0.00739115 -0.03075115 0.44053087"/>
       <parent link="${arm_id}_link3"/>
       <child link="${arm_id}_link4"/>
@@ -141,4 +143,5 @@
       <limit effort="1000.0" lower="-1.77" upper="1.77" velocity="0.5"/>
     </joint>
+<!--
     <link name="${arm_id}_link5">
       <visual>
@@ -365,5 +368,5 @@
             <mechanicalReduction>1</mechanicalReduction>
         </actuator>
-    </transmission>
+    </transmission> -->
   </xacro:macro>
 </robot>

File: manipulator_description/robots/timon_arm_hand_base.urdf.xacro (robot description, xacro)
@@ -3,21 +3,22 @@
   <link name = "world">
   </link>
-  <xacro:include filename="$(find manipulator_description)/robots/base.xacro"/>
+  <!-- <xacro:include filename="$(find manipulator_description)/robots/base.xacro"/> -->
   <xacro:include filename="$(find manipulator_description)/robots/timon_arm.urdf.xacro"/>
-  <xacro:include filename="$(find manipulator_description)/robots/camera.xacro"/>
-    <joint name ="world_to_base" type="fixed">
+  <!-- <xacro:include filename="$(find manipulator_description)/robots/camera.xacro"/>
+   -->
+    <!-- <joint name ="world_to_base" type="fixed">
         <origin rpy="0 0 0" xyz="0.6 0 1.56"/>
         <parent link="world"/>
         <child link = "base_to_manipulator"/>
-    </joint>
+    </joint> -->
     <joint name ="base_to_timon" type="fixed">
         <origin rpy="0 0 -1.571" xyz="0 0 0.1"/>
-        <parent link="base_to_manipulator"/>
+        <parent link="world"/>
         <child link = "invisible_link"/>
     </joint>
-    <joint name ="base_to_camera" type="fixed">
+    <!-- <joint name ="base_to_camera" type="fixed">
         <origin rpy="-1.571 3.1415 -1.571" xyz="0.0661 0.426 0.0123"/>
         <parent link="timon_link7"/>
         <child link = "camera"/>
-    </joint>
+    </joint> -->
 </robot>

Commit message: finished first version

File: manipulator_description/robots/timon_arm.xacro (robot description, xacro)
@@ -137,5 +137,6 @@
     <joint name="${arm_id}_joint4" type="revolute">
       <safety_controller k_position="100.0" k_velocity="40.0" soft_lower_limit="-1.77" soft_upper_limit="1.77"/>
-      <origin rpy="0 0 0" xyz="0.00739115 -0.03075115 0.44053087"/>
+      <origin rpy="0 0 0" xyz="-0.00739115 -0.03075115 0.44053087"/>
+      <!-- 0.00739115 -->
       <parent link="${arm_id}_link3"/>
       <child link="${arm_id}_link4"/>
@@ -143,29 +144,30 @@
       <limit effort="1000.0" lower="-1.77" upper="1.77" velocity="0.5"/>
     </joint>
-<!--
     <link name="${arm_id}_link5">
       <visual>
-        <origin xyz="0.0 0.0 0.0" rpy="0 0 -0.75" />
-        <geometry>
-          <mesh filename="package://${description_pkg}/meshes/visual/link6.dae"/>
-        </geometry>
-      </visual>
-      <collision>
-        <origin xyz="0.0 0.0 0.0" rpy="0 0 -0.75" />
-        <geometry>
-          <mesh filename="package://${description_pkg}/meshes/visual/link6.dae"/>
-        </geometry>
-      </collision>
-      <inertial>
-        <origin xyz="0.0 0.0 0.0" rpy="0 0 -0.75 "/>
+        <origin xyz="0.0 0.0 0.0" rpy="0 0 0" />
+        <geometry>
+          <mesh filename="package://${description_pkg}/meshes/JeRoTIMON/id_6.dae"/>
+        </geometry>
+      </visual>
+      <collision>
+        <origin xyz="0.0 0.0 0.0" rpy="0 0 0" />
+        <geometry>
+          <mesh filename="package://${description_pkg}/meshes/JeRoTIMON/id_6.dae"/>
+        </geometry>
+      </collision>
+      <inertial>
+        <origin xyz="0.0 0.0 0.0" rpy="0 0 0 "/>
         <mass value="0.16505359"/>
         <inertia ixx="7.89080915e-5"  ixy="-3.13361612e-9"  ixz="4.40720922e-9" iyy="4.40037283e-5" iyz="-2.02636752e-6" izz="6.23905424e-5" />
       </inertial>
     </link>
-    <joint name="${arm_id}_joint5" type="fixed">
-      <origin rpy="0 0 0" xyz="0.03 0.451 -0.015"/>
+    <joint name="${arm_id}_joint5" type="continuous">
+      <origin rpy="0 0 0" xyz="0 0 0.027"/>
       <parent link="${arm_id}_link4"/>
       <child link="${arm_id}_link5"/>
-    </joint>
+      <axis xyz="0 1 0" rpy="0 0 0"/>
+    </joint>
+<!--
     <link name="${arm_id}_link6">
       <visual>

Commit message: change joints names

File: manipulator_description/robots/timon_arm.xacro (robot description, xacro)
@@ -59,5 +59,5 @@
       </inertial>
     </link>
-    <joint name="${arm_id}_joint1" type="continuous">
+    <joint name="id_1" type="continuous">
       <safety_controller k_position="100.0" k_velocity="40.0"/>
       <origin rpy="0 0 0" xyz="0 0 0.12715351"/>
@@ -85,5 +85,5 @@
       </inertial>
     </link>
-    <joint name="${arm_id}_joint2" type="continuous">
+    <joint name="id_2" type="continuous">
       <origin rpy="0 0 0" xyz="0 0 0.03900000"/>
       <parent link="${arm_id}_link1"/>
@@ -110,5 +110,5 @@
       </inertial>
     </link>
-    <joint name="${arm_id}_joint3" type="continuous">
+    <joint name="id_3" type="continuous">
       <origin rpy="0 0.0 0.0" xyz="0 0.02683555 0.46242180"/>
       <parent link="${arm_id}_link2"/>
@@ -135,5 +135,5 @@
       </inertial>
     </link>
-    <joint name="${arm_id}_joint4" type="revolute">
+    <joint name="id_4" type="revolute">
       <safety_controller k_position="100.0" k_velocity="40.0" soft_lower_limit="-1.77" soft_upper_limit="1.77"/>
       <origin rpy="0 0 0" xyz="-0.00739115 -0.03075115 0.44053087"/>
@@ -163,5 +163,5 @@
       </inertial>
     </link>
-    <joint name="${arm_id}_joint5" type="continuous">
+    <joint name="id_5" type="continuous">
       <origin rpy="0 0 0" xyz="0 0 0.027"/>
       <parent link="${arm_id}_link4"/>
@@ -169,4 +169,54 @@
       <axis xyz="0 1 0" rpy="0 0 0"/>
     </joint>
+    <transmission name="trans_timon_joint1">
+        <type>transmission_interface/SimpleTransmission</type>
+        <joint name="id_1">
+            <hardwareInterface>hardware_interface/PositionJointInterface</hardwareInterface>
+        </joint>
+        <actuator name="timon_joint1_motor">
+            <hardwareInterface>hardware_interface/PositionJointInterface</hardwareInterface>
+            <mechanicalReduction>1</mechanicalReduction>
+        </actuator>
+    </transmission>
+    <transmission name="trans_timon_joint2">
+        <type>transmission_interface/SimpleTransmission</type>
+        <joint name="id_2">
+            <hardwareInterface>hardware_interface/PositionJointInterface</hardwareInterface>
+        </joint>
+        <actuator name="timon_joint2_motor">
+            <hardwareInterface>hardware_interface/PositionJointInterface</hardwareInterface>
+            <mechanicalReduction>1</mechanicalReduction>
+        </actuator>
+    </transmission>
+    <transmission name="trans_timon_joint3">
+        <type>transmission_interface/SimpleTransmission</type>
+        <joint name="id_3">
+            <hardwareInterface>hardware_interface/PositionJointInterface</hardwareInterface>
+        </joint>
+        <actuator name="timon_joint3_motor">
+            <hardwareInterface>hardware_interface/PositionJointInterface</hardwareInterface>
+            <mechanicalReduction>1</mechanicalReduction>
+        </actuator>
+    </transmission>
+    <transmission name="trans_timon_joint4">
+        <type>transmission_interface/SimpleTransmission</type>
+        <joint name="id_4">
+            <hardwareInterface>hardware_interface/PositionJointInterface</hardwareInterface>
+        </joint>
+        <actuator name="timon_joint4_motor">
+            <hardwareInterface>hardware_interface/PositionJointInterface</hardwareInterface>
+            <mechanicalReduction>1</mechanicalReduction>
+        </actuator>
+    </transmission>
+    <transmission name="trans_timon_joint5">
+        <type>transmission_interface/SimpleTransmission</type>
+        <joint name="id_5">
+            <hardwareInterface>hardware_interface/PositionJointInterface</hardwareInterface>
+        </joint>
+        <actuator name="timon_joint5_motor">
+            <hardwareInterface>hardware_interface/PositionJointInterface</hardwareInterface>
+            <mechanicalReduction>1</mechanicalReduction>
+        </actuator>
+    </transmission>
 <!--
     <link name="${arm_id}_link6">
@@ -321,54 +371,5 @@
       <limit effort="1000.0" lower="-1.90" upper="1.90" velocity="0.5"/>
     </joint>
-    <transmission name="trans_timon_joint1">
-        <type>transmission_interface/SimpleTransmission</type>
-        <joint name="timon_joint1">
-            <hardwareInterface>hardware_interface/PositionJointInterface</hardwareInterface>
-        </joint>
-        <actuator name="timon_joint1_motor">
-            <hardwareInterface>hardware_interface/PositionJointInterface</hardwareInterface>
-            <mechanicalReduction>1</mechanicalReduction>
-        </actuator>
-    </transmission>
-    <transmission name="trans_timon_joint4">
-        <type>transmission_interface/SimpleTransmission</type>
-        <joint name="timon_joint4">
-            <hardwareInterface>hardware_interface/PositionJointInterface</hardwareInterface>
-        </joint>
-        <actuator name="timon_joint4_motor">
-            <hardwareInterface>hardware_interface/PositionJointInterface</hardwareInterface>
-            <mechanicalReduction>1</mechanicalReduction>
-        </actuator>
-    </transmission>
-    <transmission name="trans_timon_joint7">
-        <type>transmission_interface/SimpleTransmission</type>
-        <joint name="timon_joint7">
-            <hardwareInterface>hardware_interface/PositionJointInterface</hardwareInterface>
-        </joint>
-        <actuator name="timon_joint7_motor">
-            <hardwareInterface>hardware_interface/PositionJointInterface</hardwareInterface>
-            <mechanicalReduction>1</mechanicalReduction>
-        </actuator>
-    </transmission>
-    <transmission name="trans_timon_joint9">
-        <type>transmission_interface/SimpleTransmission</type>
-        <joint name="timon_joint9">
-            <hardwareInterface>hardware_interface/PositionJointInterface</hardwareInterface>
-        </joint>
-        <actuator name="timon_joint9_motor">
-            <hardwareInterface>hardware_interface/PositionJointInterface</hardwareInterface>
-            <mechanicalReduction>1</mechanicalReduction>
-        </actuator>
-    </transmission>
-    <transmission name="trans_timon_joint11">
-        <type>transmission_interface/SimpleTransmission</type>
-        <joint name="timon_joint11">
-            <hardwareInterface>hardware_interface/PositionJointInterface</hardwareInterface>
-        </joint>
-        <actuator name="timon_joint11_motor">
-            <hardwareInterface>hardware_interface/PositionJointInterface</hardwareInterface>
-            <mechanicalReduction>1</mechanicalReduction>
-        </actuator>
-    </transmission> -->
+ -->
   </xacro:macro>
 </robot>

Commit message: added camera and change frame 42

File: manipulator_description/robots/timon_arm.xacro (robot description, xacro)
@@ -120,4 +120,29 @@
         <origin xyz="0 0 0" rpy="0 0 0" />
         <geometry>
+          <mesh filename="package://${description_pkg}/meshes/JeRoTIMON/suport_cam.dae"/>
+        </geometry>
+      </visual>
+      <collision>
+        <origin xyz="0 0 0" rpy="0 0 0" />
+        <geometry>
+          <mesh filename="package://${description_pkg}/meshes/JeRoTIMON/suport_cam.dae"/>
+        </geometry>
+      </collision>
+      <inertial>
+        <origin xyz="0 0 0" rpy="0 0 0 "/>
+        <mass value="0.20608656"/>
+        <inertia ixx="0.00039102"  ixy="0"  ixz="-8.254e-9" iyy="0.00045673" iyz="-0.00006629" izz="0.00023588" />
+      </inertial>
+    </link>
+    <joint name="suport_cam" type="fixed">
+      <origin rpy="0 0.0 0.0" xyz="-0.00754115 -0.03075116 0.37653086"/>
+      <parent link="${arm_id}_link3"/>
+      <child link="${arm_id}_link4"/>
+      <axis xyz="0 0 0" rpy="0 0 0"/>
+    </joint>
+    <link name="${arm_id}_link5">
+      <visual>
+        <origin xyz="0 0 0" rpy="0 0 0" />
+        <geometry>
           <mesh filename="package://${description_pkg}/meshes/JeRoTIMON/id_5.dae"/>
         </geometry>
@@ -137,12 +162,12 @@
     <joint name="id_4" type="revolute">
       <safety_controller k_position="100.0" k_velocity="40.0" soft_lower_limit="-1.77" soft_upper_limit="1.77"/>
-      <origin rpy="0 0 0" xyz="-0.00739115 -0.03075115 0.44053087"/>
+      <origin rpy="0 0 0" xyz="0 0 0.06370001"/>
       <!-- 0.00739115 -->
-      <parent link="${arm_id}_link3"/>
-      <child link="${arm_id}_link4"/>
+      <parent link="${arm_id}_link4"/>
+      <child link="${arm_id}_link5"/>
       <axis xyz="0 0 1"/>
       <limit effort="1000.0" lower="-1.77" upper="1.77" velocity="0.5"/>
     </joint>
-    <link name="${arm_id}_link5">
+    <link name="${arm_id}_link6">
       <visual>
         <origin xyz="0.0 0.0 0.0" rpy="0 0 0" />
@@ -159,12 +184,12 @@
       <inertial>
         <origin xyz="0.0 0.0 0.0" rpy="0 0 0 "/>
-        <mass value="0.16505359"/>
-        <inertia ixx="7.89080915e-5"  ixy="-3.13361612e-9"  ixz="4.40720922e-9" iyy="4.40037283e-5" iyz="-2.02636752e-6" izz="6.23905424e-5" />
+        <mass value="0.08694786"/>
+        <inertia ixx="0.00012963"  ixy="0"  ixz="0" iyy="0.00012601" iyz="-0.00000408" izz="0.00003715" />
       </inertial>
     </link>
     <joint name="id_5" type="continuous">
-      <origin rpy="0 0 0" xyz="0 0 0.027"/>
-      <parent link="${arm_id}_link4"/>
-      <child link="${arm_id}_link5"/>
+      <origin rpy="0 0 0" xyz="0 -0.00607092 0.027"/>
+      <parent link="${arm_id}_link5"/>
+      <child link="${arm_id}_link6"/>
       <axis xyz="0 1 0" rpy="0 0 0"/>
     </joint>

File: manipulator_description/robots/timon_arm_hand_base.urdf.xacro (robot description, xacro)
@@ -5,6 +5,5 @@
   <!-- <xacro:include filename="$(find manipulator_description)/robots/base.xacro"/> -->
   <xacro:include filename="$(find manipulator_description)/robots/timon_arm.urdf.xacro"/>
-  <!-- <xacro:include filename="$(find manipulator_description)/robots/camera.xacro"/>
-   -->
+   <xacro:include filename="$(find manipulator_description)/robots/camera.xacro"/>
     <!-- <joint name ="world_to_base" type="fixed">
         <origin rpy="0 0 0" xyz="0.6 0 1.56"/>
@@ -17,8 +16,9 @@
         <child link = "invisible_link"/>
     </joint>
-    <!-- <joint name ="base_to_camera" type="fixed">
-        <origin rpy="-1.571 3.1415 -1.571" xyz="0.0661 0.426 0.0123"/>
-        <parent link="timon_link7"/>
+    <joint name ="base_to_camera" type="fixed">
+        <origin rpy="0 -1.57 -1.57" xyz="0 0.07134918 0.02016139"/>
+        <!-- <origin rpy="-1.571 3.1415 -1.571" xyz="0.0661 0.426 0.0123"/> -->
+        <parent link="timon_link4"/>
         <child link = "camera"/>
-    </joint> -->
+    </joint>
 </robot>
