Commit message: fix link position

File: manipulator_description/robots/timon_arm.xacro (robot description, xacro)
@@ -111,5 +111,5 @@
     </link>
     <joint name="id_3" type="continuous">
-      <origin rpy="0 0.0 0.0" xyz="0 0.02683555 0.46242180"/>
+      <origin rpy="0 0.0 -3.14" xyz="-0.01400000 0.02683555 0.46242180"/>
       <parent link="${arm_id}_link2"/>
       <child link="${arm_id}_link3"/>

Commit message: fix link position

File: manipulator_description/robots/timon_arm.xacro (robot description, xacro)
@@ -111,5 +111,5 @@
     </link>
     <joint name="id_3" type="continuous">
-      <origin rpy="0 0.0 -3.14" xyz="-0.01400000 0.02683555 0.46242180"/>
+      <origin rpy="0 0.0 0" xyz="0 0.02683555 0.46242180"/>
       <parent link="${arm_id}_link2"/>
       <child link="${arm_id}_link3"/>
@@ -136,5 +136,5 @@
     </link>
     <joint name="suport_cam" type="fixed">
-      <origin rpy="0 0.0 0.0" xyz="-0.00754115 -0.03075116 0.37653086"/>
+      <origin rpy="0 0.0 -3.14" xyz="-0.00754115 -0.03075116 0.37653086"/>
       <parent link="${arm_id}_link3"/>
       <child link="${arm_id}_link4"/>

Commit message: adding joint limits

File: manipulator_description/robots/timon_arm.xacro (robot description, xacro)
@@ -59,10 +59,10 @@
       </inertial>
     </link>
-    <joint name="id_1" type="continuous">
-      <safety_controller k_position="100.0" k_velocity="40.0"/>
+    <joint name="id_1" type="revolute">
       <origin rpy="0 0 0" xyz="0 0 0.12715351"/>
       <parent link="${arm_id}_link0"/>
       <child link="${arm_id}_link1"/>
       <axis xyz="0 0 1" rpy="0 0 0"/>
+      <limit effort="1000.0" lower="-1.5" upper="1.5" velocity="0.5"/> <!--  -0.783    0.783-->
     </joint>
     <link name="${arm_id}_link2">
@@ -85,9 +85,10 @@
       </inertial>
     </link>
-    <joint name="id_2" type="continuous">
+    <joint name="id_2" type="revolute">
       <origin rpy="0 0 0" xyz="0 0 0.03900000"/>
       <parent link="${arm_id}_link1"/>
       <child link="${arm_id}_link2"/>
       <axis xyz="-1 0 0" rpy="0 0 0"/>
+      <limit effort="1000.0" lower="-3.14" upper="3.14" velocity="0.5"/> <!-- -1.5708   1.5708-->
     </joint>
     <link name="${arm_id}_link3">
@@ -110,9 +111,10 @@
       </inertial>
     </link>
-    <joint name="id_3" type="continuous">
+    <joint name="id_3" type="revolute">
       <origin rpy="0 0.0 0.0" xyz="0 0.02683555 0.46242180"/>
       <parent link="${arm_id}_link2"/>
       <child link="${arm_id}_link3"/>
       <axis xyz="-1 0 0" rpy="0 0 0"/>
+      <limit effort="1000.0" lower="-3.14" upper="3.14" velocity="0.5"/>  <!-- -0.74    3.03-->
     </joint>
     <link name="${arm_id}_link4">
@@ -167,5 +169,5 @@
       <child link="${arm_id}_link5"/>
       <axis xyz="0 0 1"/>
-      <limit effort="1000.0" lower="-1.77" upper="1.77" velocity="0.5"/>
+      <limit effort="1000.0" lower="-3.14" upper="3.14" velocity="0.5"/>   <!-- -1.5708     1.5708  -->
     </joint>
     <link name="${arm_id}_link6">
@@ -188,9 +190,10 @@
       </inertial>
     </link>
-    <joint name="id_5" type="continuous">
+    <joint name="id_5" type="revolute">
       <origin rpy="0 0 0" xyz="0 -0.00607092 0.027"/>
       <parent link="${arm_id}_link5"/>
       <child link="${arm_id}_link6"/>
       <axis xyz="0 1 0" rpy="0 0 0"/>
+      <limit effort="1000.0" lower="-3.14" upper="3.14" velocity="0.5"/> <!-- -1.5708     1.5708  -->
     </joint>
     <transmission name="trans_timon_joint1">

Commit message: change planning settings

File: manipulator_description/robots/timon_arm.xacro (robot description, xacro)
@@ -64,5 +64,5 @@
       <child link="${arm_id}_link1"/>
       <axis xyz="0 0 1" rpy="0 0 0"/>
-      <limit effort="1000.0" lower="-1.5" upper="1.5" velocity="0.5"/> <!--  -0.783    0.783-->
+      <limit effort="1000.0" lower="-3.14" upper="3.14" velocity="0.5"/> <!--  -0.783    0.783-->
     </joint>
     <link name="${arm_id}_link2">

Commit message: add real box and aruco start script

File: manipulator_description/robots/timon_arm.xacro (robot description, xacro)
@@ -168,5 +168,5 @@
       <parent link="${arm_id}_link4"/>
       <child link="${arm_id}_link5"/>
-      <axis xyz="0 0 1"/>
+      <axis xyz="0 0 -1"/>
       <limit effort="1000.0" lower="-3.14" upper="3.14" velocity="0.5"/>   <!-- -1.5708     1.5708  -->
     </joint>

File: manipulator_description/robots/timon_arm_hand_base.urdf.xacro (robot description, xacro)
@@ -3,12 +3,12 @@
   <link name = "world">
   </link>
-  <xacro:include filename="$(find manipulator_description)/robots/base.xacro"/>
+  <!-- <xacro:include filename="$(find manipulator_description)/robots/base.xacro"/> -->
   <xacro:include filename="$(find manipulator_description)/robots/timon_arm.urdf.xacro"/>
    <xacro:include filename="$(find manipulator_description)/robots/camera.xacro"/>
-    <joint name ="world_to_base" type="fixed">
+    <!-- <joint name ="world_to_base" type="fixed">
         <origin rpy="0 0 0" xyz="0.0 0 -0.01"/>
         <parent link="world"/>
         <child link = "base_to_manipulator"/>
-    </joint>
+    </joint> -->
     <joint name ="base_to_timon" type="fixed">
         <origin rpy="0 0 0" xyz="0 0 0"/>

File: manipulator_description/urdf/botao.xacro (robot description, xacro)
@@ -23,14 +23,12 @@
   </link>
  <joint name="caixa_to_botao" type="fixed">
-    <parent link="caixa"/>
+    <parent link="box_link"/>
     <child link="botao"/>
-    <origin rpy="0 0 0" xyz="0 0.215 0.1165"/> <!--vertical: rpy="1.571 0 0" xyz="0 -0.1165 0.215" --> <!-- horizontal: rpy="0 0 0" xyz="0 0.215 0.1165"-->
-    <!-- <axis xyz="0 1 0"/>
-    <limit lower="0.0" upper="0.00" effort="1" velocity="1"/> -->
+    <origin rpy="0 0 0" xyz="0 0 0"/>
   </joint>
   <joint name ="botao_fake" type ="fixed">
     <parent link="botao"/>
     <child link="fake_botao"/>
-    <origin rpy="0.0 0.0 0.0" xyz="0.0 0.0 0.1"/>
+    <origin rpy="0.0 0.0 0.0" xyz="0.0 0.0 0.2"/>
   </joint>
 </robot>

File: manipulator_description/urdf/box.urdf.xacro (robot description, xacro)
@@ -3,11 +3,11 @@
   <link name ="box_link">
   </link>
-  <xacro:include filename="$(find manipulator_description)/urdf/caixa.xacro"/>
+  <!-- <xacro:include filename="$(find manipulator_description)/urdf/caixa.xacro"/> -->
+  <xacro:include filename="$(find manipulator_description)/urdf/botao.xacro"/>
   <xacro:include filename="$(find manipulator_description)/urdf/tag.xacro"/>
-  <xacro:include filename="$(find manipulator_description)/urdf/botao.xacro"/>
-  <joint name="base_to_box" type="fixed">
-    <origin xyz="-0.4 0.0 1.66" rpy="0 0 -1.571"/>   <!--vertical: xyz="-0.4 0.0 1.56" rpy="0 0 1.571"--> <!-- horizontal: xyz="-0.4 0.0 1.66" rpy="0 0 -1.571"-->
+  <!-- <joint name="base_to_box" type="fixed">
+    <origin xyz="0 0 0" rpy="0 0 -1.571"/>
     <parent link="box_link"/>
-    <child link="caixa"/>
-  </joint>
+    <child link="botao"/>
+  </joint> -->
 </robot>

File: manipulator_description/urdf/tag.xacro (robot description, xacro)
@@ -28,5 +28,5 @@
         </gazebo>
     <joint name="box_to_tag" type="fixed">
-        <origin rpy="0 0 3.1415" xyz="0.0 -0.1 -0.013"/> <!--caixa na vertical: rpy="0 0 0" -->  <!-- horizontal: rpy="0 0 3.1415" -->
+        <origin rpy="0 0 3.1415" xyz="0.0 0.06 0"/> <!--caixa na vertical: rpy="0 0 0" -->  <!-- horizontal: rpy="0 0 3.1415" -->
         <parent link="botao"/>
         <child link = "tag_aruco_4"/>

Commit message: update test code & add objects code

File: manipulator_description/robots/timon_arm.xacro (robot description, xacro)
@@ -64,5 +64,5 @@
       <child link="${arm_id}_link1"/>
       <axis xyz="0 0 1" rpy="0 0 0"/>
-      <limit effort="1000.0" lower="-3.14" upper="3.14" velocity="0.5"/> <!--  -0.783    0.783-->
+      <limit effort="1000.0" lower="-0.8" upper="0.8" velocity="0.5"/> <!--  -0.783    0.783-->
     </joint>
     <link name="${arm_id}_link2">
@@ -90,5 +90,5 @@
       <child link="${arm_id}_link2"/>
       <axis xyz="-1 0 0" rpy="0 0 0"/>
-      <limit effort="1000.0" lower="-3.14" upper="3.14" velocity="0.5"/> <!-- -1.5708   1.5708-->
+      <limit effort="1000.0" lower="-1.5708" upper="1.5708" velocity="0.5"/> <!-- -1.5708   1.5708-->
     </joint>
     <link name="${arm_id}_link3">
@@ -116,5 +116,5 @@
       <child link="${arm_id}_link3"/>
       <axis xyz="-1 0 0" rpy="0 0 0"/>
-      <limit effort="1000.0" lower="-3.14" upper="3.14" velocity="0.5"/>  <!-- -0.74    3.03-->
+      <limit effort="1000.0" lower="-0.74" upper="3.03" velocity="0.5"/>  <!-- -0.74    3.03-->
     </joint>
     <link name="${arm_id}_link4">
@@ -169,5 +169,5 @@
       <child link="${arm_id}_link5"/>
       <axis xyz="0 0 -1"/>
-      <limit effort="1000.0" lower="-3.14" upper="3.14" velocity="0.5"/>   <!-- -1.5708     1.5708  -->
+      <limit effort="1000.0" lower="-1.5708" upper="1.5708" velocity="0.5"/>   <!-- -1.5708     1.5708  -->
     </joint>
     <link name="${arm_id}_link6">
@@ -195,5 +195,5 @@
       <child link="${arm_id}_link6"/>
       <axis xyz="0 1 0" rpy="0 0 0"/>
-      <limit effort="1000.0" lower="-3.14" upper="3.14" velocity="0.5"/> <!-- -1.5708     1.5708  -->
+      <limit effort="1000.0" lower="-1.5708" upper="1.5708" velocity="0.5"/> <!-- -1.5708     1.5708  -->
     </joint>
     <transmission name="trans_timon_joint1">

File: manipulator_description/urdf/botao.xacro (robot description, xacro)
@@ -30,5 +30,5 @@
     <parent link="botao"/>
     <child link="fake_botao"/>
-    <origin rpy="0.0 0.0 0.0" xyz="0.0 0.0 0.2"/>
+    <origin rpy="0.0 0.0 0.0" xyz="0.0 0.0 0.25"/>
   </joint>
 </robot>

File: manipulator_description/urdf/botao_vertical.xacro (robot description, xacro)
@@ -32,5 +32,5 @@
     <parent link="botao"/>
     <child link="fake_botao"/>
-    <origin rpy="0.0 0.0 0.0" xyz="0.0 0.0 0.1"/>
+    <origin rpy="0.0 0.0 0.0" xyz="0.0 0.0 1.0"/>
   </joint>
 </robot>

Commit message: fix base orientation

File: manipulator_description/robots/timon_arm.xacro (robot description, xacro)
@@ -36,5 +36,5 @@
     </link>
      <joint name ="invisble_joint" type="fixed">
-        <origin rpy="0 0 0" xyz="0 0 0"/>
+        <origin rpy="0 0 3.14" xyz="0 0 0"/>
         <parent link="invisible_link"/>
         <child link = "${arm_id}_link0"/>

Commit message: Set a new moveit setup assistant

File: manipulator_description/robots/timon_arm.xacro (robot description, xacro)
@@ -64,5 +64,5 @@
       <child link="${arm_id}_link1"/>
       <axis xyz="0 0 1" rpy="0 0 0"/>
-      <limit effort="1000.0" lower="-0.8" upper="0.8" velocity="0.5"/> <!--  -0.783    0.783-->
+      <limit effort="1000.0" lower="-0.8" upper="0.8" velocity="0.5"/>
     </joint>
     <link name="${arm_id}_link2">
@@ -90,5 +90,5 @@
       <child link="${arm_id}_link2"/>
       <axis xyz="1 0 0" rpy="0 0 0"/>
-      <limit effort="1000.0" lower="-1.5708" upper="1.5708" velocity="0.5"/> <!-- -1.5708   1.5708-->
+      <limit effort="1000.0" lower="-1.5708" upper="1.5708" velocity="0.5"/>
     </joint>
     <link name="${arm_id}_link3">
@@ -116,31 +116,6 @@
       <child link="${arm_id}_link3"/>
       <axis xyz="1 0 0" rpy="0 0 0"/>
-      <limit effort="1000.0" lower="-0.74" upper="3.03" velocity="0.5"/>  <!-- -0.74    3.03-->
+      <limit effort="1000.0" lower="-0.74" upper="3.03" velocity="0.5"/>
     </joint>
-    <!-- <link name="${arm_id}_link4">
-      <visual>
-        <origin xyz="0 0 0" rpy="0 0 0" />
-        <geometry>
-          <mesh filename="package://${description_pkg}/meshes/JeRoTIMON/suport_cam.dae"/>
-        </geometry>
-      </visual>
-      <collision>
-        <origin xyz="0 0 0" rpy="0 0 0" />
-        <geometry>
-          <mesh filename="package://${description_pkg}/meshes/JeRoTIMON/suport_cam.dae"/>
-        </geometry>
-      </collision>
-      <inertial>
-        <origin xyz="0 0 0" rpy="0 0 0 "/>
-        <mass value="0.20608656"/>
-        <inertia ixx="0.00039102"  ixy="0"  ixz="-8.254e-9" iyy="0.00045673" iyz="-0.00006629" izz="0.00023588" />
-      </inertial>
-    </link>
-    <joint name="suport_cam" type="fixed">
-      <origin rpy="0 0.0 3.1415" xyz="-0.00754115 -0.03075116 0.37653086"/>
-      <parent link="${arm_id}_link3"/>
-      <child link="${arm_id}_link4"/>
-      <axis xyz="0 0 0" rpy="0 0 0"/>
-    </joint> -->
     <link name="${arm_id}_link4">
       <visual>
@@ -164,36 +139,9 @@
     <joint name="id_4" type="revolute">
       <safety_controller k_position="100.0" k_velocity="40.0" soft_lower_limit="-2.974" soft_upper_limit="2.974"/>
-      <origin rpy="0 0 0" xyz="0.00025000 0.02278775 0.44101451"/>
-      <!-- 0.00739115 -->
+      <origin rpy="0 0 0" xyz="0.00025000 0.03075115 0.44053087"/>
       <parent link="${arm_id}_link3"/>
       <child link="${arm_id}_link4"/>
       <axis xyz="0 0 -1"/>
-      <limit effort="1000.0" lower="-2.974" upper="2.974" velocity="0.5"/>   <!-- -1.5708     1.5708  -->
-    </joint>
-    <link name="${arm_id}_link5">
-      <visual>
-        <origin xyz="0.0 0.0 0.0" rpy="0 0 0" />
-        <geometry>
-          <mesh filename="package://${description_pkg}/meshes/JeRoTIMON/id_6.dae"/>
-        </geometry>
-      </visual>
-      <collision>
-        <origin xyz="0.0 0.0 0.0" rpy="0 0 0" />
-        <geometry>
-          <mesh filename="package://${description_pkg}/meshes/JeRoTIMON/id_6.dae"/>
-        </geometry>
-      </collision>
-      <inertial>
-        <origin xyz="0.0 0.0 0.0" rpy="0 0 0 "/>
-        <mass value="0.08694786"/>
-        <inertia ixx="0.00012963"  ixy="0"  ixz="0" iyy="0.00012601" iyz="-0.00000408" izz="0.00003715" />
-      </inertial>
-    </link>
-    <joint name="id_5" type="revolute">
-      <origin rpy="0 0 0" xyz="0 0 0.02699559"/>
-      <parent link="${arm_id}_link4"/>
-      <child link="${arm_id}_link5"/>
-      <axis xyz="0 1 0" rpy="0 0 0"/>
-      <limit effort="1000.0" lower="-1.5708" upper="1.5708" velocity="0.5"/> <!-- -1.5708     1.5708  -->
+      <limit effort="1000.0" lower="-2.974" upper="2.974" velocity="0.5"/>
     </joint>
     <transmission name="trans_timon_joint1">
@@ -237,167 +185,4 @@
         </actuator>
     </transmission>
-    <transmission name="trans_timon_joint5">
-        <type>transmission_interface/SimpleTransmission</type>
-        <joint name="id_5">
-            <hardwareInterface>hardware_interface/PositionJointInterface</hardwareInterface>
-        </joint>
-        <actuator name="timon_joint5_motor">
-            <hardwareInterface>hardware_interface/PositionJointInterface</hardwareInterface>
-            <mechanicalReduction>1</mechanicalReduction>
-        </actuator>
-    </transmission>
-<!--
-    <link name="${arm_id}_link6">
-      <visual>
-        <origin xyz="0.0 0.0 0.0" rpy="0 0 0.75" />
-        <geometry>
-          <mesh filename="package://${description_pkg}/meshes/visual/link7.dae"/>
-        </geometry>
-      </visual>
-      <collision>
-        <origin xyz="0.0 0.0 0.0" rpy="0 0 0.75" />
-        <geometry>
-          <mesh filename="package://${description_pkg}/meshes/visual/link7.dae"/>
-        </geometry>
-      </collision>
-      <inertial>
-        <origin xyz="0.0 0.0 0.0" rpy="0 0 0.75 "/>
-        <mass value="0.16499216"/>
-        <inertia ixx="7.88952550e-5"  ixy="-3.13065901e-9"  ixz="4.40693303e-9" iyy="4.39861799e-5" iyz="-2.02737764e-6" izz="6.23603662e-5" />
-      </inertial>
-    </link>
-    <joint name="${arm_id}_joint6" type="fixed">
-      <origin rpy="0 3.14 0" xyz="0.0 0.0 -0.05"/>
-      <parent link="${arm_id}_link5"/>
-      <child link="${arm_id}_link6"/>
-    </joint>
-    <link name="${arm_id}_link7">
-      <visual>
-        <origin xyz="-0.01 0.015 0.0" rpy="0.0 1.571 0.0" />
-        <geometry>
-          <mesh filename="package://${description_pkg}/meshes/visual/link8.dae"/>
-        </geometry>
-      </visual>
-      <collision>
-        <origin xyz="-0.01 0.015 0.0" rpy="0.0 1.571 0.0" />
-        <geometry>
-          <mesh filename="package://${description_pkg}/meshes/visual/link8.dae"/>
-        </geometry>
-      </collision>
-      <inertial>
-        <origin xyz="-0.01 0.015 0.0" rpy="0.0 1.571 0.0"/>
-        <mass value="0.58301843"/>
-        <inertia ixx="7.66412604e-3"  ixy="9.16805313e-10"  ixz="2.16130814e-14" iyy="5.98440184e-4" iyz="4.07885374e-6" izz="7.70339943e-3" />
-      </inertial>
-    </link>
-    <joint name="${arm_id}_joint7" type="revolute">
-      <safety_controller k_position="100.0" k_velocity="40.0" soft_lower_limit="-0.95" soft_upper_limit="2.36"/>
-      <origin rpy="0.0 0.0 0.0" xyz="0.0 0.001 -0.0375"/>
-      <parent link="${arm_id}_link6"/>
-      <child link="${arm_id}_link7"/>
-      <axis xyz="0 0 1"/>
-      <limit effort="1000.0" lower="-0.95" upper="2.36" velocity="0.5"/>
-    </joint>
-    <link name="${arm_id}_link8">
-      <visual>
-        <origin xyz="0.0 0.0 0.0" rpy="0.0 0.0 0.0" />
-        <geometry>
-          <mesh filename="package://manipulator_description/meshes/visual/link9.dae"/>
-        </geometry>
-      </visual>
-      <collision>
-        <origin xyz="0.0 0.0 0.0" rpy="0.0 0.0 0.0" />
-        <geometry>
-          <mesh filename="package://manipulator_description/meshes/visual/link9.dae"/>
-        </geometry>
-      </collision>
-      <inertial>
-        <origin xyz="0.0 0.0 0.0" rpy="0.0 0.0 0.0"/>
-        <mass value="0.16499216"/>
-        <inertia ixx="7.88952550e-5"  ixy="-3.13065901e-9"  ixz="4.40693303e-9" iyy="4.39861799e-5" iyz="-2.02737764e-6" izz="6.23603662e-5" />
-      </inertial>
-    </link>
-    <joint name="${arm_id}_joint8" type="fixed">
-      <origin rpy="0 -1.571 -1.571" xyz="0 0.41 0.013"/>
-      <parent link="${arm_id}_link7"/>
-      <child link="${arm_id}_link8"/>
-    </joint>
-    <link name="${arm_id}_link9">
-      <visual>
-        <origin xyz="0.0 0.0 0.0" rpy="1.571 0.0 0.0" />
-        <geometry>
-          <mesh filename="package://manipulator_description/meshes/visual/link10.dae"/>
-        </geometry>
-      </visual>
-      <collision>
-        <origin xyz="0.0 0.0 0.0" rpy="1.571 0.0 0.0" />
-        <geometry>
-          <mesh filename="package://manipulator_description/meshes/visual/link10.dae"/>
-        </geometry>
-      </collision>
-      <inertial>
-        <origin xyz="0.0 0.0 0.0" rpy="1.571 0.0 0.0"/>
-        <mass value="0.007"/>
-        <inertia ixx="1.48840827e-6"  ixy="2.49592487e-8"  ixz="5.30644674e-12" iyy="2.08108627e-6" iyz="2.38181240e-14" izz="6.88193128e-7" />
-      </inertial>
-    </link>
-    <joint name="${arm_id}_joint9" type="continuous">
-      <origin rpy="0 0 1.571" xyz="0 0 0.025"/>
-      <parent link="${arm_id}_link8"/>
-      <child link="${arm_id}_link9"/>
-      <axis xyz="0 0 1" rpy="0 0 0"/>
-    </joint>
-    <link name="${arm_id}_link10">
-      <visual>
-        <origin xyz="0.0225 -0.007 0.0" rpy="0.0 0.0 0.0" />
-        <geometry>
-          <mesh filename="package://manipulator_description/meshes/visual/link11.dae"/>
-        </geometry>
-      </visual>
-      <collision>
-        <origin xyz="0.0225 -0.007 0.0" rpy="0.0 0.0 0.0" />
-        <geometry>
-          <mesh filename="package://manipulator_description/meshes/visual/link11.dae"/>
-        </geometry>
-      </collision>
-      <inertial>
-        <origin xyz="0.0225 -0.007 0.0" rpy="0.0 0.0 0.0"/>
-        <mass value="0.16499216"/>
-        <inertia ixx="7.88952550e-5"  ixy="-3.13065901e-9"  ixz="4.40693303e-9" iyy="4.39861799e-5" iyz="-2.02737764e-6" izz="6.23603662e-5" />
-      </inertial>
-    </link>
-    <joint name="${arm_id}_joint10" type="fixed">
-      <origin rpy="1.5701 0.0 0.0" xyz="0.0 -0.001 0.055"/>
-      <parent link="${arm_id}_link9"/>
-      <child link="${arm_id}_link10"/>
-    </joint>
-   <link name="${arm_id}_link11">
-      <visual>
-        <origin xyz="0.0 0.0 0.0" rpy="0.0 1.571 0.0" />
-        <geometry>
-          <mesh filename="package://manipulator_description/meshes/visual/link12.dae"/>
-        </geometry>
-      </visual>
-      <collision>
-        <origin xyz="0.0 0.0 0.0" rpy="0.0 1.571 0.0" />
-        <geometry>
-          <mesh filename="package://manipulator_description/meshes/visual/link12.dae"/>
-        </geometry>
-      </collision>
-      <inertial>
-        <origin xyz="0.0 0.0 0.0" rpy="0.0 1.571 0.0"/>
-        <mass value="0.01873963"/>
-        <inertia ixx="4.49588271e-6"  ixy="0.00000000e+0"  ixz="0.00000000e+0" iyy="1.08113872e-5" iyz="0.00000000e+0" izz="1.12040418e-5" />
-      </inertial>
-    </link>
-    <joint name="${arm_id}_joint11" type="revolute">
-      <safety_controller k_position="100.0" k_velocity="40.0" soft_lower_limit="-1.90" soft_upper_limit="1.90"/>
-      <origin rpy="0.0 0.0 0.0" xyz="0.0 0.0 0.0"/>
-      <parent link="${arm_id}_link10"/>
-      <child link="${arm_id}_link11"/>
-      <axis xyz="0 0 1"/>
-      <limit effort="1000.0" lower="-1.90" upper="1.90" velocity="0.5"/>
-    </joint>
- -->
   </xacro:macro>
 </robot>

File: manipulator_description/robots/timon_arm_hand_base.urdf.xacro (robot description, xacro)
@@ -3,12 +3,5 @@
   <link name = "world">
   </link>
-  <!-- <xacro:include filename="$(find manipulator_description)/robots/base.xacro"/> -->
   <xacro:include filename="$(find manipulator_description)/robots/timon_arm.urdf.xacro"/>
-   <xacro:include filename="$(find manipulator_description)/robots/camera.xacro"/>
-    <!-- <joint name ="world_to_base" type="fixed">
-        <origin rpy="0 0 0" xyz="0.0 0 -0.01"/>
-        <parent link="world"/>
-        <child link = "base_to_manipulator"/>
-    </joint> -->
     <joint name ="base_to_timon" type="fixed">
         <origin rpy="0 0 0" xyz="0 0 0"/>
@@ -16,9 +9,3 @@
         <child link = "invisible_link"/>
     </joint>
-    <joint name ="base_to_camera" type="fixed">
-        <origin rpy="-1.5701 -1.5701 0" xyz="0.00015000 0.10012477 0.39638054"/>
-        <!-- <origin rpy="-1.571 3.1415 -1.571" xyz="0.0661 0.426 0.0123"/> -->
-        <parent link="timon_link3"/>
-        <child link = "camera"/>
-    </joint>
 </robot>
